File: pcb_test/test/test.kicad_sch (KiCad schematic)
At the start: 13 parts, among them T2 BC817, T3 BC847BPN

Commit message: WIP
Parts:
- added C1: TBD, Capacitor_THT:CP_Radial_D8.0mm_P3.50mm, symbol Device:C_Small
Connections:
- net GND: now also C1.2
- net at C2.1, R16.1, T3.4 (E2): now also C1.1
Changed lines of the file:
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@@
+	)
+	(junction
+		(at 120.65 102.87)
+		(diameter 0)
+		(color 0 0 0 0)
 	)
 	(junction
@@
 	(wire
 		(pts
+			(xy 120.65 102.87) (xy 120.65 110.49)
+		)
+		(stroke
+			(width 0)
+			(type default)
+		)
+	)
+	(wire
+		(pts
 			(xy 69.85 86.36) (xy 69.85 87.63)
 		)
@@
 	(wire
 		(pts
+			(xy 120.65 102.87) (xy 127 102.87)
+		)
+		(stroke
+			(width 0)
+			(type default)
+		)
+	)
+	(wire
+		(pts
 			(xy 80.01 125.73) (xy 80.01 121.92)
 		)
@@
 	(wire
 		(pts
+			(xy 120.65 119.38) (xy 120.65 115.57)
+		)
+		(stroke
+			(width 0)
+			(type default)
+		)
+	)
+	(wire
+		(pts
 			(xy 62.23 87.63) (xy 62.23 88.9)
 		)
@@
 	(wire
 		(pts
-			(xy 86.36 102.87) (xy 127 102.87)
+			(xy 86.36 102.87) (xy 120.65 102.87)
 		)
 		(stroke
@@
 	)
 	(symbol
+		(lib_id "power:GND")
+		(at 120.65 119.38 0)
+		(unit 1)
+		(exclude_from_sim no)
+		(in_bom yes)
+		(on_board yes)
+		(dnp no)
+		(property "Reference" "#PWR01"
+			(at 120.65 125.73 0)
+			(effects
+				(font
+					(size 1.27 1.27)
+				)
+				(hide yes)
+			)
+		)
+		(property "Value" "GND"
+			(at 122.682 123.444 0)
+			(effects
+				(font
+					(size 1.27 1.27)
+				)
+				(justify right)
+			)
+		)
+		(property "Footprint" ""
+			(at 120.65 119.38 0)
+			(effects
+				(font
+					(size 1.27 1.27)
+				)
+				(hide yes)
+			)
+		)
+		(property "Datasheet" ""
+			(at 120.65 119.38 0)
+			(effects
+				(font
+					(size 1.27 1.27)
+				)
+				(hide yes)
+			)
+		)
+		(property "Description" "Power symbol creates a global label with name \"GND\" , ground"
+			(at 120.65 119.38 0)
+			(effects
+				(font
+					(size 1.27 1.27)
+				)
+				(hide yes)
+			)
+		)
+		(pin "1"
+		)
+		(instances
+			(project "test"
+				(path "/4a6824fc-4e09-4227-a791-1eeca3a5516c"
+					(reference "#PWR01")
+					(unit 1)
+				)
+			)
+		)
+	)
+	(symbol
 		(lib_name "GND_1")
 		(lib_id "power:GND")
@@
 					(unit 1)
 				)
+			)
+		)
+	)
+	(symbol
+		(lib_id "Device:C_Small")
+		(at 120.65 113.03 0)
+		(unit 1)
+		(exclude_from_sim no)
+		(in_bom yes)
+		(on_board yes)
+		(dnp no)
+		(property "Reference" "C1"
+			(at 116.078 112.014 0)
+			(effects
+				(font
+					(size 1 1)
+				)
+				(justify left)
+			)
+		)
+		(property "Value" "TBD"
+			(at 116.078 114.554 0)
+			(effects
+				(font
+					(size 1 1)
+				)
+				(justify left)
+			)
+		)
+		(property "Footprint" "Capacitor_THT:CP_Radial_D8.0mm_P3.50mm"
+			(at 120.65 113.03 0)
+			(effects
+				(font
+					(size 1.27 1.27)
+				)
+				(hide yes)
+			)
+		)
+		(property "Datasheet" "~"
+			(at 120.65 113.03 0)
+			(effects
+				(font
+					(size 1.27 1.27)
+				)
+				(hide yes)
+			)
+		)
+		(property "Description" "Unpolarized capacitor, small symbol"
+			(at 120.65 113.03 0)
+			(effects
+				(font
+					(size 1.27 1.27)
+				)
+				(hide yes)
+			)
+		)
+		(pin "1"
+		)
+		(pin "2"
+		)
+		(instances
+			(project "test"
+				(path "/4a6824fc-4e09-4227-a791-1eeca3a5516c"
+					(reference "C1")
+					(unit 1)
+				)

Commit message: WIP
Parts:
- added D1: 5V6, Diode_SMD:D_MiniMELF, symbol Device:D_Zener
- added D2, D5, D6: LED, LED_THT:LED_D3.0mm_Horizontal_O1.27mm_Z2.0mm, symbol Device:LED
- added D4: 1N4148W, Diode_SMD:D_SOD-123, symbol Diode:1N4148W
- added D7: LL4148, Diode_SMD:D_MiniMELF, symbol Diode:LL4148
- added J1: M- Eingang, Connector_PinHeader_2.54mm:PinHeader_1x01_P2.54mm_Vertical, symbol Connector:Conn_01x01_Pin
- added J2: P Eingang 24V, Connector_PinHeader_2.54mm:PinHeader_1x01_P2.54mm_Vertical, symbol Connector:Conn_01x01_Pin
- added J3, J4: BUS IN, Connector_PinHeader_2.54mm:PinHeader_1x01_P2.54mm_Vertical, symbol Connector:Conn_01x01_Pin
- added K1: Fujitsu_FTR-LYAA005x, Relay_THT:Relay_SPST-NO_Fujitsu_FTR-LYAA005x_FormA_Vertical, symbol Relay:Fujitsu_FTR-LYAA005x
- added R1: 47K, Resistor_SMD:R_0805_2012Metric, symbol Device:R
- added R15, R18, R19: 680, Resistor_SMD:R_0805_2012Metric, symbol Device:R
- added R17, R6: 470, Resistor_SMD:R_0805_2012Metric, symbol Device:R
- added R3: 2K2, Resistor_SMD:R_0805_2012Metric, symbol Device:R
- added R4: 100K, Resistor_SMD:R_0805_2012Metric, symbol Device:R
- added R5: 6K8, Resistor_SMD:R_0805_2012Metric, symbol Device:R
- added S1: SW_Push, Button_Switch_THT:SW_Tactile_SPST_Angled_PTS645Vx31-2LFS, symbol Switch:SW_Push
- added T1, T7: BC817, Package_TO_SOT_SMD:SOT-23, symbol Transistor_BJT:BC817
- added U1: PIC16F627A-ISS, Package_SO:SSOP-20_4.4x6.5mm_P0.65mm, symbol MCU_Microchip_PIC16:PIC16F627A-ISS
- C1: value TBD -> 47uF; footprint Capacitor_THT:CP_Radial_D8.0mm_P3.50mm -> Capacitor_THT:CP_Radial_D4.0mm_P1.50mm
- C2: value TBD -> 100nF
- D3: footprint Diode_SMD:D_1206_3216Metric -> Diode_SMD:D_MELF
- renumbered D7 to D10
Connections:
- net MCU PIN UNTEN LINKS is gone; now on net VDD: R16.2
- net GND: now also C2.2, D1.2 (A), D2.2 (A), D5.2 (A), D6.2 (A), R3.1, S1.2, T7.2 (E), U1.5 (VSS), U1.6 (VSS)
- net VDD: now reaches C1.1, C2.1, T3.4 (E2)
- net VDD: now also R14.1, T1.2 (E), U1.15 (VDD), U1.16 (VDD); no longer R16.1
- net BUS_WIRE1: no longer names the net of D10.1
- net BUS_WIRE1: now also J4.1 (Pin_1)
- net BUS_WIRE2: no longer names the net of D10.2
- net BUS_WIRE2: now also J3.1 (Pin_1)
- net MCU 2 PIN UNTEN LINKS renamed RB2
- net RB2: now also U1.9 (RB2/TX/CK)
- net MCU PIN 4 LINKS: no longer names the net of R14.2
- net MCU PIN 4 LINKS: now also U1.4 (~{MCLR}/Vpp/RA5)
- removed net MCU PIN MITTE RECHTS: C2.2, R14.1
- net MCU PIN UNTEN RECHTS renamed RB4
- net RB4: now also U1.11 (RB4/PGM)
- new net: D4.1 (K), D7.1 (K), K1.A2, R1.2, R6.2
- new net: D7.2 (A), K1.A1, T7.3 (C)
- new net: D2.1 (K), R15.1
- new net: D5.1 (K), R19.1
- new net: R17.1, T7.1 (B)
- new net: D1.1 (K), R1.1, T1.1 (B)
- new net: D6.1 (K), R18.1
- new net: R6.1, T1.3 (C)
- new net: D4.2 (A), J2.1 (Pin_1)
- new net: J1.1 (Pin_1), R5.1
- new net: R3.2, R4.1, R5.2
- new net RB1: R17.2, R18.2, U1.8 (RB1/RX/DT)
- new net RB3: R16.1, S1.1, U1.10 (RB3/CCP1)
- new net RB5: R4.2, U1.12 (RB5)
- new net RB6: R15.2, U1.13 (RB6/T1OSC0/T1CKI/PGC)
- new net RB7: R19.2, U1.14 (RB7/T1OSI/PGD)
- no-connect marks 0 -> 10
Other:
- note added: "BUS TX"
- note added: "INPUT STATUS LED"
- note added: "PROGRAMMING MODE BUTTON"
- note added: "PROGRAMMING MODE LED"
- note added: "RELAY STATUS LED"
- note added: "Spannungseingang für PIC uC"
- note added: "Wahrscheinlich BUS RX"
- note removed: "Wahrscheinlich BUS TX"
- moved on the sheet: C1, C2, D10, D3, R10, R11, R12, R14, R16, R7, R8, R9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
