File: pcb/doorman.kicad_sch (KiCad schematic)
At the start: 42 parts, among them J1 USB_C_Receptacle_USB2.0, J2 Terminal, J3 3V3 Test Pad, J4 Conn_02x07_Odd_Even, J6 BUS Test Pad, J7 BUS RX Test Pad, J8 TX Test Pad, J9 RX Test Pad, Q1 BC847BPN, Q2 BC817, SW1 Reset Button, SW2 Flash Button, U2 AP63203WU, U3 GAQY252G3S, U4 ESP32-S3-MINI-1

Commit message: FIX
Connections:
- net +3.3V: now also Q1.4 (E2); no longer Q1.3 (C2)
- net BUS_RX: now also Q1.3 (C2); no longer Q1.4 (E2)
Changed lines of the file:
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@@
 	(title_block
 		(title "Doorman S3")
-		(date "2026-02-04")
+		(date "2026-02-05")
 		(rev "2.0")
 		(comment 1 "TC:Bus Intercom Gateway")
@@
 		(lib_id "Transistor_BJT:BC847BPN")
 		(at 191.77 104.14 0)
+		(mirror x)
 		(unit 2)
 		(exclude_from_sim no)
@@
 		(dnp no)
 		(property "Reference" "Q1"
-			(at 196.596 103.378 0)
+			(at 196.596 104.902 0)
 			(effects
 				(font
@@
 		)
 		(property "Value" "BC847BPN"
-			(at 196.596 104.9019 0)
+			(at 196.596 103.3781 0)
 			(effects
 				(font
@@
 		)
 		(property "Footprint" "Package_TO_SOT_SMD:SOT-363_SC-70-6"
-			(at 196.85 101.6 0)
+			(at 196.85 106.68 0)
 			(effects
 				(font

Commit message: WIP
Parts:
- R10: value 62 -> 62R
- R11, R8: value 1.2 -> 1R2
- R12, R5: value 39K -> 47K5; LCSC C23153 -> C22375093; MPN 0603WAF3902T5E -> FRC0603F47R5TS
- R2: value 2.2K -> 2K2
- R3: value 5.1K -> 5K1
- R7: value 470 -> 470R
- R9: value 150 -> 150R
Changed lines of the file:
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@@
 			)
 		)
-		(property "Value" "39K"
+		(property "Value" "47K5"
 			(at 194.31 118.11 90)
 			(effects
@@
 			)
 		)
-		(property "Description" "-55℃~+155℃ 100mW 39kΩ 75V Thick Film Resistor ±1% ±100ppm/℃ 0603 Chip Resistor - Surface Mount ROHS"
+		(property "Description" "-55℃~+155℃ 100mW 47.5Ω 75V Thick Film Resistor ±1% ±100ppm/℃ 0603 Chip Resistor - Surface Mount ROHS"
 			(at 194.31 118.11 0)
 			(effects
@@
 			)
 		)
-		(property "LCSC" "C23153"
+		(property "LCSC" "C22375093"
 			(at 194.31 118.11 0)
 			(effects
@@
 			)
 		)
-		(property "MPN" "0603WAF3902T5E"
+		(property "MPN" "FRC0603F47R5TS"
 			(at 194.31 118.11 0)
 			(effects
@@
 			)
 		)
-		(property "Value" "1.2"
+		(property "Value" "1R2"
 			(at 144.78 119.38 90)
 			(effects
@@
 			)
 		)
-		(property "Value" "150"
+		(property "Value" "150R"
 			(at 39.37 157.48 90)
 			(effects
@@
 			)
 		)
-		(property "Value" "5.1K"
+		(property "Value" "5K1"
 			(at 264.16 76.2 90)
 			(effects
@@
 			)
 		)
-		(property "Value" "2.2K"
+		(property "Value" "2K2"
 			(at 128.27 104.14 90)
 			(effects
@@
 			)
 		)
-		(property "Value" "62"
+		(property "Value" "62R"
 			(at 114.3 35.56 90)
 			(effects
@@
 			)
 		)
-		(property "Value" "39K"
+		(property "Value" "47K5"
 			(at 179.07 93.98 90)
 			(effects
@@
 			)
 		)
-		(property "Description" "-55℃~+155℃ 100mW 39kΩ 75V Thick Film Resistor ±1% ±100ppm/℃ 0603 Chip Resistor - Surface Mount ROHS"
+		(property "Description" "-55℃~+155℃ 100mW 47.5Ω 75V Thick Film Resistor ±1% ±100ppm/℃ 0603 Chip Resistor - Surface Mount ROHS"
 			(at 179.07 93.98 0)
 			(effects
@@
 			)
 		)
-		(property "LCSC" "C23153"
+		(property "LCSC" "C22375093"
 			(at 179.07 93.98 0)
 			(effects
@@
 			)
 		)
-		(property "MPN" "0603WAF3902T5E"
+		(property "MPN" "FRC0603F47R5TS"
 			(at 179.07 93.98 0)
 			(effects
@@
 			)
 		)
-		(property "Value" "470"
+		(property "Value" "470R"
 			(at 138.43 154.94 90)
 			(effects
@@
 			)
 		)
-		(property "Value" "1.2"
+		(property "Value" "1R2"
 			(at 147.32 119.38 90)
 			(effects

Commit message: WIP
Parts:
- J1: value USB_C_Receptacle_USB2.0 -> USB-C Connector
- J2: value Terminal -> Screw Terminals
- J4: value Conn_02x07_Odd_Even -> Extension Board Connector
Other:
- note removed: "Extension Board Connector"
- note removed: "Screw Terminals"
Changed lines of the file:
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@@
 	(title_block
 		(title "Doorman S3")
-		(date "2026-02-05")
+		(date "2026-02-10")
 		(rev "2.0")
 		(comment 1 "TC:Bus Intercom Gateway")
 	)
-	(text "Screw Terminals"
-		(exclude_from_sim no)
-		(at 240.03 125.984 0)
-		(effects
-			(font
-				(size 1.27 1.27)
-			)
-			(justify left bottom)
-		)
-	)
 	(text "USB-C"
 		(exclude_from_sim no)
@@
 		)
 	)
-	(text "Extension Board Connector"
-		(exclude_from_sim no)
-		(at 236.728 163.576 0)
-		(effects
-			(font
-				(size 1.27 1.27)
-			)
-			(justify left bottom)
-		)
-	)
 	(text "Transmitting Data"
 		(exclude_from_sim no)
@@
 	(wire
 		(pts
+			(xy 173.99 149.86) (xy 179.07 149.86)
+		)
+		(stroke
+			(width 0)
+			(type default)
+		)
+	)
+	(wire
+		(pts
 			(xy 179.07 121.92) (xy 179.07 127)
 		)
@@
 	(wire
 		(pts
+			(xy 173.99 157.48) (xy 179.07 157.48)
+		)
+		(stroke
+			(width 0)
+			(type default)
+		)
+	)
+	(wire
+		(pts
 			(xy 269.24 40.64) (xy 269.24 35.56)
 		)
@@
 	)
 	(global_label "IO16"
-		(shape input)
+		(shape bidirectional)
 		(at 242.57 180.34 180)
 		(fields_autoplaced yes)
@@
 		)
 		(property "Intersheetrefs" "${INTERSHEET_REFS}"
-			(at 231.9648 180.34 0)
+			(at 234.1192 180.34 0)
 			(effects
 				(font
@@
 	)
 	(global_label "IO7"
-		(shape input)
+		(shape bidirectional)
 		(at 255.27 182.88 0)
 		(fields_autoplaced yes)
@@
 	)
 	(global_label "I2C_CLK"
-		(shape input)
+		(shape bidirectional)
 		(at 242.57 172.72 180)
 		(fields_autoplaced yes)
@@
 	)
 	(global_label "IO14"
-		(shape input)
+		(shape bidirectional)
 		(at 242.57 177.8 180)
 		(fields_autoplaced yes)
@@
 		)
 		(property "Intersheetrefs" "${INTERSHEET_REFS}"
-			(at 231.9648 177.8 0)
+			(at 234.1192 177.8 0)
 			(effects
 				(font
@@
 	)
 	(global_label "IO15"
-		(shape input)
+		(shape bidirectional)
 		(at 52.07 106.68 180)
 		(fields_autoplaced yes)
@@
 	)
 	(global_label "IO18"
-		(shape input)
+		(shape bidirectional)
 		(at 242.57 182.88 180)
 		(fields_autoplaced yes)
@@
 		)
 		(property "Intersheetrefs" "${INTERSHEET_REFS}"
-			(at 232.3277 182.88 0)
+			(at 234.1192 182.88 0)
 			(effects
 				(font
@@
 	)
 	(global_label "BUS_WIRE1"
-		(shape input)
+		(shape bidirectional)
 		(at 243.84 133.35 0)
 		(fields_autoplaced yes)
@@
 		)
 		(property "Intersheetrefs" "${INTERSHEET_REFS}"
-			(at 257.2875 133.35 0)
+			(at 258.3988 133.35 0)
 			(effects
 				(font
@@
 	)
 	(global_label "IO17"
-		(shape input)
+		(shape bidirectional)
 		(at 52.07 111.76 180)
 		(fields_autoplaced yes)
@@
 	)
 	(global_label "IO17"
-		(shape input)
+		(shape bidirectional)
 		(at 255.27 180.34 0)
 		(fields_autoplaced yes)
@@
 	)
 	(global_label "IO16"
-		(shape input)
+		(shape bidirectional)
 		(at 52.07 109.22 180)
 		(fields_autoplaced yes)
@@
 	)
 	(global_label "BUS_WIRE1"
-		(shape input)
+		(shape bidirectional)
 		(at 255.27 187.96 0)
 		(fields_autoplaced yes)
@@
 	)
 	(global_label "I2C_CLK"
-		(shape input)
+		(shape bidirectional)
 		(at 52.07 99.06 180)
 		(fields_autoplaced yes)
@@
 	)
 	(global_label "BUS_WIRE2"
-		(shape input)
+		(shape bidirectional)
 		(at 243.84 130.81 0)
 		(fields_autoplaced yes)
@@
 		)
 		(property "Intersheetrefs" "${INTERSHEET_REFS}"
-			(at 257.2875 130.81 0)
+			(at 258.3988 130.81 0)
 			(effects
 				(font
@@
 	)
 	(global_label "IO7"
-		(shape input)
+		(shape bidirectional)
 		(at 52.07 86.36 180)
 		(fields_autoplaced yes)
@@
 	)
 	(global_label "IO14"
-		(shape input)
+		(shape bidirectional)
 		(at 52.07 104.14 180)
 		(fields_autoplaced yes)
@@
 	)
 	(global_label "BUS_WIRE2"
-		(shape input)
+		(shape bidirectional)
 		(at 242.57 187.96 180)
 		(fields_autoplaced yes)
@@
 	)
 	(global_label "I2C_DAT"
-		(shape input)
+		(shape bidirectional)
 		(at 255.27 175.26 0)
 		(fields_autoplaced yes)
@@
 	)
 	(global_label "I2C_DAT"
-		(shape input)
+		(shape bidirectional)
 		(at 52.07 101.6 180)
 		(fields_autoplaced yes)
@@
 	)
 	(global_label "IO18"
-		(shape input)
+		(shape bidirectional)
 		(at 52.07 114.3 180)
 		(fields_autoplaced yes)
@@
 	)
 	(global_label "BUS_WIRE1"
-		(shape input)
+		(shape bidirectional)
 		(at 248.92 27.94 0)
 		(fields_autoplaced yes)
@@
 		)
 		(property "Intersheetrefs" "${INTERSHEET_REFS}"
-			(at 262.3675 27.94 0)
+			(at 263.4788 27.94 0)
 			(effects
 				(font
@@
 	)
 	(global_label "BUS_WIRE2"
-		(shape input)
+		(shape bidirectional)
 		(at 248.92 43.18 0)
 		(fields_autoplaced yes)
@@
 		)
 		(property "Intersheetrefs" "${INTERSHEET_REFS}"
-			(at 262.3675 43.18 0)
+			(at 263.4788 43.18 0)
 			(effects
 				(font
@@
 	)
 	(global_label "IO15"
-		(shape input)
+		(shape bidirectional)
 		(at 255.27 177.8 0)
 		(fields_autoplaced yes)
@@
 			)
 		)
-		(property "Value" "USB_C_Receptacle_USB2.0"
+		(property "Value" "USB-C Connector"
 			(at 242.316 66.294 0)
 			(effects
@@
 		(lib_name "GND_2")
 		(lib_id "power:GND")
-		(at 179.07 157.48 0)
+		(at 173.99 157.48 0)
 		(unit 1)
 		(exclude_from_sim no)
@@
 		(dnp no)
 		(property "Reference" "#PWR042"
-			(at 179.07 163.83 0)
+			(at 173.99 163.83 0)
 			(effects
 				(font
@@
 		)
 		(property "Value" "GND"
-			(at 179.07 161.544 0)
+			(at 173.99 161.544 0)
 			(effects
 				(font
@@
 		)
 		(property "Footprint" ""
-			(at 179.07 157.48 0)
+			(at 173.99 157.48 0)
 			(effects
 				(font
@@
 		)
 		(property "Datasheet" ""
-			(at 179.07 157.48 0)
+			(at 173.99 157.48 0)
 			(effects
 				(font
@@
 		)
 		(property "Description" "Power symbol creates a global label with name \"GND\" , ground"
-			(at 179.07 157.48 0)
+			(at 173.99 157.48 0)
 			(effects
 				(font
@@
 		(lib_name "+3.3V_1")
 		(lib_id "power:+3.3V")
-		(at 179.07 149.86 0)
+		(at 173.99 149.86 0)
 		(unit 1)
 		(exclude_from_sim no)
@@
 		(dnp no)
 		(property "Reference" "#PWR043"
-			(at 179.07 153.67 0)
+			(at 173.99 153.67 0)
 			(effects
 				(font
@@
 		)
 		(property "Value" "+3.3V"
-			(at 176.022 145.542 0)
+			(at 170.942 145.542 0)
 			(effects
 				(font
@@
 		)
 		(property "Footprint" ""
-			(at 179.07 149.86 0)
+			(at 173.99 149.86 0)
 			(effects
 				(font
@@
 		)
 		(property "Datasheet" ""
-			(at 179.07 149.86 0)
+			(at 173.99 149.86 0)
 			(effects
 				(font
@@
 		)
 		(property "Description" "Power symbol creates a global label with name \"+3.3V\""
-			(at 179.07 149.86 0)
+			(at 173.99 149.86 0)
 			(effects
 				(font
@@
 			)
 		)
+		(property "Sim.Pins" "1=K 2=A"
+			(at 146.05 154.94 0)
+			(effects
+				(font
+					(size 1.27 1.27)
+				)
+				(hide yes)
+			)
+		)
 		(pin "1"
 		)
@@
 			)
 		)
-		(property "Value" "Terminal"
-			(at 235.712 142.494 90)
+		(property "Value" "Screw Terminals"
+			(at 235.712 146.304 90)
 			(effects
 				(font
@@
 			)
 		)
-		(property "Value" "Conn_02x07_Odd_Even"
+		(property "Value" "Extension Board Connector"
 			(at 248.92 168.91 0)
 			(effects

Commit message: WIP
Parts:
- C4: LCSC C13585 -> C89632; MPN CL31A106KBHNNNE -> CL31B106KBHNNNE
- J4: LCSC C3975171 -> C22373875; MPN PM200-2-07-S-4.3 -> HC-PM200-4.3H-2x7PS
- L1: LCSC C96899 -> C6808101; MPN SWPA4030S3R9MT -> ANR4030T3R9M
- SW1: value Reset Button -> Button
- SW2: value Flash Button -> Button
Other:
- note added: "Flash"
- note added: "Reset"
Changed lines of the file:
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@@
 		)
 	)
+	(text "Flash"
+		(exclude_from_sim no)
+		(at 36.068 70.866 0)
+		(effects
+			(font
+				(size 0.8 0.8)
+			)
+			(justify right bottom)
+		)
+	)
 	(text "ESP32-S3"
 		(exclude_from_sim no)
@@
 		)
 	)
+	(text "Reset"
+		(exclude_from_sim no)
+		(at 34.544 46.736 0)
+		(effects
+			(font
+				(size 0.8 0.8)
+			)
+			(justify right bottom)
+		)
+	)
 	(text "RELAY"
 		(exclude_from_sim no)
@@
 			)
 		)
-		(property "Description" "100mW Thick Film Resistors ±100ppm/℃ ±1% 10kΩ 0603 Chip Resistor - Surface Mount ROHS"
+		(property "Description" "-55℃~+155℃ 100mW 10kΩ 75V Thick Film Resistor ±1% ±100ppm/℃ 0603 Chip Resistor - Surface Mount ROHS"
 			(at 46.99 29.21 0)
 			(effects
@@
 			)
 		)
-		(property "Description" "2.1A 3.9uH ±20% 3A SMD,4x4x3mm  Power Inductors ROHS"
+		(property "Description" "2.3A 3.3A 3.9uH Magnetic Shielded Inductor ±20% SMD,4x4mm Power Inductors ROHS"
 			(at 185.42 49.53 0)
 			(effects
@@
 			)
 		)
-		(property "LCSC" "C96899"
+		(property "LCSC" "C6808101"
 			(at 185.42 49.53 90)
 			(effects
@@
 			)
 		)
-		(property "MPN" "SWPA4030S3R9MT"
+		(property "MPN" "ANR4030T3R9M"
 			(at 185.42 49.53 0)
 			(effects
@@
 			)
 		)
-		(property "Value" "Reset Button"
+		(property "Value" "Button"
 			(at 33.02 40.386 0)
 			(effects
@@
 			)
 		)
-		(property "Description" "-40℃~+105℃ 1.5A 14P 2 2mm 2mm 2x7P 4.3mm Brass Square Hole Surface Mount,Vertical Top SMD,P=2mm Female Headers ROHS"
+		(property "Description" "-40℃~+105℃ 1.5A 14P 2 2mm 2mm 2x7P 4.3mm Brass Gold Square Hole Surface Mount,Vertical Top SMD,P=2mm Female Headers ROHS"
 			(at 247.65 180.34 0)
 			(effects
@@
 			)
 		)
-		(property "LCSC" "C3975171"
+		(property "LCSC" "C22373875"
 			(at 247.65 180.34 0)
 			(effects
@@
 			)
 		)
-		(property "MPN" "PM200-2-07-S-4.3"
+		(property "MPN" "HC-PM200-4.3H-2x7PS"
 			(at 247.65 180.34 0)
 			(effects
@@
 			)
 		)
-		(property "Description" "-40℃~+125℃ 2A 350mA 40V 5uA@30V 600mV@200mA Independent SOD-323 Schottky Diodes ROHS-40℃~+125℃ 2A 350mA 40V 5uA@30V 600mV@200mA Independent SOD-323 Schottky Diodes ROHS"
+		(property "Description" "-40℃~+125℃ 2A 350mA 40V 5uA@30V 600mV@200mA Independent SOD-323 Schottky Diodes ROHS"
 			(at 127 44.45 0)
 			(effects
@@
 			)
 		)
-		(property "Description" "50V 10uF X5R ±10% 1206 Multilayer Ceramic Capacitors MLCC - SMD/SMT ROHS"
+		(property "Description" "10uF ±10% 50V Ceramic Capacitor X7R 1206"
 			(at 139.7 55.88 0)
 			(effects
@@
 			)
 		)
-		(property "LCSC" "C13585"
+		(property "LCSC" "C89632"
 			(at 139.7 55.88 0)
 			(effects
@@
 			)
 		)
-		(property "MPN" "CL31A106KBHNNNE"
+		(property "MPN" "CL31B106KBHNNNE"
 			(at 139.7 55.88 0)
 			(effects
@@
 			)
 		)
-		(property "Value" "Flash Button"
+		(property "Value" "Button"
 			(at 34.29 64.516 0)
 			(effects

Commit message: WIP
Parts:
- D4: LCSC C965799 -> C2286; MPN XL-1608SURC-06 -> KT-0603R
- Q2: value BC817 -> BC817-40; LCSC C609806 -> C52801; MPN BC817-40 -> BC817-40,215
Changed lines of the file:
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@@
 			)
 		)
-		(property "Value" "BC817"
+		(property "Value" "BC817-40"
 			(at 151.892 105.41 0)
 			(effects
@@
 			)
 		)
-		(property "Description" "1 NPN 100MHz 100nA 250 300mW 45V 500mA 5V 700mV NPN SOT-23 Bipolar (BJT) ROHS"
+		(property "Description" "-65℃~+150℃ 1 NPN 100MHz 100nA 250 345mW 45V 500mA 5V 700mV NPN SOT-23 Bipolar (BJT) ROHS"
 			(at 144.78 104.14 0)
 			(effects
@@
 			)
 		)
-		(property "MPN" "BC817-40"
+		(property "MPN" "BC817-40,215"
 			(at 144.78 104.14 0)
 			(effects
@@
 			)
 		)
-		(property "LCSC" "C609806"
+		(property "LCSC" "C52801"
 			(at 144.78 104.14 0)
 			(effects
@@
 			)
 		)
-		(property "Description" "25mA 无色透明透镜 -30℃~+85℃ Positive post 617nm~621nm Red 120° 55mW 0603  Light Emitting Diodes (LED) ROHS"
+		(property "Description" "-40℃~+85℃ 120° 2.4V 20mA 300mcd 40mW 615nm~630nm 645nm Discrete Diode Red Water Clear 0603 LED Indication - Discrete ROHS"
 			(at 146.05 154.94 0)
 			(effects
@@
 			)
 		)
-		(property "LCSC" "C965799"
+		(property "LCSC" "C2286"
 			(at 146.05 154.94 0)
 			(effects
@@
 			)
 		)
-		(property "MPN" "XL-1608SURC-06"
+		(property "MPN" "KT-0603R"
 			(at 146.05 154.94 0)
 			(effects

Commit message: WIP
Changed lines of the file:
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@@
 	(title_block
 		(title "Doorman S3")
-		(date "2026-02-10")
+		(date "2026-02-11")
 		(rev "2.0")
 		(comment 1 "TC:Bus Intercom Gateway")
@@
 	)
 	(global_label "BUS_TX"
-		(shape input)
+		(shape output)
 		(at 123.19 104.14 180)
 		(fields_autoplaced yes)

Commit message: WIP
Parts:
- added Q3, Q4: BC817-40, Package_TO_SOT_SMD:SOT-23, symbol Transistor_BJT:BC817
- added Q5, Q6: BC807-40, Package_TO_SOT_SMD:SOT-23, symbol Transistor_BJT:BC807
- added R13: 200R, Resistor_SMD:R_0805_2012Metric, symbol Device:R
- added R14, R16, R17, R19, R4: 10K, Resistor_SMD:R_0603_1608Metric, symbol Device:R
- added R15: 10R, Resistor_SMD:R_0805_2012Metric, symbol Device:R
- added R18, R21: 1K, Resistor_SMD:R_0603_1608Metric, symbol Device:R
- added R20: 2K, Resistor_SMD:R_0603_1608Metric, symbol Device:R
Connections:
- net +3.3V: now also Q5.3 (C), Q6.3 (C)
- net BUS_RX: no longer U4.14 (IO10)
- net GND: now also Q3.2 (E), Q4.2 (E), R17.2, R18.2, R20.2, R21.2
- net SIEDLE_RX_CAR: now reaches U4.10 (IO6)
- net SIEDLE_RX_CAR: now also Q6.2 (E), R21.1
- net SIEDLE_TX_CAR: now reaches U4.15 (IO11)
- net SIEDLE_TX_CAR: now also R4.1
- net SIEDLE_RX_DAT: now reaches U4.25 (IO21)
- net SIEDLE_RX_DAT: now also Q5.2 (E), R18.1
- net +24V Bus renamed VBUS
- net VBUS: now also R13.1, R15.1, R16.1, R19.1
- new net: Q3.1 (B), R4.2
- new net: Q3.3 (C), R13.2
- new net: Q4.3 (C), R15.2
- new net: Q6.1 (B), R19.2, R20.1
- new net: Q5.1 (B), R16.2, R17.1
- new net: Q4.1 (B), R14.2
- new net SIEDLE_TX_DAT: R14.1, U4.14 (IO10)
- no-connect marks 22 -> 19
Other:
- note added: "SIEDLE IN-HOME:BUS COMMUNICATION"
- moved on the sheet: D4, D8, R7
