File: pcb/doorman.kicad_pcb (KiCad board)
At the start: 4 copper layers, 37.1 x 37.2 mm, 44 parts, among them J1 USB_C_Receptacle_USB2.0, J2 Terminal, J3 3V3 Test Pad, J4 TX Test Pad, J5 RX Test Pad, J6 BUS Test Pad, J7 BUS RX Test Pad, Q1 BC817, SW1 Reset Button, SW2 Flash Button, U1 ESP32-S3-WROOM-1, U2 AP63203WU, U3 GAQY252G3S

Commit message: WIP
Parts:
- removed 11, 8: 10K, Resistor_SMD:R_1206_3216Metric_Pad1.30x1.75mm_HandSolder
- removed J4: TX Test Pad, TestPoint:TestPoint_Pad_D1.0mm
- removed J5: RX Test Pad, TestPoint:TestPoint_Pad_D1.0mm
- removed JP2: SolderJumper_2_Open, Jumper:SolderJumper-2_P1.3mm_Open_RoundedPad1.0x1.5mm
- added C10: 0.1uF, Capacitor_SMD:C_0603_1608Metric, F.Cu at (137.7, 106.7)
- added C11: 10uF, Capacitor_SMD:C_0603_1608Metric, F.Cu at (137.8, 108.2)
- added C12: 33uF, Capacitor_SMD:C_1206_3216Metric, F.Cu at (151.0, 100.6)
- added C17: 10uF, Capacitor_SMD:C_0603_1608Metric, F.Cu at (139.6, 104.8)
- added C18: 100nF, Capacitor_SMD:C_0603_1608Metric, F.Cu at (144.7, 102.0)
- added C19: 10uF, Capacitor_SMD:C_0603_1608Metric, F.Cu at (146.1, 102.0)
- added C20: 100nF, Capacitor_SMD:C_0603_1608Metric, F.Cu at (146.1, 99.1)
- added C21: 10uF, Capacitor_SMD:C_0603_1608Metric, F.Cu at (144.6, 99.1)
- added C9: 1uF, Capacitor_SMD:C_0603_1608Metric, F.Cu at (147.6, 99.1)
- added D7: 6.2V, Diode_SMD:D_MELF, F.Cu at (155.3, 101.6)
- added J8: TX Test Pad, TestPoint:TestPoint_Pad_D1.0mm, B.Cu at (148.6, 87.6)
- added J9: RX Test Pad, TestPoint:TestPoint_Pad_D1.0mm, B.Cu at (148.6, 85.6)
- added Q2: BC817, Package_TO_SOT_SMD:SOT-23, F.Cu at (154.5, 96.3)
- added R11: 1.2, Resistor_SMD:R_0805_2012Metric, F.Cu at (153.5, 92.7)
- added R12: 10K, Resistor_SMD:R_0603_1608Metric, F.Cu at (135.2, 98.1)
- added R13: 10K, Resistor_SMD:R_0402_1005Metric, F.Cu at (139.8, 98.4)
- added R14: 10K, Resistor_SMD:R_0402_1005Metric, F.Cu at (137.2, 99.2)
- added R15: 33, Resistor_SMD:R_0402_1005Metric, F.Cu at (137.2, 100.2)
- added R16: 33, Resistor_SMD:R_0402_1005Metric, F.Cu at (137.2, 101.1)
- added R17: 33, Resistor_SMD:R_0402_1005Metric, F.Cu at (137.2, 103.0)
- added R18: 33, Resistor_SMD:R_0402_1005Metric, F.Cu at (137.2, 102.1)
- added R19: 33, Resistor_SMD:R_0402_1005Metric, F.Cu at (137.2, 103.9)
- added R20: 10K, Resistor_SMD:R_0603_1608Metric, F.Cu at (149.0, 99.1)
- added R21: 10K, Resistor_SMD:R_0603_1608Metric, F.Cu at (147.6, 102.1)
- added R8: 1.2, Resistor_SMD:R_0805_2012Metric, F.Cu at (155.4, 92.7)
- added U4: ESP32-S3-MINI-1, RF_Module:ESP32-S2-MINI-1, F.Cu at (143.9, 87.0)
- C8: value 33uF -> 1uF; footprint Capacitor_SMD:C_1206_3216Metric_Pad1.33x1.80mm_HandSolder -> Capacitor_SMD:C_0603_1608Metric; moved to F.Cu
- Q1: value BC817 -> BC847BPN; footprint Package_TO_SOT_SMD:SOT-23 -> Package_TO_SOT_SMD:SOT-363_SC-70-6
- R2: value 1K -> 2.2K
- R4: value 5.1K -> 10
- R5: value 1M -> 47K
- R6: value 147K -> 10K
- U1: value ESP32-S3-WROOM-1 -> ES8388; footprint RF_Module:ESP32-S3-WROOM-1 -> Package_DFN_QFN:QFN-28-1EP_4x4mm_P0.45mm_EP2.6x2.6mm
- moved Q1 23.8 mm to (154.8, 89.0), turned to 180 degrees
- moved R2 22.3 mm to (156.7, 96.4)
- moved J7 17.8 mm to (136.3, 93.9)
- moved U1 12.6 mm to (141.2, 101.5)
- moved C8 5.80 mm to (142.5, 104.8), turned to 0 degrees
- moved R3 5.77 mm to (139.9, 108.6), turned to 90 degrees
- moved R6 4.53 mm to (153.0, 100.2)
- moved R5 3.97 mm to (153.0, 103.3), turned to -90 degrees
- moved R9 3.72 mm to (153.9, 85.4), turned to 180 degrees
- moved R4 3.24 mm to (144.9, 104.8), turned to 0 degrees
- moved D2 0.84 mm to (154.2, 109.2)
- moved G*** 0.60 mm to (145.1, 101.6)
- moved C2 0.20 mm to (135.0, 84.6)
- moved D1 0.17 mm to (138.4, 111.4)
- moved J6 0.15 mm to (153.5, 104.7)
Connections:
- C8 pad 1: Net-(JP2-B) -> Net-(U1-LOUT1)
- C8 pad 2: ADC_IN -> Net-(C8-Pad2)
- J1 pad B5: Net-(J1-CC2) -> Net-(J1-CC1)
- J7 pad 1: BUS_ANA -> BUS_RX
- Q1 pad 1: Net-(Q1-B) -> GND
- Q1 pad 2: GND -> Net-(Q1A-B1)
- Q1 pad 3: +24V Bus -> +3.3V
- R2 pad 1: Net-(Q1-B) -> BUS_TX
- R2 pad 2: BUS_TX -> Net-(Q1A-C1)
- R4 pad 1: GND -> Net-(C8-Pad2)
- R4 pad 2: Net-(J1-CC2) -> AUDIO_OUT
- R5 pad 1: +24V Bus -> Net-(Q1B-B2)
- R5 pad 2: BUS_ANA -> +24V Bus
- R6 pad 1: BUS_ANA -> Net-(Q1B-B2)
- U1 pad 1: GND -> Net-(U1-MCLK)
- U1 pad 10: unconnected-(U1-IO17-Pad10) -> Net-(U1-VREF)
- U1 pad 12: BUS_TX -> Net-(U1-LOUT1)
- U1 pad 13: USB_D- -> GND
- U1 pad 14: USB_D+ -> unconnected-(U1-ROUT2-Pad14)
- U1 pad 16: unconnected-(U1-IO46-Pad16) -> +3.3V
- U1 pad 17: BUS_ANA -> +3.3V
- U1 pad 18: BUS_ANA -> GND
- U1 pad 19: unconnected-(U1-IO11-Pad19) -> Net-(U1-ADCVREF)
- U1 pad 20: unconnected-(U1-IO12-Pad20) -> Net-(U1-VMID)
- U1 pad 24: unconnected-(U1-IO47-Pad24) -> Net-(U1-LIN1)
- U1 pad 26: unconnected-(U1-IO45-Pad26) -> I2C_AD
- U1 pad 27: /FLASH -> I2C_DAT
- U1 pad 28: unconnected-(U1-IO35-Pad28) -> I2C_CLK
- U1 pad 29: unconnected-(U1-IO36-Pad29) -> GND
- U1 pad 3: /EN -> +3.3V
- U1 pad 4: unconnected-(U1-IO4-Pad4) -> GND
- U1 pad 5: unconnected-(U1-IO5-Pad5) -> Net-(U1-SCLK)
- U1 pad 6: unconnected-(U1-IO6-Pad6) -> Net-(U1-DSDIN)
- U1 pad 7: ADC_IN -> Net-(U1-LRCK)
- U1 pad 8: unconnected-(U1-IO15-Pad8) -> Net-(U1-ASDOUT)
Routing:
- net +3.3V: track 68.3 -> 138.5 mm, vias 5 -> 13
- net BUS_RX: track 0.00 -> 26.1 mm, vias 0 -> 3
- net /FLASH: track 34.6 -> 9.33 mm
- net BUS_ANA: track 19.4 -> 0.00 mm, vias 2 -> 0
- net Net-(Q1B-B2): track 0.00 -> 15.7 mm, vias 0 -> 2
- net LED_RED: track 9.43 -> 24.3 mm
- net LED_RGB: track 12.2 -> 26.9 mm
- net ADC_IN: track 14.6 -> 0.00 mm, vias 1 -> 0
- net Net-(Q1A-C1): track 0.00 -> 14.5 mm, vias 0 -> 2
- net BUS_TX: track 8.82 -> 23.1 mm, vias 0 -> 2
- net Net-(JP2-B): track 13.7 -> 0.00 mm
- net /EN: track 14.0 -> 26.5 mm
- net I2S_DAT_OUT: track 0.00 -> 12.0 mm, vias 0 -> 2
- net Net-(Q1A-B1): track 0.00 -> 11.3 mm
- net I2S_SCLK: track 0.00 -> 10.3 mm, vias 0 -> 2
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Other:
- outline, holes or cut-outs redrawn
- board text added: "TC:RX"
- board text removed: "ESP32-S3 WROOM-1"
- board text removed: "SERIAL"
- board text removed: "VD"

Commit message: WIP
Parts:
- removed C10: 0.1uF, Capacitor_SMD:C_0603_1608Metric
- removed C11, C17, C19, C21: 10uF, Capacitor_SMD:C_0603_1608Metric
- removed C12: 33uF, Capacitor_SMD:C_1206_3216Metric
- removed C18, C20: 100nF, Capacitor_SMD:C_0603_1608Metric
- removed C8, C9: 1uF, Capacitor_SMD:C_0603_1608Metric
- removed R13, R14: 10K, Resistor_SMD:R_0402_1005Metric
- removed R15, R16, R17, R18, R19: 33, Resistor_SMD:R_0402_1005Metric
- removed R20, R21: 10K, Resistor_SMD:R_0603_1608Metric
- removed R4: 10, Resistor_SMD:R_0402_1005Metric
- removed U1: ES8388, Package_DFN_QFN:QFN-28-1EP_4x4mm_P0.45mm_EP2.6x2.6mm
- added J4: Conn_02x07_Odd_Even, Connector_PinSocket_2.00mm:PinSocket_2x07_P2.00mm_Vertical_SMD, F.Cu at (143.9, 101.5)
- moved J6 3.64 mm to (154.8, 101.2)
- moved G*** 0.58 mm to (145.5, 101.2)
Connections:
- net Net-(D1-K) renamed /VCC_IN
- U4 pad 11: unconnected-(U4-IO7-Pad11) -> IO7
- U4 pad 15: I2S_SCLK -> unconnected-(U4-IO11-Pad15)
- U4 pad 16: I2S_MCLK -> I2C_CLK
- U4 pad 17: I2S_DAT_IN -> I2C_DAT
- U4 pad 18: I2S_LRCK -> IO14
- U4 pad 19: I2S_DAT_OUT -> IO15
- U4 pad 20: I2C_CLK -> IO16
- U4 pad 21: I2C_DAT -> IO17
- U4 pad 22: I2C_AD -> IO18
Routing:
- net +3.3V: track 138.5 -> 82.2 mm, vias 13 -> 7
- net /VCC_IN: track 54.5 -> 71.0 mm, vias 2 -> 4
- net IO7: track 0.00 -> 14.8 mm, vias 0 -> 2
- net I2S_DAT_OUT: track 12.0 -> 0.00 mm, vias 2 -> 0
- net I2S_SCLK: track 10.3 -> 0.00 mm, vias 2 -> 0
- net I2S_LRCK: track 10.1 -> 0.00 mm, vias 2 -> 0
- net IO18: track 0.00 -> 9.85 mm, vias 0 -> 2
- net BUS_WIRE2: track 10.3 -> 19.0 mm, vias 1 -> 2
- net I2S_DAT_IN: track 8.48 -> 0.00 mm, vias 2 -> 0
- net IO16: track 0.00 -> 8.30 mm
- net IO14: track 0.00 -> 7.89 mm
- net Net-(U1-LIN1): track 7.11 -> 0.00 mm
- net I2S_MCLK: track 7.04 -> 0.00 mm, vias 2 -> 0
- net +24V Bus: track 38.2 -> 31.2 mm
- net GND: track 11.5 -> 5.83 mm, vias 85 -> 96
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- added copper zone on F.Cu, net VCC
- removed copper zone on F.Cu, net /VCC_IN

Commit message: WIP
Connections:
- J7 pad 1: BUS_RX -> BUS_CONN
- Q1 pad 4: BUS_RX -> BUS_CONN
- R12 pad 1: BUS_RX -> BUS_CONN
- U4 pad 13: BUS_RX -> BUS_CONN
- U4 pad 14: unconnected-(U4-IO10-Pad14) -> BUS_CONN
Routing:
- net BUS_CONN: track 0.00 -> 27.0 mm, vias 0 -> 3
- net BUS_RX: track 26.1 -> 0.00 mm, vias 3 -> 0

Commit message: WIP
Connections:
- J4 pad 1: GND -> I2C_CLK
- J4 pad 3: I2C_CLK -> GND
Routing:
- net +3.3V: track 82.2 -> 78.0 mm
- net unconnected-(U4-IO11-Pad15): track 1.38 -> 0.19 mm, vias 1 -> 0
- net BUS_CONN: track 27.0 -> 27.6 mm
- net GND: vias 96 -> 97
- added copper zone on F.Cu, net /VCC_IN
- removed copper zone on F.Cu, net VCC

Commit message: WIP
Parts:
- removed D3: WS2812B, Doorman:LED-SMD_4P-L2.0-W1.8_CY-0807
- added D8: XL-2020RGBC-SK6812B, Doorman:LED-SMD_6P-L2.0-W2.0_XL-2020RGBC, F.Cu at (160.9, 79.7)
- moved R12 22.3 mm to (154.5, 86.9), turned to 0 degrees
- moved Q1 0.26 mm to (154.5, 89.1)
- moved R9 0.17 mm to (154.1, 85.4)
Routing:
- net BUS_CONN: track 27.6 -> 23.7 mm
- net USB_D-: track 16.3 -> 15.0 mm
- net LED_RGB: track 26.9 -> 27.7 mm
- net +24V Bus: track 31.2 -> 30.6 mm
- net /VCC_IN: track 71.0 -> 71.5 mm
- net GND: track 5.83 -> 6.26 mm, vias 97 -> 101

Commit message: WIP
Other:
- board size 37.1 x 37.2 mm -> 37 x 37.2 mm
Changed lines of the file:
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@@
 		(layer "Dwgs.User")
 	)
-	(gr_line
-		(start 126.83033 108.68)
-		(end 126.83033 111.88)
+	(gr_arc
+		(start 161.9 76.68)
+		(mid 163.307144 77.262858)
+		(end 163.890002 78.670002)
 		(stroke
-			(width 0.1)
+			(width 0.05)
 			(type default)
 		)
@@
 	)
 	(gr_line
-		(start 163.9 109)
-		(end 163.9 111.88)
+		(start 136.02 76.68)
+		(end 136.02 81.79)
 		(stroke
-			(width 0.1)
-			(type default)
-		)
-		(layer "Edge.Cuts")
-	)
-	(gr_arc
-		(start 163.9 111.88)
-		(mid 163.314215 113.294224)
-		(end 161.9 113.88)
-		(stroke
-			(width 0.1)
-			(type default)
-		)
-		(layer "Edge.Cuts")
-	)
-	(gr_line
-		(start 126.83033 108.68)
-		(end 126.83033 78.68)
-		(stroke
-			(width 0.1)
+			(width 0.05)
 			(type default)
 		)
@@
 		(end 151.83 81.79)
 		(stroke
-			(width 0.1)
+			(width 0.05)
 			(type default)
 		)
@@
 		(end 136.02 81.79)
 		(stroke
-			(width 0.1)
+			(width 0.05)
+			(type default)
+		)
+		(layer "Edge.Cuts")
+	)
+	(gr_line
+		(start 161.9 113.870002)
+		(end 128.83033 113.870002)
+		(stroke
+			(width 0.05)
+			(type default)
+		)
+		(layer "Edge.Cuts")
+	)
+	(gr_line
+		(start 163.890002 78.670002)
+		(end 163.890002 111.88)
+		(stroke
+			(width 0.05)
 			(type default)
 		)
@@
 	)
 	(gr_arc
-		(start 126.83033 78.68)
-		(mid 127.416116 77.265786)
+		(start 126.840328 78.670002)
+		(mid 127.423186 77.262858)
 		(end 128.83033 76.68)
 		(stroke
-			(width 0.1)
+			(width 0.05)
 			(type default)
 		)
@@
 	)
 	(gr_line
-		(start 161.9 113.88)
-		(end 128.83033 113.88)
+		(start 126.840328 78.670002)
+		(end 126.840328 111.88)
 		(stroke
-			(width 0.1)
-			(type default)
-		)
-		(layer "Edge.Cuts")
-	)
-	(gr_line
-		(start 163.899999 78.7)
-		(end 163.9 109)
-		(stroke
-			(width 0.1)
+			(width 0.05)
 			(type default)
 		)
@@
 	)
 	(gr_arc
-		(start 128.83033 113.88)
-		(mid 127.416116 113.294214)
-		(end 126.83033 111.88)
+		(start 128.83033 113.870002)
+		(mid 127.423186 113.287144)
+		(end 126.840328 111.88)
 		(stroke
-			(width 0.1)
-			(type default)
-		)
-		(layer "Edge.Cuts")
-	)
-	(gr_arc
-		(start 161.9 76.679871)
-		(mid 163.321339 77.272795)
-		(end 163.899999 78.7)
-		(stroke
-			(width 0.1)
+			(width 0.05)
 			(type default)
 		)
@@
 		(end 136.02 76.68)
 		(stroke
-			(width 0.1)
-			(type default)
-		)
-		(layer "Edge.Cuts")
-	)
-	(gr_line
-		(start 136.02 81.79)
-		(end 136.02 76.68)
-		(stroke
-			(width 0.1)
+			(width 0.05)
 			(type default)
 		)
@@
 		(end 161.9 76.68)
 		(stroke
-			(width 0.1)
+			(width 0.05)
 			(type default)
 		)
+		(layer "Edge.Cuts")
+	)
+	(gr_arc
+		(start 163.890002 111.88)
+		(mid 163.307144 113.287144)
+		(end 161.9 113.870002)
+		(stroke
+			(width 0.05)
+			(type default)
+		)

Commit message: WIP
Parts:
- R12: value 10K -> 39K
- R5: value 47K -> 39K
Connections:
- net BUS_CONN renamed BUS_RX
Routing:
- net IO18: track 9.85 -> 10.7 mm

Commit message: WIP
Routing:
- net GND: vias 101 -> 103
Changed lines of the file:
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@@
 	(title_block
 		(title "Doorman S3")
-		(date "2026-01-26")
-		(rev "1.7")
+		(date "2026-02-04")
+		(rev "2.0")
 		(comment 1 "TC:Bus Intercom Gateway")
 	)
@@
 		)
 		(fp_line
-			(start 5 -7.5)
-			(end 5 7.5)
+			(start 4.13 -7.5)
+			(end 4.13 7.5)
 			(stroke
 				(width 0.05)
@@
 		)
 		(fp_line
-			(start -5 -7.5)
-			(end 5 -7.5)
+			(start -4.07 -7.5)
+			(end 4.13 -7.5)
 			(stroke
 				(width 0.05)
@@
 		)
 		(fp_line
-			(start 5 7.5)
-			(end -5 7.5)
+			(start 4.13 7.5)
+			(end -4.07 7.5)
 			(stroke
 				(width 0.05)
@@
 		)
 		(fp_line
-			(start -5 7.5)
-			(end -5 -7.5)
+			(start -4.07 7.5)
+			(end -4.07 -7.5)
 			(stroke
 				(width 0.05)
@@
 	)
 	(via
+		(at 145.934015 105.459)
+		(size 0.6)
+		(drill 0.3)
+		(layers "F.Cu" "B.Cu")
+		(free yes)
+		(net 2)
+	)
+	(via
 		(at 150.17 85.97)
 		(size 0.6)
@@
 	)
 	(via
+		(at 154.46 94.5)
+		(size 0.6)
+		(drill 0.3)
+		(layers "F.Cu" "B.Cu")
+		(free yes)
+		(net 2)
+	)
+	(via
 		(at 130.1 99.73)
 		(size 0.6)
@@
 	)
 	(segment
-		(start 154.84 95.28)
-		(end 154.84 95.459998)
-		(width 0.2)
-		(layer "F.Cu")
-		(net 33)
-	)
-	(segment
 		(start 156.68 95.61)
-		(end 156.38 95.31)
-		(width 0.2)
-		(layer "F.Cu")
-		(net 33)
-	)
-	(segment
-		(start 155.464999 95.31)
-		(end 155.45 95.324999)
-		(width 0.2)
-		(layer "F.Cu")
-		(net 33)
-	)
-	(segment
-		(start 155.405001 95.28)
-		(end 155.45 95.324999)
+		(end 156.394999 95.324999)
 		(width 0.2)
 		(layer "F.Cu")
@@
 	)
 	(segment
-		(start 154.84 95.28)
-		(end 155.405001 95.28)
+		(start 154.97 95.324999)
+		(end 155.45 95.324999)
 		(width 0.2)
 		(layer "F.Cu")
@@
 	)
 	(segment
-		(start 156.38 95.31)
-		(end 155.464999 95.31)
+		(start 156.394999 95.324999)
+		(end 155.45 95.324999)
 		(width 0.2)
 		(layer "F.Cu")
@@
 	)
 	(via
-		(at 154.84 95.28)
+		(at 154.97 95.324999)
 		(size 0.6)
 		(drill 0.3)
@@
 	)
 	(segment
-		(start 150.13 93.15)
-		(end 152.26 95.28)
+		(start 152.304999 95.324999)
+		(end 150.13 93.15)
 		(width 0.2)
 		(layer "B.Cu")
@@
 	)
 	(segment
-		(start 150.13 90.87)
-		(end 150.13 93.15)
+		(start 151.22 89.78)
+		(end 152.92 89.78)
 		(width 0.2)
 		(layer "B.Cu")
@@
 	)
 	(segment
-		(start 151.22 89.78)
-		(end 150.13 90.87)
+		(start 154.97 95.324999)
+		(end 152.304999 95.324999)
 		(width 0.2)
 		(layer "B.Cu")
@@
 	)
 	(segment
-		(start 152.92 89.78)
+		(start 150.13 90.87)
 		(end 151.22 89.78)
 		(width 0.2)
@@
 	)
 	(segment
-		(start 152.26 95.28)
-		(end 154.84 95.28)
+		(start 150.13 93.15)
+		(end 150.13 90.87)
 		(width 0.2)
 		(layer "B.Cu")
@@
 	)
 	(segment
-		(start 153.01 100.116344)
-		(end 153.868891 100.975235)
+		(start 154.52 92.93)
+		(end 153.01 94.44)
 		(width 0.4)
 		(layer "In1.Cu")
@@
 	)
 	(segment
-		(start 154.52 89.98)
-		(end 154.52 93.13)
+		(start 153.01 100.116344)
+		(end 153.868891 100.975235)
 		(width 0.4)
 		(layer "In1.Cu")
@@
 	)
 	(segment
-		(start 154.52 93.13)
-		(end 153.01 94.64)
+		(start 153.01 94.44)
+		(end 153.01 100.116344)
 		(width 0.4)
 		(layer "In1.Cu")
@@
 	)
 	(segment
-		(start 153.01 94.64)
-		(end 153.01 100.116344)
+		(start 154.52 89.98)
+		(end 154.52 92.93)
 		(width 0.4)
 		(layer "In1.Cu")
