File: pcb/doorman.kicad_pcb (KiCad board)
At the start: 4 copper layers, 37 x 37.2 mm, 60 parts, among them J1 USB-C Connector, J2 Screw Terminals, J3 3V3 Test Pad, J4 Extension Board Connector, J6 BUS Test Pad, J7 BUS RX Test Pad, J8 TX Test Pad, J9 RX Test Pad, Q1 BC847BPN, Q2 BC817-40, Q3 BC817-40, Q4 BC817-40, Q5 BC807-40, Q6 BC807-40, SW1 Button, SW2 Button, U2 AP63203WU, U3 GAQY252G3S, U4 ESP32-S3-MINI-1

Commit message: WIP
Parts:
- removed the G*** at (131.4, 107.9)
- moved R14 14.5 mm to (128.2, 106.0), turned to -90 degrees
- moved Q4 13.1 mm to (130.9, 109.4), turned to 0 degrees
- moved R21 10.8 mm to (133.4, 103.9), turned to -90 degrees
- moved R20 8.68 mm to (134.8, 103.9), turned to -90 degrees
- moved Q5 8.16 mm to (139.8, 100.4), turned to 90 degrees
- moved R15 8.09 mm to (134.7, 109.4), turned to 180 degrees
- moved R18 7.93 mm to (138.3, 103.8)
- moved R4 7.91 mm to (129.9, 100.8), turned to -90 degrees
- moved R19 7.66 mm to (136.3, 103.9)
- moved Q3 6.23 mm to (130.9, 104.4)
- moved Q6 6.13 mm to (134.8, 100.4), turned to 90 degrees
- moved R13 5.09 mm to (134.7, 107.0), turned to 180 degrees
- moved R17 2.17 mm to (139.8, 103.8), turned to -90 degrees
- moved R16 1.59 mm to (141.3, 103.8), turned to 90 degrees
- moved R3 0.91 mm to (140.0, 108.9)
Connections:
- U4 pad 10: SIEDLE_RX_CAR -> SIEDLE_TX_CAR
- U4 pad 14: SIEDLE_TX_DAT -> SIEDLE_RX_CAR
- U4 pad 15: SIEDLE_TX_CAR -> SIEDLE_RX_DAT
- U4 pad 25: SIEDLE_RX_DAT -> unconnected-(U4-IO21-Pad25)
- U4 pad 9: unconnected-(U4-IO5-Pad9) -> SIEDLE_TX_DAT
Routing:
- net SIEDLE_RX_DAT: track 34.3 -> 12.2 mm, vias 3 -> 1
- net SIEDLE_TX_DAT: track 6.33 -> 24.6 mm
- net +3.3V: track 102.8 -> 87.1 mm
- net SIEDLE_TX_CAR: track 1.91 -> 13.5 mm
- net VBUS: track 43.5 -> 54.5 mm, vias 1 -> 2
- net /VCC_IN: track 72.3 -> 66.8 mm
- net Net-(Q4-B): track 1.55 -> 4.96 mm
- net BUS_WIRE1: track 24.9 -> 28.0 mm
- net Net-(Q3-C): track 2.19 -> 4.24 mm
- net SIEDLE_RX_CAR: track 9.56 -> 11.2 mm
- net Net-(Q3-B): track 3.48 -> 1.85 mm
- net Net-(Q1B-B2): track 15.1 -> 16.0 mm
- net Net-(J1-CC1): track 12.0 -> 11.3 mm
- net GND: vias 122 -> 123
Other:
- board text removed: "CHECK"
- board text removed: "THE DOCS"

Commit message: WIP
Parts:
- added R22: 5K1, Resistor_SMD:R_0402_1005Metric, F.Cu at (140.1, 108.9)
- moved R3 1.32 mm to (138.7, 108.9)
- moved J7 0.31 mm to (140.0, 87.5)
- moved Q6 0.16 mm to (134.7, 100.5)
- moved Q5 0.14 mm to (139.6, 100.4)
Connections:
- J1 pad B5: Net-(J1-CC1) -> Net-(J1-CC2)
- R3 pad 1: Net-(J1-CC1) -> Net-(J1-CC2)
Routing:
- net Net-(J1-CC2): track 0.00 -> 11.8 mm
- net Net-(J1-CC1): track 11.3 -> 6.77 mm
- net +3.3V: track 87.1 -> 88.3 mm, vias 8 -> 7
- net VBUS: track 54.5 -> 53.4 mm
- net SIEDLE_RX_CAR: track 11.2 -> 10.3 mm

Commit message: WIP
Routing:
- net SIEDLE_TX_DAT: track 24.6 -> 25.3 mm
- net SIEDLE_RX_DAT: track 12.0 -> 11.3 mm
- net GND: vias 123 -> 125
Changed lines of the file:
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@@
 			)
 		)
-		(property "Description" "-40℃~+85℃ -98.2dBm 2.4GHz 20.5dBm 355mA 3V~3.6V 95mA Bluetooth5.0 ESP32-S3 On-board PCB Antenna UART、SPI、I2C、GPIO、I2S、USB SMD WiFi Modules ROHS"
+		(property "Description" "-103.5dBm -40℃~+85℃ 2.4GHz 20.5dBm 355mA 3V~3.6V 95mA Bluetooth5.0 ESP32-S3 On-board PCB Antenna UART、SPI、I2C、GPIO、I2S、USB SMD WiFi Modules ROHS"
 			(at 0 0 0)
 			(unlocked yes)
@@
 	)
 	(via
-		(at 136.88 98.17)
+		(at 136.92 97.9)
 		(size 0.6)
 		(drill 0.3)
@@
 	)
 	(via
-		(at 133.35 105.38)
+		(at 133.46 105.4)
 		(size 0.6)
 		(drill 0.3)
@@
 	)
 	(via
+		(at 146.5 95.06)
+		(size 0.6)
+		(drill 0.3)
+		(layers "F.Cu" "B.Cu")
+		(free yes)
+		(net 2)
+	)
+	(via
 		(at 163.290002 94.48)
 		(size 0.6)
@@
 	)
 	(via
-		(at 138.69 88.79)
+		(at 138.49 88.6)
 		(size 0.6)
 		(drill 0.3)
@@
 	)
 	(via
+		(at 134.82 104.04)
+		(size 0.6)
+		(drill 0.3)
+		(layers "F.Cu" "B.Cu")
+		(free yes)
+		(net 2)
+	)
+	(via
 		(at 162.675288 113.033702)
 		(size 0.6)
@@
 	)
 	(via
+		(at 134.809976 100.742499)
+		(size 0.6)
+		(drill 0.3)
+		(layers "F.Cu" "B.Cu")
+		(free yes)
+		(net 2)
+	)
+	(via
 		(at 129.59 106)
 		(size 0.6)
@@
 	)
 	(via
-		(at 135.35 95.53)
+		(at 135.38 95.38)
 		(size 0.8)
 		(drill 0.4)
@@
 	)
 	(via
-		(at 137.51 101.45)
-		(size 0.6)
-		(drill 0.3)
-		(layers "F.Cu" "B.Cu")
-		(free yes)
-		(net 2)
-	)
-	(via
 		(at 129.87 107.88)
 		(size 0.6)
@@
 	)
 	(via
-		(at 136.55 100.69)
+		(at 136.83 100.52)
 		(size 0.6)
 		(drill 0.3)
@@
 	)
 	(segment
-		(start 137.71 95.54)
-		(end 137.705 95.535)
+		(start 135.51 100.485801)
+		(end 135.51 96.45)
 		(width 0.2)
 		(layer "F.Cu")
@@
 	)
 	(segment
-		(start 137.705 95.535)
+		(start 135.51 96.45)
+		(end 136.425 95.535)
+		(width 0.2)
+		(layer "F.Cu")
+		(net 68)
+	)
+	(segment
+		(start 137.39 101.51)
+		(end 136.534199 101.51)
+		(width 0.2)
+		(layer "F.Cu")
+		(net 68)
+	)
+	(segment
+		(start 136.534199 101.51)
+		(end 135.51 100.485801)
+		(width 0.2)
+		(layer "F.Cu")
+		(net 68)
+	)
+	(segment
+		(start 136.425 95.535)
 		(end 136.93 95.535)
 		(width 0.2)
@@
 	)
 	(via
-		(at 137.71 95.54)
+		(at 137.39 101.51)
 		(size 0.6)
 		(drill 0.3)
@@
 	)
 	(segment
-		(start 141.15 97.07)
-		(end 139.62 95.54)
-		(width 0.2)
-		(layer "B.Cu")
-		(net 68)
-	)
-	(segment
-		(start 139.62 95.54)
-		(end 137.71 95.54)
+		(start 137.39 101.51)
+		(end 137.39 102.05)
 		(width 0.2)
 		(layer "B.Cu")
@@
 	)
 	(segment
-		(start 141.15 99.32)
-		(end 141.15 97.07)
+		(start 137.39 102.05)
+		(end 138.35 103.01)
 		(width 0.2)
 		(layer "B.Cu")
@@
 	)
 	(segment
-		(start 138.6 101.87)
-		(end 141.15 99.32)
-		(width 0.2)
-		(layer "B.Cu")
-		(net 68)
-	)
-	(segment
-		(start 138.07 90.06)
-		(end 137.695 90.435)
+		(start 138.565187 89.57008)
+		(end 137.700267 90.435)
 		(width 0.2)
 		(layer "F.Cu")
@@
 	)
 	(segment
-		(start 138.07 89.55)
-		(end 138.07 90.06)
-		(width 0.2)
-		(layer "F.Cu")
-		(net 69)
-	)
-	(segment
-		(start 137.695 90.435)
+		(start 137.700267 90.435)
 		(end 136.93 90.435)
 		(width 0.2)
@@
 	)
 	(via
-		(at 138.07 89.55)
+		(at 138.565187 89.57008)
 		(size 0.6)
 		(drill 0.3)
@@
 	)
 	(segment
+		(start 138.545107 89.55)
+		(end 132.89 89.55)
+		(width 0.2)
+		(layer "B.Cu")
+		(net 69)
+	)
+	(segment
 		(start 128.28 94.16)
 		(end 128.28 105.165)
@@
 	)
 	(segment
-		(start 132.89 89.55)
-		(end 128.28 94.16)
+		(start 138.565187 89.57008)
+		(end 138.545107 89.55)
 		(width 0.2)
 		(layer "B.Cu")
@@
 	)
 	(segment
-		(start 138.07 89.55)
-		(end 132.89 89.55)
+		(start 132.89 89.55)
+		(end 128.28 94.16)
 		(width 0.2)
 		(layer "B.Cu")
@@
 			(thermal_gap 0.5)
 			(thermal_bridge_width 0.5)
-			(island_removal_mode 1)
-			(island_area_min 10)
 		)
 		(polygon

Commit message: WIP
Routing:
- net VBUS: track 53.4 -> 40.2 mm, vias 2 -> 3
- net SIEDLE_RX_DAT: track 11.3 -> 10.6 mm
- net GND: vias 125 -> 120
- added copper zone on B.Cu, net VBUS
Changed lines of the file:
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@@
 			(at 0 -1.17 90)
 			(layer "F.SilkS")
+			(hide yes)
 			(effects
 				(font
@@
 			(net 70 "VBUS")
 			(pintype "passive")
+			(zone_connect 2)
 		)
 		(pad "2" smd roundrect
@@
 			(net 70 "VBUS")
 			(pintype "passive")
+			(zone_connect 2)
 		)
 		(pad "2" smd roundrect
@@
 			(net 70 "VBUS")
 			(pintype "passive")
+			(zone_connect 2)
 		)
 		(pad "2" smd roundrect
@@
 			(net 70 "VBUS")
 			(pintype "passive")
+			(zone_connect 2)
 		)
 		(pad "2" smd roundrect
@@
 	)
 	(via
-		(at 136.77 108.17)
-		(size 0.6)
-		(drill 0.3)
-		(layers "F.Cu" "B.Cu")
-		(free yes)
-		(net 2)
-	)
-	(via
 		(at 154.12 106.15)
 		(size 0.9)
@@
 	)
 	(via
-		(at 133.46 105.4)
-		(size 0.6)
-		(drill 0.3)
-		(layers "F.Cu" "B.Cu")
-		(free yes)
-		(net 2)
-	)
-	(via
 		(at 159.25 107.625)
 		(size 0.6)
@@
 	)
 	(via
-		(at 134.49 105.38)
+		(at 134.1 104.68)
 		(size 0.6)
 		(drill 0.3)
@@
 	)
 	(via
-		(at 138.34 105.36)
+		(at 139.08 104.66)
 		(size 0.6)
 		(drill 0.3)
@@
 	)
 	(via
-		(at 135.17 105.38)
-		(size 0.6)
-		(drill 0.3)
-		(layers "F.Cu" "B.Cu")
-		(free yes)
-		(net 2)
-	)
-	(via
 		(at 128.94 108.51)
 		(size 0.6)
@@
 	)
 	(via
-		(at 139.42 105.34)
-		(size 0.6)
-		(drill 0.3)
-		(layers "F.Cu" "B.Cu")
-		(free yes)
-		(net 2)
-	)
-	(via
 		(at 140.91 84.3)
 		(size 0.6)
@@
 	)
 	(via
-		(at 140.17 105.35)
-		(size 0.6)
-		(drill 0.3)
-		(layers "F.Cu" "B.Cu")
-		(free yes)
-		(net 2)
-	)
-	(via
-		(at 136.83 100.52)
+		(at 136.41 100.36)
 		(size 0.6)
 		(drill 0.3)
@@
 	)
 	(segment
-		(start 135.51 100.485801)
-		(end 135.51 96.45)
+		(start 135.51 96.45)
+		(end 136.425 95.535)
 		(width 0.2)
 		(layer "F.Cu")
@@
 	)
 	(segment
-		(start 135.51 96.45)
-		(end 136.425 95.535)
+		(start 136.374199 101.35)
+		(end 135.51 100.485801)
 		(width 0.2)
 		(layer "F.Cu")
@@
 	)
 	(segment
-		(start 137.39 101.51)
-		(end 136.534199 101.51)
+		(start 136.425 95.535)
+		(end 136.93 95.535)
 		(width 0.2)
 		(layer "F.Cu")
@@
 	)
 	(segment
-		(start 136.534199 101.51)
-		(end 135.51 100.485801)
+		(start 135.51 100.485801)
+		(end 135.51 96.45)
 		(width 0.2)
 		(layer "F.Cu")
@@
 	)
 	(segment
-		(start 136.425 95.535)
-		(end 136.93 95.535)
+		(start 137.85 101.35)
+		(end 136.374199 101.35)
 		(width 0.2)
 		(layer "F.Cu")
@@
 	)
 	(via
-		(at 137.39 101.51)
+		(at 137.85 101.35)
 		(size 0.6)
 		(drill 0.3)
@@
 	)
 	(segment
-		(start 137.39 101.51)
-		(end 137.39 102.05)
+		(start 137.85 101.35)
+		(end 138.66 101.35)
 		(width 0.2)
 		(layer "B.Cu")
@@
 	)
 	(segment
-		(start 137.39 102.05)
-		(end 138.35 103.01)
-		(width 0.2)
-		(layer "B.Cu")
-		(net 68)
-	)
-	(segment
 		(start 138.565187 89.57008)
 		(end 137.700267 90.435)
@@
 	)
 	(via
-		(at 138.619999 107.02)
+		(at 136.92 106.16)
 		(size 0.9)
 		(drill 0.5)
@@
 	)
 	(via
-		(at 155.35 102.74)
+		(at 138.985 106.185)
 		(size 0.9)
 		(drill 0.5)
@@
 		(net 70)
 	)
-	(segment
-		(start 137.07 107.02)
-		(end 136.905 107.02)
-		(width 0.9)
-		(layer "B.Cu")
-		(net 70)
-	)
-	(segment
-		(start 138.619999 107.02)
-		(end 140 107.02)
-		(width 0.9)
-		(layer "B.Cu")
-		(net 70)
-	)
-	(segment
-		(start 136.285 106.4)
-		(end 136.285 104.685001)
-		(width 0.9)
-		(layer "B.Cu")
+	(via
+		(at 155.35 102.74)
+		(size 0.9)
+		(drill 0.5)
+		(layers "F.Cu" "B.Cu")
 		(net 70)
 	)
@@
 	)
 	(segment
-		(start 136.905 107.02)
-		(end 136.285 106.4)
-		(width 0.9)
-		(layer "B.Cu")
-		(net 70)
-	)
-	(segment
-		(start 138.619999 107.02)
-		(end 138.619999 107.880001)
-		(width 0.9)
-		(layer "B.Cu")
-		(net 70)
-	)
-	(segment
-		(start 135.665 107.02)
-		(end 135.635 107.05)
-		(width 0.9)
-		(layer "B.Cu")
-		(net 70)
-	)
-	(segment
-		(start 140 107.02)
-		(end 141.28 105.74)
-		(width 0.9)
-		(layer "B.Cu")
-		(net 70)
-	)
-	(segment
-		(start 137.14 109.36)
-		(end 135.6325 109.36)
-		(width 0.9)
-		(layer "B.Cu")
-		(net 70)
-	)
-	(segment
 		(start 155.35 102.74)
 		(end 156.68 102.74)
@@
 	)
 	(segment
-		(start 135.6625 109.33)
-		(end 135.6325 109.36)
-		(width 0.9)
-		(layer "B.Cu")
-		(net 70)
-	)
-	(segment
-		(start 141.28 105.74)
-		(end 141.28 104.66)
-		(width 0.9)
-		(layer "B.Cu")
-		(net 70)
-	)
-	(segment
-		(start 138.619999 107.02)
-		(end 135.665 107.02)
-		(width 0.9)
-		(layer "B.Cu")
-		(net 70)
-	)
-	(segment
-		(start 138.619999 107.880001)
-		(end 137.14 109.36)
-		(width 0.9)
-		(layer "B.Cu")
-		(net 70)
-	)
-	(segment
-		(start 141.235 105.775)
-		(end 144.27 102.74)
+		(start 136.92 106.16)
+		(end 139.01 106.16)
 		(width 0.9)
 		(layer "In1.Cu")
@@
 	)
 	(segment
-		(start 141.235 105.785)
-		(end 141.235 105.775)
-		(width 0.9)
-		(layer "In1.Cu")
-		(net 70)
-	)
-	(segment
-		(start 140 107.02)
-		(end 141.235 105.785)
+		(start 155.35 102.74)
+		(end 141.78 102.74)
 		(width 0.9)
 		(layer "In1.Cu")
@@
 	)
 	(segment
-		(start 138.619999 107.02)
-		(end 140 107.02)
+		(start 139.01 106.16)
+		(end 142.43 102.74)
 		(width 0.9)
 		(layer "In1.Cu")
@@
 	)
 	(segment
-		(start 155.35 102.74)
-		(end 141.78 102.74)
+		(start 142.43 102.74)
+		(end 144.27 102.74)
 		(width 0.9)
 		(layer "In1.Cu")
@@
 			)
 		)
+	)
+	(zone
+		(net 70)
+		(net_name "VBUS")
+		(layer "B.Cu")
+		(hatch edge 0.5)
+		(priority 5)
+		(connect_pads
+			(clearance 0.3)
+		)
+		(min_thickness 0.25)
+		(filled_areas_thickness no)
+		(fill yes
+			(thermal_gap 0.5)
+			(thermal_bridge_width 0.5)
+		)
+		(polygon
+			(pts
+				(xy 135.14 106.38) (xy 135.81 105.51) (xy 135.81 104.26) (xy 141.78 104.26) (xy 141.78 106.39) (xy 140.08 106.39)
+				(xy 137.7 108.49) (xy 137.7 110.06) (xy 135.14 110.06)
+			)
+		)

Commit message: WIP
Parts:
- added J5: Siedle BUS RX Test Pad, TestPoint:TestPoint_Pad_D1.0mm, B.Cu at (136.0, 97.7)
- R2: moved to B.Cu
- moved R2 3.10 mm to (153.8, 97.2), turned to 0 degrees
Connections:
- J4 pad 5: IO14 -> IO15
- J4 pad 6: IO15 -> IO16
- J4 pad 7: IO16 -> IO17
- J4 pad 8: IO17 -> IO18
- J4 pad 9: IO18 -> IO12
- U4 pad 16: I2C_CLK -> IO12
- U4 pad 17: I2C_DAT -> I2C_CLK
- U4 pad 18: IO14 -> I2C_DAT
Routing:
- net IO12: track 0.00 -> 14.5 mm, vias 0 -> 2
- net IO14: track 7.89 -> 0.00 mm
- net IO18: track 10.6 -> 3.14 mm, vias 2 -> 0
- net IO16: track 8.30 -> 3.02 mm
- net IO15: track 3.37 -> 7.54 mm
- net IO17: track 3.62 -> 7.67 mm
- net BUS_TX: track 22.1 -> 18.1 mm, vias 2 -> 1
- net SIEDLE_RX_DAT: track 10.6 -> 14.0 mm, vias 1 -> 2
- net Net-(Q1A-C1): track 12.0 -> 15.4 mm
- net VBUS: track 40.2 -> 38.4 mm
- net Net-(J1-CC2): track 11.8 -> 11.1 mm
Other:
- board text added: "B U S"
- board text added: "IH:RX"
- board text removed: "TC:BUS"

Commit message: WIP
Parts:
- moved C1 61.3 mm to (84.4, 43.4)
- moved C6 61.3 mm to (88.3, 49.0)
- moved G*** 61.3 mm to (115.6, 44.4)
- moved J9 61.3 mm to (101.8, 45.0)
- moved R1 61.3 mm to (82.2, 44.2)
- moved R14 61.3 mm to (82.3, 65.5)
- moved R21 61.3 mm to (87.5, 63.3)
- moved R5 61.3 mm to (106.7, 62.5)
- moved C2 61.3 mm to (89.1, 44.0)
- moved C5 61.3 mm to (82.3, 52.2)
- moved C7 61.3 mm to (86.9, 49.0)
- moved D4 61.3 mm to (110.5, 39.1)
- moved D5 61.3 mm to (114.2, 70.9)
- moved D6 61.3 mm to (82.4, 60.1)
- moved J6 61.3 mm to (110.8, 62.2)
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
Commit message: WIP
Parts:
- added C8: 10uF, Capacitor_SMD:C_1206_3216Metric, B.Cu at (82.3, 55.0)
- JP1: value Bus power Jumper -> Bus Power
- moved R10 3.72 mm to (82.6, 60.7), turned to 90 degrees
- moved D6 3.32 mm to (84.4, 57.5), turned to 0 degrees
Connections:
- D6 pad 1: /VCC_IN -> Net-(D6-K)
- JP1 pad 1: Net-(JP1-A) -> Net-(D6-A)
- R10 pad 1: Net-(D6-A) -> /VCC_IN
- R10 pad 2: Net-(JP1-A) -> Net-(D6-K)
- U4 pad 10: SIEDLE_TX_CAR -> SIEDLE_TX_DAT
- U4 pad 9: SIEDLE_TX_DAT -> SIEDLE_TX_CAR
Routing:
- net SIEDLE_TX_DAT: track 25.3 -> 19.7 mm
- net Net-(D6-K): track 0.00 -> 4.23 mm, vias 0 -> 1
- net Net-(JP1-A): track 2.47 -> 0.00 mm
- net /VCC_IN: track 66.8 -> 65.6 mm
- net Net-(D6-A): track 1.91 -> 2.41 mm

Commit message: WIP
Parts:
- moved Q2 0.87 mm to (109.5, 55.7)
- moved C8 0.13 mm to (82.4, 54.9)
- moved JP1 0.11 mm to (86.1, 59.6)
Routing:
- net GND: vias 120 -> 119
