File: pcb/doorman.kicad_pcb (KiCad board)
At the start: 4 copper layers, 37 x 37.2 mm, 62 parts, among them J1 USB-C Connector, J2 Screw Terminals, J3 3V3 Test Pad, J4 Extension Board Connector, J5 Siedle BUS RX Test Pad, J6 BUS Test Pad, J7 BUS RX Test Pad, J8 TX Test Pad, J9 RX Test Pad, Q1 BC847BPN, Q2 BC817-40, Q3 BC817-40, Q4 BC817-40, Q5 BC807-40, Q6 BC807-40, SW1 Button, SW2 Button, U2 AP63203WU, U3 GAQY252G3S, U4 ESP32-S3-MINI-1

Commit message: WIP
Parts:
- R18, R21: footprint Resistor_SMD:R_0603_1608Metric -> Resistor_SMD:R_0402_1005Metric
- moved J5 8.85 mm to (96.9, 62.8)
- moved R18 4.23 mm to (95.5, 60.3)
- moved R21 2.98 mm to (87.8, 60.3)
- moved R16 2.11 mm to (93.3, 63.7)
- moved R20 1.54 mm to (90.4, 63.7)
- moved R19 1.54 mm to (91.9, 63.7)
- moved Q6 1.24 mm to (89.9, 60.3)
- moved R17 0.99 mm to (94.8, 63.7)
- moved Q5 0.62 mm to (93.3, 60.3)
Connections:
- Q5 pad 2: SIEDLE_RX_DAT -> +3.3V
- Q5 pad 3: +3.3V -> SIEDLE_RX_DAT
- Q6 pad 2: SIEDLE_RX_CAR -> +3.3V
- Q6 pad 3: +3.3V -> SIEDLE_RX_CAR
Routing:
- net SIEDLE_RX_DAT: track 14.0 -> 12.0 mm, vias 2 -> 1
- net SIEDLE_RX_CAR: track 10.3 -> 8.56 mm
- net +3.3V: track 88.3 -> 89.3 mm
- net VBUS: track 38.2 -> 37.4 mm
- net Net-(Q6-B): track 3.10 -> 3.84 mm
- net Net-(Q5-B): track 3.15 -> 3.74 mm
- net GND: vias 119 -> 122

Commit message: WIP
Parts:
- moved D6 0.10 mm to (84.3, 57.5)
Changed lines of the file:
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@@
 	(footprint "Diode_SMD:D_SOD-323"
 		(layer "F.Cu")
-		(at 84.4125 57.47)
+		(at 84.3125 57.48)
 		(descr "SOD-323")
 		(tags "SOD-323")
@@
 	)
 	(segment
-		(start 86.14 58.11)
-		(end 86.14 59.62)
+		(start 85.3625 57.48)
+		(end 85.51 57.48)
 		(width 0.9)
 		(layer "F.Cu")
@@
 	)
 	(segment
-		(start 85.5 57.47)
-		(end 86.14 58.11)
+		(start 86.14 58.11)
+		(end 86.14 59.62)
 		(width 0.9)
 		(layer "F.Cu")
@@
 	)
 	(segment
-		(start 85.4625 57.47)
-		(end 85.5 57.47)
+		(start 85.51 57.48)
+		(end 86.14 58.11)
 		(width 0.9)
 		(layer "F.Cu")
@@
 	(segment
 		(start 82.45 58.0225)
-		(end 82.45 57.97)
+		(end 82.45 59.105)
 		(width 0.9)
 		(layer "F.Cu")
@@
 	)
 	(segment
-		(start 82.45 58.0225)
-		(end 82.45 59.105)
+		(start 82.95 57.47)
+		(end 83.2525 57.47)
 		(width 0.9)
 		(layer "F.Cu")
@@
 	)
 	(segment
-		(start 82.95 57.47)
-		(end 83.3625 57.47)
+		(start 83.2525 57.47)
+		(end 83.2625 57.48)
 		(width 0.9)
 		(layer "F.Cu")
@@
 		(net 26)
 	)
+	(segment
+		(start 82.45 58.0225)
+		(end 82.45 57.97)
+		(width 0.9)
+		(layer "F.Cu")
+		(net 26)
+	)
 	(via
 		(at 82.45 58.0225)
@@
 	)
 	(segment
-		(start 87.9 56.215)
-		(end 87.9 55.115001)
-		(width 1)
-		(layer "F.Cu")
-		(net 54)
-	)
-	(segment
 		(start 85.71 66.23)
 		(end 85.71 64.18)
@@
 	)
 	(segment
-		(start 85.36 64.13)
-		(end 83.23 64.13)
-		(width 0.9)
+		(start 85.71 64.17)
+		(end 85.71 64.18)
+		(width 1)
 		(layer "F.Cu")
 		(net 54)
 	)
 	(segment
-		(start 87.9 56.215)
-		(end 87.9 61.99)
-		(width 1)
+		(start 85.36 64.13)
+		(end 83.23 64.13)
+		(width 0.9)
 		(layer "F.Cu")
 		(net 54)
@@
 	)
 	(segment
-		(start 87.9 61.99)
-		(end 85.71 64.18)
-		(width 1)
-		(layer "F.Cu")
-		(net 54)
-	)
-	(segment
-		(start 87.9 55.115001)
-		(end 87.84 55.055001)
-		(width 1)
-		(layer "F.Cu")
-		(net 54)
-	)
-	(segment
 		(start 87.835 55.060001)
 		(end 87.835 55.130001)
@@
 	)
 	(segment
+		(start 88.24 55.455001)
+		(end 87.84 55.055001)
+		(width 1)
+		(layer "F.Cu")
+		(net 54)
+	)
+	(segment
 		(start 83.23 64.13)
 		(end 82.63 63.53)
@@
 	)
 	(segment
+		(start 88.24 56.41)
+		(end 88.24 55.455001)
+		(width 1)
+		(layer "F.Cu")
+		(net 54)
+	)
+	(segment
 		(start 90.335 70.855)
 		(end 91.4925 70.855)
@@
 		(net 54)
 	)
+	(segment
+		(start 88.24 56.41)
+		(end 88.24 61.64)
+		(width 1)
+		(layer "F.Cu")
+		(net 54)
+	)
+	(segment
+		(start 88.24 61.64)
+		(end 85.71 64.17)
+		(width 1)
+		(layer "F.Cu")
+		(net 54)
+	)
 	(via
 		(at 102.03 60.56)
@@
 	)
 	(via
-		(at 87.9 56.215)
+		(at 88.24 56.41)
 		(size 0.9)
 		(drill 0.5)
@@
 	)
 	(segment
-		(start 100.38 58.91)
-		(end 102.03 60.56)
+		(start 88.24 56.41)
+		(end 93.82 56.41)
 		(width 1)
 		(layer "In1.Cu")
@@
 	)
 	(segment
-		(start 93.625 56.215)
-		(end 96.32 58.91)
-		(width 1)
-		(layer "In1.Cu")
-		(net 54)
-	)
-	(segment
 		(start 111.895 70.87)
 		(end 111.91 70.855)
@@
 	)
 	(segment
-		(start 87.9 56.215)
-		(end 93.625 56.215)
+		(start 96.32 58.91)
+		(end 100.38 58.91)
 		(width 1)
 		(layer "In1.Cu")
@@
 	)
 	(segment
-		(start 96.32 58.91)
-		(end 100.38 58.91)
+		(start 93.82 56.41)
+		(end 96.32 58.91)
+		(width 1)
+		(layer "In1.Cu")
+		(net 54)
+	)
+	(segment
+		(start 100.38 58.91)
+		(end 102.03 60.56)
 		(width 1)
 		(layer "In1.Cu")
@@
 	(segment
 		(start 89.92 59.394999)
-		(end 88.165001 59.394999)
+		(end 89.92 59.81)
 		(width 0.2)
 		(layer "B.Cu")
@@
 	)
 	(segment
-		(start 88.165001 59.394999)
+		(start 89.92 59.81)
 		(end 87.75 59.81)
 		(width 0.2)
@@
 	)
 	(segment
+		(start 93.32 59.81)
+		(end 93.32 59.384999)
+		(width 0.2)
+		(layer "B.Cu")
+		(net 59)
+	)
+	(segment
 		(start 95.49 59.81)
 		(end 95.99 59.81)
@@
 	)
 	(segment
-		(start 95.064999 59.384999)
-		(end 93.32 59.384999)
+		(start 95.49 59.81)
+		(end 93.32 59.81)
 		(width 0.2)
 		(layer "B.Cu")
@@
 	)
 	(segment
-		(start 95.49 59.81)
-		(end 95.064999 59.384999)
-		(width 0.2)
-		(layer "B.Cu")
-		(net 59)
-	)
-	(segment
 		(start 96.63 62.55)
 		(end 96.89 62.81)
@@
 	)
 	(segment
-		(start 82.19 64.475)
-		(end 82.35 64.635)
+		(start 84.94 56.742958)
+		(end 84.94 59.77)
 		(width 0.2)
 		(layer "B.Cu")
@@
 	)
 	(segment
-		(start 91.8 50.71)
-		(end 90.972958 50.71)
+		(start 82.19 64.475)
+		(end 82.35 64.635)
 		(width 0.2)
 		(layer "B.Cu")
@@
 	)
 	(segment
-		(start 83.24 60.35)
-		(end 82.35 61.24)
+		(start 90.972958 50.71)
+		(end 84.94 56.742958)
 		(width 0.2)
 		(layer "B.Cu")
@@
 	)
 	(segment
-		(start 84.79 59.92)
-		(end 84.36 60.35)
+		(start 91.8 50.71)
+		(end 90.972958 50.71)
 		(width 0.2)
 		(layer "B.Cu")
@@
 	)
 	(segment
-		(start 84.79 56.892958)
-		(end 84.79 59.92)
+		(start 84.45 60.26)
+		(end 83.33 60.26)
 		(width 0.2)
 		(layer "B.Cu")
@@
 	)
 	(segment
-		(start 90.972958 50.71)
-		(end 84.79 56.892958)
+		(start 83.33 60.26)
+		(end 82.35 61.24)
 		(width 0.2)
 		(layer "B.Cu")
@@
 	)
 	(segment
-		(start 84.36 60.35)
-		(end 83.24 60.35)
+		(start 84.94 59.77)
+		(end 84.45 60.26)
 		(width 0.2)
 		(layer "B.Cu")

Commit message: WIP
Parts:
- removed Q5: BC807-40, Package_TO_SOT_SMD:SOT-23
- removed R19: 10K, Resistor_SMD:R_0603_1608Metric
- removed R20: 2K, Resistor_SMD:R_0603_1608Metric
- removed R21: 1K, Resistor_SMD:R_0402_1005Metric
- added D3: 5.1V, Diode_SMD:D_SOD-123, B.Cu at (89.5, 62.4)
- added J10: VCC Test Pad, TestPoint:TestPoint_Pad_D1.0mm, B.Cu at (103.0, 59.3)
- Q6: value BC807-40 -> BC847BPN; footprint Package_TO_SOT_SMD:SOT-23 -> Package_TO_SOT_SMD:SOT-363_SC-70-6
- R13, R15: footprint Resistor_SMD:R_0805_2012Metric -> Resistor_SMD:R_1206_3216Metric
- moved J5 8.98 mm to (89.4, 57.9)
- moved R18 6.87 mm to (91.0, 55.1), turned to 180 degrees
- moved Q6 3.79 mm to (93.7, 59.8), turned to 180 degrees
- moved J3 3.13 mm to (86.1, 47.9)
- moved J6 2.71 mm to (108.1, 62.1)
- moved R17 0.65 mm to (94.3, 63.3)
- moved R16 0.65 mm to (92.9, 63.3)
- moved R13 0.53 mm to (89.4, 66.5)
- moved R15 0.52 mm to (89.3, 68.8)
Connections:
- net BUS_TX renamed BUS_TX_TC
- net SIEDLE_TX_CAR renamed BUS_TX_IHB_CAR
- net SIEDLE_TX_DAT renamed BUS_TX_IHB
- J5 pad 1: SIEDLE_RX_DAT -> BUS_RX_IHB
- Q6 pad 1: Net-(Q6-B) -> unconnected-(Q6A-E1-Pad1)
- Q6 pad 2: +3.3V -> unconnected-(Q6A-B1-Pad2)
- Q6 pad 3: SIEDLE_RX_CAR -> BUS_RX_IHB
- R16 pad 2: Net-(Q5-B) -> Net-(D3-K)
- R17 pad 1: Net-(Q5-B) -> Net-(D3-K)
- R18 pad 1: SIEDLE_RX_DAT -> BUS_RX_IHB
- U4 pad 14: SIEDLE_RX_CAR -> BUS_RX_IHB
- U4 pad 15: SIEDLE_RX_DAT -> unconnected-(U4-IO11-Pad15)
Routing:
- net BUS_RX_IHB: track 0.00 -> 13.4 mm, vias 0 -> 1
- net SIEDLE_RX_DAT: track 12.2 -> 0.00 mm, vias 1 -> 0
- net SIEDLE_RX_CAR: track 8.80 -> 0.00 mm, vias 1 -> 0
- net Net-(D3-K): track 0.00 -> 6.51 mm
- net Net-(Q6-B): track 3.84 -> 0.00 mm
- net Net-(Q5-B): track 3.74 -> 0.00 mm
- net BUS_WIRE1: track 28.0 -> 25.4 mm
- net +3.3V: track 89.3 -> 87.5 mm
- net /VCC_IN: track 65.5 -> 67.2 mm
- net GND: vias 122 -> 130
Other:
- board text added: "IHB:RX"
- board text added: "RXD"
- board text added: "TXD"
- board text added: "VBUS"
- board text added: "VIN"
- board text removed: "IH:RX"
- board text removed: "RX"
- board text removed: "TX"

Commit message: WIP
Parts:
- added L2: 100uH, Inductor_SMD:L_Sunlord_SWPA3015S, B.Cu at (106.9, 70.4)
- added L3: 100uH, Inductor_SMD:L_Sunlord_SWPA3015S, B.Cu at (110.4, 70.4)
- moved D5 0.39 mm to (114.6, 70.8)
Connections:
- D2 pad 1: BUS_WIRE1 -> Net-(D2-Pad1)
- D2 pad 2: BUS_WIRE2 -> Net-(D2-Pad2)
Routing:
- net BUS_WIRE2: track 24.0 -> 21.1 mm, vias 2 -> 1
- net Net-(D2-Pad2): track 0.00 -> 2.84 mm, vias 0 -> 1
- net BUS_WIRE1: track 25.4 -> 23.3 mm, vias 2 -> 1
- net Net-(D2-Pad1): track 0.00 -> 1.91 mm, vias 0 -> 1
- net /VCC_IN: track 67.2 -> 68.7 mm
- net GND: vias 130 -> 132
Other:
- board text added: "BUS"

Commit message: WIP
Routing:
- net GND: vias 132 -> 131
Changed lines of the file:
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@@
 	)
 	(via
-		(at 84.91 61.87)
-		(size 0.6)
-		(drill 0.3)
-		(layers "F.Cu" "B.Cu")
-		(free yes)
-		(net 2)
-	)
-	(via
 		(at 90.5 64.22)
 		(size 0.6)
@@
 	)
 	(via
-		(at 85.78 61.86)
+		(at 85.860639 61.940001)
 		(size 0.6)
 		(drill 0.3)
@@
 	)
 	(segment
+		(start 106.93 68.77)
+		(end 106.93 69.21)
+		(width 0.8)
+		(layer "B.Cu")
+		(net 18)
+	)
+	(segment
 		(start 115.61 62.87)
 		(end 115.14 62.87)
@@
 	)
 	(segment
-		(start 106.93 68.77)
-		(end 106.93 69.21)
-		(width 0.8)
-		(layer "B.Cu")
-		(net 18)
-	)
-	(segment
 		(start 115.61 62.87)
 		(end 113.01 62.87)
@@
 	)
 	(segment
-		(start 110.45 68.76)
-		(end 110.44 68.77)
+		(start 110.44 68.77)
+		(end 110.44 69.21)
 		(width 0.8)
 		(layer "B.Cu")
@@
 	)
 	(segment
-		(start 110.44 68.77)
-		(end 110.44 69.21)
+		(start 110.45 68.76)
+		(end 110.44 68.77)
 		(width 0.8)
 		(layer "B.Cu")
@@
 	)
 	(segment
-		(start 91.265 49.865)
-		(end 84.31 56.82)
-		(width 0.2)
-		(layer "B.Cu")
-		(net 69)
-	)
-	(segment
-		(start 91.810267 49.865)
-		(end 91.265 49.865)
-		(width 0.2)
-		(layer "B.Cu")
-		(net 69)
-	)
-	(segment
-		(start 84.31 59.135)
+		(start 84.02 57.655267)
 		(end 84.02 59.425)
 		(width 0.2)
@@
 	)
 	(segment
-		(start 84.31 56.82)
-		(end 84.31 59.135)
+		(start 91.810267 49.865)
+		(end 84.02 57.655267)
 		(width 0.2)
 		(layer "B.Cu")
@@
 	)
 	(segment
-		(start 84.94 57.1)
-		(end 84.94 59.77)
-		(width 0.2)
-		(layer "B.Cu")
-		(net 70)
-	)
-	(segment
-		(start 84.45 60.26)
-		(end 83.33 60.26)
+		(start 91.8 50.71)
+		(end 84.94 57.57)
 		(width 0.2)
 		(layer "B.Cu")
@@
 	)
 	(segment
-		(start 82.35 61.24)
+		(start 82.19 64.475)
 		(end 82.35 64.635)
 		(width 0.2)
@@
 	)
 	(segment
-		(start 82.19 64.475)
-		(end 82.35 64.635)
+		(start 84.5 60.26)
+		(end 83.3 60.26)
 		(width 0.2)
 		(layer "B.Cu")
@@
 	)
 	(segment
-		(start 83.33 60.26)
-		(end 82.35 61.24)
+		(start 84.94 59.82)
+		(end 84.5 60.26)
 		(width 0.2)
 		(layer "B.Cu")
@@
 	)
 	(segment
-		(start 91.8 50.71)
-		(end 91.33 50.71)
+		(start 82.35 61.21)
+		(end 82.35 64.635)
 		(width 0.2)
 		(layer "B.Cu")
@@
 	)
 	(segment
-		(start 91.33 50.71)
-		(end 84.94 57.1)
+		(start 83.3 60.26)
+		(end 82.35 61.21)
 		(width 0.2)
 		(layer "B.Cu")
@@
 	)
 	(segment
-		(start 84.94 59.77)
-		(end 84.45 60.26)
+		(start 84.94 57.57)
+		(end 84.94 59.82)
 		(width 0.2)
 		(layer "B.Cu")

Commit message: WIP
Parts:
- removed L2, L3: 100uH, Inductor_SMD:L_Sunlord_SWPA3015S
Connections:
- D2 pad 1: Net-(D2-Pad1) -> BUS_WIRE1
- D2 pad 2: Net-(D2-Pad2) -> BUS_WIRE2
Routing:
- net BUS_WIRE2: track 21.1 -> 24.7 mm, vias 1 -> 2
- net Net-(D2-Pad2): track 2.84 -> 0.00 mm, vias 1 -> 0
- net BUS_WIRE1: track 23.3 -> 25.8 mm, vias 1 -> 2
- net Net-(D2-Pad1): track 1.91 -> 0.00 mm, vias 1 -> 0
- net /VCC_IN: track 68.7 -> 67.6 mm
- net GND: vias 131 -> 129

Commit message: WIP
Parts:
- moved J5 1.37 mm to (90.1, 56.7)
Routing:
- net BUS_RX_IHB: track 13.4 -> 11.9 mm
Changed lines of the file:
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@@
 	(footprint "TestPoint:TestPoint_Pad_D1.0mm"
 		(layer "B.Cu")
-		(at 89.4 57.85 180)
+		(at 90.11 56.68 180)
 		(descr "SMD pad as test Point, diameter 1.0mm")
 		(tags "test point SMD pad")
@@
 	)
 	(segment
-		(start 93.44 54.86)
-		(end 92.75 54.86)
+		(start 92.09 55.52)
+		(end 92.09 56.015)
 		(width 0.2)
 		(layer "F.Cu")
@@
 	)
 	(segment
-		(start 92.09 55.52)
-		(end 92.09 56.015)
+		(start 98.19 60.81)
+		(end 98.2 60.8)
 		(width 0.2)
 		(layer "F.Cu")
@@
 	)
 	(segment
-		(start 98.19 60.81)
-		(end 98.2 60.8)
+		(start 92.91 54.7)
+		(end 92.09 55.52)
 		(width 0.2)
 		(layer "F.Cu")
@@
 	)
 	(segment
-		(start 92.75 54.86)
-		(end 92.09 55.52)
+		(start 93.68 54.7)
+		(end 92.91 54.7)
 		(width 0.2)
 		(layer "F.Cu")
@@
 	)
 	(via
-		(at 93.44 54.86)
+		(at 93.68 54.7)
 		(size 0.6)
 		(drill 0.3)
@@
 	)
 	(segment
-		(start 93.44 54.86)
-		(end 94.05 54.86)
+		(start 93.68 54.7)
+		(end 94.04 54.7)
 		(width 0.2)
 		(layer "B.Cu")
@@
 	)
 	(segment
-		(start 97.97 58.78)
+		(start 97.97 58.63)
 		(end 97.97 60.81)
 		(width 0.2)
@@
 	)
 	(segment
-		(start 94.05 54.86)
-		(end 97.97 58.78)
+		(start 94.04 54.7)
+		(end 97.97 58.63)
 		(width 0.2)
 		(layer "B.Cu")
@@
 	)
 	(segment
-		(start 94.7 57.15)
-		(end 95.39 57.84)
-		(width 0.2)
-		(layer "B.Cu")
-		(net 67)
-	)
-	(segment
-		(start 91.55 56.12)
-		(end 92.58 57.15)
-		(width 0.2)
-		(layer "B.Cu")
-		(net 67)
-	)
-	(segment
-		(start 91.55 54.42)
-		(end 91.55 55.09)
+		(start 94.98 60.4)
+		(end 94.62 60.4)
 		(width 0.2)
 		(layer "B.Cu")
@@
 	)
 	(segment
-		(start 91.55 55.09)
-		(end 91.55 55.71)
-		(width 0.2)
-		(layer "B.Cu")
-		(net 67)
-	)
-	(segment
-		(start 95.39 57.84)
+		(start 95.39 58.31)
 		(end 95.39 59.99)
 		(width 0.2)
@@
 	)
 	(segment
-		(start 91.85 54.12)
-		(end 91.55 54.42)
+		(start 91.55 54.42)
+		(end 91.55 55.09)
 		(width 0.2)
 		(layer "B.Cu")
@@
 	)
 	(segment
-		(start 91.13 56.12)
-		(end 89.4 57.85)
+		(start 91.55 55.24)
+		(end 90.11 56.68)
 		(width 0.2)
 		(layer "B.Cu")
@@
 	)
 	(segment
-		(start 91.55 56.12)
-		(end 91.13 56.12)
+		(start 91.55 55.09)
+		(end 92.17 55.09)
 		(width 0.2)
 		(layer "B.Cu")
@@
 	)
 	(segment
-		(start 92.58 57.15)
-		(end 94.7 57.15)
+		(start 91.85 54.12)
+		(end 91.55 54.42)
 		(width 0.2)
 		(layer "B.Cu")
@@
 	)
 	(segment
-		(start 91.55 55.71)
-		(end 91.55 56.12)
+		(start 91.55 55.09)
+		(end 91.55 55.24)
 		(width 0.2)
 		(layer "B.Cu")
@@
 	)
 	(segment
-		(start 94.98 60.4)
-		(end 94.62 60.4)
+		(start 92.17 55.09)
+		(end 95.39 58.31)
 		(width 0.2)
 		(layer "B.Cu")
