File: pcb_extension_audio/doorman_audio_extension.kicad_pcb (KiCad board)
At the start: 4 copper layers, 31.4 x 29.6 mm, 39 parts, among them J1 Audio Out CH2, J4 Conn_02x07_Odd_Even, J5 Audio In CH2, U1 ES8388

Commit message: WIP
Parts:
- C1, C10: value 0.1uF -> 100nF; moved to F.Cu
- C11, C12, C13, C14, C17, C18, C19, C2, C20, C21, C3, C4, C5, C6, C7, D1, D2, R1, R13, R14, R15, R16, R17, R18, R19, R2, R20, R21, R3, R5, R6, U1: moved to F.Cu
- G***, REF**: moved to B.Cu
- J1: value Audio Out CH2 -> Audio Out; moved to B.Cu
- J4: value Conn_02x07_Odd_Even -> Extension Board Connector; moved to F.Cu
- J5: value Audio In CH2 -> Audio In; moved to B.Cu
- moved J1 77.0 mm to (205.6, 86.3), turned to 180 degrees
- moved REF** 72.6 mm to (203.1, 98.6), turned to 180 degrees
- moved D2 65.3 mm to (199.8, 87.0)
- moved R13 62.4 mm to (198.3, 98.7)
- moved R14 62.4 mm to (198.3, 101.9)
- moved R6 60.8 mm to (192.4, 107.3), turned to 180 degrees
- moved R1 60.1 mm to (197.1, 88.1)
- moved R3 60.1 mm to (197.1, 85.1)
- moved R17 58.7 mm to (196.4, 93.3), turned to 0 degrees
- moved R19 58.7 mm to (196.4, 91.8), turned to 0 degrees
- moved C17 58.7 mm to (196.4, 90.3), turned to 180 degrees
- moved C13 57.2 mm to (195.7, 85.1)
- moved C6 57.2 mm to (195.7, 88.1)
- moved C14 55.3 mm to (187.9, 107.3), turned to 0 degrees
- moved C7 52.6 mm to (193.3, 85.8), turned to 0 degrees
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Connections:
- J5 pad 1: AUDIO_IN_R1 -> AUDIO_IN_R2
- J5 pad 3: AUDIO_IN_R2 -> AUDIO_IN_R1
- U1 pad : GND -> (no net)
Routing:
- net AUDIO_OUT_L1: track 12.5 -> 34.2 mm, vias 0 -> 2
- net BUS_WIRE2: track 26.1 -> 10.8 mm, vias 2 -> 0
- net GND: track 18.9 -> 12.3 mm, vias 70 -> 68
- net +3.3V: track 56.0 -> 53.0 mm
- net I2C_CLK: track 18.8 -> 20.5 mm
- net AUDIO_IN_L1: track 17.0 -> 16.0 mm
- net AUDIO_OUT_L2: track 15.1 -> 16.0 mm
- net I2C_DAT: track 17.2 -> 17.8 mm
- net Net-(C14-Pad2): track 2.12 -> 1.61 mm
- net AUDIO_OUT_R1: track 9.69 -> 9.53 mm, vias 1 -> 0
Other:
- outline, holes or cut-outs redrawn
- board text added: "PCB3D_BR_doorman_ea"
- board text added: "PCB3D_TL_doorman_ea"
- board text removed: "PCB3D_BR_doorman"
- board text removed: "PCB3D_TL_doorman"

Commit message: WIP
Parts:
- removed R20, R21: 10K, Resistor_SMD:R_0603_1608Metric
- R6: value 1K -> 200
- moved D1 3.31 mm to (180.2, 92.9), turned to 90 degrees
Routing:
- net +3.3V: track 53.0 -> 52.2 mm
- net AUDIO_IN_L1: track 16.0 -> 15.2 mm
- net GND: vias 68 -> 74
Other:
- board text added: "AUDIO IN"
- board text added: "AUDIO OUT"
- board text added: "INPUTS"
- board text added: "OUTPUTS"

Commit message: WIP
Parts:
- C12, C14: value 1uF -> 10uF
- moved D1 0.76 mm to (180.2, 93.7)
Routing:
- net +3.3V: track 52.2 -> 51.1 mm
- net AUDIO_OUT_L2: track 16.0 -> 15.0 mm
- net GND: vias 74 -> 77
Other:
- board text added: "ES8388"
- board text added: "ONLY FOR TC:BUS INTERCOM SYSTEMS"
- board text removed: "AUDIO IN"
- board text removed: "AUDIO OUT"
- board text removed: "DO NOT USE THIS WITH NON TC:BUS INTERCOM SYSTEMS"

Commit message: WIP
Parts:
- removed C4: 1uF, Capacitor_SMD:C_0603_1608Metric
- added G***: LOGO, Doorman:doorman-web-qr, F.Cu at (202.8, 98.3)
- J5: footprint Connector_PinHeader_2.54mm:PinHeader_1x03_P2.54mm_Vertical -> Connector_PinHeader_2.54mm:PinHeader_1x02_P2.54mm_Vertical
- moved C12 3.40 mm to (180.2, 96.2)
- moved D1 1.61 mm to (179.2, 92.5), turned to 180 degrees
Connections:
- U1 pad 23: Net-(U1-RIN1) -> AUDIO_OUT_L1
Routing:
- net AUDIO_OUT_L1: track 34.2 -> 44.8 mm, vias 2 -> 4
- net AUDIO_IN_R1: track 6.10 -> 0.00 mm
- net AUDIO_IN_L1: track 15.1 -> 11.6 mm, vias 2 -> 0
- net BUS_WIRE2: track 10.8 -> 14.3 mm
- net Net-(U1-RIN1): track 3.31 -> 0.00 mm
- net GND: vias 77 -> 79
Other:
- board text added: "SCAN ME"
- board text removed: "ONLY FOR TC:BUS INTERCOM SYSTEMS"

Commit message: WIP
Parts:
- moved C14 1.61 mm to (187.9, 108.9)
- moved R6 1.61 mm to (192.4, 108.9)
- moved G*** 0.63 mm to (203.1, 98.8)
Connections:
- U1 pad : (no net) -> GND
Routing:
- net BUS_WIRE2: track 14.3 -> 15.9 mm
- net AUDIO_OUT_L1: track 44.8 -> 46.4 mm
- net GND: vias 79 -> 80
Other:
- board text added: "02 01"
- board text added: "02 04 06 08 10 12 14 01 03 05 07 09 11 13"
- board text added: "04 03"
- board text added: "06 05"
- board text added: "08 07"
- board text added: "10 09"
- board text added: "12 11"
- board text added: "13 I²CCLK 11 GND 09 I²SOUT 07 I²SBCLK 05 - 03 GND 01 TC:BUS"
- board text added: "14 13"
- board text added: "3V3 14 I²CDAT 12 I²SLRCK 10 I²SIN 08 I²SMCLK 06 - 04 TC:BUS 02"
- board text added: "CHECK THE DOCS"
- board text added: "EXTENSION CONNECTOR"
- board text removed: "SCAN ME"

Commit message: WIP
Parts:
- added U2: ES8388, Package_DFN_QFN:QFN-28-1EP_4x4mm_P0.45mm_EP2.6x2.6mm, F.Cu at (179.8, 108.4)
Connections:
- J4 pad 10: I2S_LRCK -> I2S_MCLK
- J4 pad 11: GND -> I2S_DAT_IN
- J4 pad 12: I2C_DAT -> I2S_LRCK
- J4 pad 13: I2C_CLK -> I2C_DAT
- J4 pad 2: BUS_WIRE1 -> GND
- J4 pad 3: GND -> unconnected-(J4-Pin_3-Pad3)
- J4 pad 4: unconnected-(J4-Pin_4-Pad4) -> I2S_BCLK
- J4 pad 5: unconnected-(J4-Pin_5-Pad5) -> I2S_DAT_OUT
- J4 pad 6: I2S_MCLK -> GND
- J4 pad 7: I2S_SCLK -> I2C_CLK
- J4 pad 8: I2S_DAT_IN -> BUS_WIRE1
- J4 pad 9: I2S_DAT_OUT -> unconnected-(J4-Pin_9-Pad9)
- R16 pad 2: I2S_SCLK -> I2S_BCLK
- U1 pad : GND -> (no net)
Routing:
- net GND: track 12.3 -> 20.9 mm, vias 80 -> 82
- net I2S_SCLK: track 7.95 -> 0.00 mm
- net I2S_BCLK: track 0.00 -> 7.95 mm
- net AUDIO_OUT_L1: track 46.4 -> 47.3 mm
Other:
- board text added: "01"
- board text added: "02"
- board text added: "03"
- board text added: "04"
- board text added: "05"
- board text added: "06"
- board text added: "07"
- board text added: "07 I²C CLK 06 GND 05 I²S OUT 04 I²S BCLK 03 - 02 GND 01 TC:BUS"
- board text added: "13"
- board text added: "14"
- board text added: "3V3 14 I²C DAT 13 I²S LRCK 12 I²S IN 11 I²S MCLK 10 - 09 TC:BUS 08"
- board text removed: "02 01"
- board text removed: "02 04 06 08 10 12 14 01 03 05 07 09 11 13"
- board text removed: "04 03"
- board text removed: "06 05"
- board text removed: "08 07"
- board text removed: "10 09"
- board text removed: "12 11"
- board text removed: "13 I²CCLK 11 GND 09 I²SOUT 07 I²SBCLK 05 - 03 GND 01 TC:BUS"
- board text removed: "14 13"
- board text removed: "3V3 14 I²CDAT 12 I²SLRCK 10 I²SIN 08 I²SMCLK 06 - 04 TC:BUS 02"

Commit message: WIP
Parts:
- removed U2: ES8388, Package_DFN_QFN:QFN-28-1EP_4x4mm_P0.45mm_EP2.6x2.6mm
Other:
- board text removed: "02"
- board text removed: "03"
- board text removed: "05"
- board text removed: "06"
- board text removed: "13"

Commit message: WIP
Parts:
- added J2: GPIO, Connector_PinHeader_2.54mm:PinHeader_1x02_P2.54mm_Vertical, F.Cu at (177.7, 108.4)
Connections:
- J4 pad 3: unconnected-(J4-Pin_3-Pad3) -> PIN3
- J4 pad 9: unconnected-(J4-Pin_9-Pad9) -> PIN9
Routing:
- net PIN3: track 0.00 -> 14.4 mm, vias 0 -> 1
- net PIN9: track 0.00 -> 12.6 mm, vias 0 -> 1
Other:
- board text added: "07 I²C CLK 06 GND 05 I²S OUT 04 I²S BCLK 03 P3 02 GND 01 TC:BUS"
- board text added: "3V3 14 I²C DAT 13 I²S LRCK 12 I²S IN 11 I²S MCLK 10 P9 09 TC:BUS 08"
- board text added: "GPIOS"
- board text added: "P3"
- board text added: "P9"
- board text removed: "04"
- board text removed: "07 I²C CLK 06 GND 05 I²S OUT 04 I²S BCLK 03 - 02 GND 01 TC:BUS"
- board text removed: "3V3 14 I²C DAT 13 I²S LRCK 12 I²S IN 11 I²S MCLK 10 - 09 TC:BUS 08"
