File: pcb_extension_audio/doorman_audio_extension.kicad_pcb (KiCad board)
At the start: 4 copper layers, 31.4 x 29.6 mm, 38 parts, among them J1 Audio Out, J2 GPIO, J4 Extension Board Connector, J5 Audio In, U1 ES8388

Commit message: WIP
Parts:
- added R4: 0, Resistor_SMD:R_0603_1608Metric, F.Cu at (184.1, 90.3)
- moved C11 4.44 mm to (187.9, 95.3)
- moved C10 4.44 mm to (189.3, 95.3)
- moved R17 3.38 mm to (193.7, 95.3), turned to -90 degrees
- moved R15 3.09 mm to (186.4, 95.3), turned to -90 degrees
- moved R16 1.91 mm to (190.8, 95.3), turned to -90 degrees
- moved R13 1.30 mm to (198.3, 100.0)
- moved R18 0.84 mm to (192.2, 95.3), turned to -90 degrees
- moved R6 0.68 mm to (192.5, 108.2)
- moved C14 0.67 mm to (187.9, 108.2)
Connections:
- net PIN9 renamed VCC
- C12 pad 2: AUDIO_IN_L1 -> Net-(D1-K)
- D1 pad 1: AUDIO_IN_L1 -> Net-(D1-K)
- J4 pad 11: I2S_DAT_IN -> I2S_BCLK
- J4 pad 4: I2S_BCLK -> I2S_DAT_IN
Routing:
- net +3.3V: track 51.1 -> 40.1 mm
- net AUDIO_IN_L1: track 11.6 -> 3.29 mm
- net GND: track 20.9 -> 14.0 mm, vias 82 -> 94
- net Net-(D1-K): track 0.00 -> 6.69 mm
- net I2S_DAT_OUT: track 20.7 -> 14.0 mm, vias 2 -> 0
- net I2S_MCLK: track 10.2 -> 4.13 mm, vias 2 -> 0
- net AUDIO_OUT_L1: track 47.3 -> 42.2 mm
- net I2S_LRCK: track 8.60 -> 3.49 mm
- net I2S_BCLK: track 7.95 -> 3.15 mm
- net I2S_DAT_IN: track 3.29 -> 7.94 mm
- net I2C_CLK: track 20.5 -> 23.0 mm
- net Net-(U1-LRCK): track 5.18 -> 2.91 mm
- net I2C_DAT: track 17.8 -> 20.0 mm
- net Net-(U1-SCLK): track 3.49 -> 1.66 mm
- net Net-(U1-DSDIN): track 3.97 -> 2.17 mm
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Other:
- board text added: "07 I²C CLK 06 GND 05 I²S OUT 04 P4 03 I²S MCLK 02 GND 01 TC:BUS"
- board text added: "3V3 14 I²C DAT 13 I²S LRCK 12 I²S IN 11 I²S BCLK 10 VCC 09 TC:BUS 08"
- board text added: "EXTRAS"
- board text added: "VCC"
- board text removed: "07 I²C CLK 06 GND 05 I²S OUT 04 I²S BCLK 03 P3 02 GND 01 TC:BUS"
- board text removed: "3V3 14 I²C DAT 13 I²S LRCK 12 I²S IN 11 I²S MCLK 10 P9 09 TC:BUS 08"
- board text removed: "GPIOS"
- board text removed: "P9"

Commit message: WIP
Parts:
- G***: moved to B.Cu
- J1: footprint Connector_PinHeader_2.54mm:PinHeader_1x03_P2.54mm_Vertical -> Connector_PinHeader_2.54mm:PinHeader_1x04_P2.54mm_Vertical
- J5: footprint Connector_PinHeader_2.54mm:PinHeader_1x02_P2.54mm_Vertical -> Connector_PinHeader_2.54mm:PinHeader_1x03_P2.54mm_Vertical
- REF**: moved to F.Cu
- moved D1 1.78 mm to (179.2, 94.3)
- moved C12 1.69 mm to (180.2, 97.9)
- moved G*** 0.39 mm to (202.8, 98.5), turned to 180 degrees
- moved REF** 0.32 mm to (203.4, 98.8), turned to 0 degrees
Routing:
- net BUS_WIRE2: track 15.3 -> 13.6 mm
- net Net-(D1-K): track 6.69 -> 8.38 mm
- net GND: vias 94 -> 91
Other:
- board text added: "G"
- board text added: "HP"
- board text added: "HP=47uF LN=1uF"
- board text added: "LN"
- board text added: "SCAN QR CODE FOR DOCS"
- board text removed: "CHECK THE DOCS"

Commit message: WIP
Parts:
- moved C1 1.48 mm to (190.3, 85.8)
- moved C2 1.46 mm to (190.3, 84.4)
Routing:
- net GND: vias 91 -> 95
Other:
- board text added: "08 TC:BUS 09 VCC 10 I²S BCLK 11 I²S IN 12 I²S LRCK 13 I²C DAT 14 3V3"
- board text added: "HP 47uF LN 1uF"
- board text added: "TC:BUS 01 GND 02 I²S MCLK 03 P4 04 I²S OUT 05 GND 06 I²C CLK 07"
- board text removed: "07 I²C CLK 06 GND 05 I²S OUT 04 P4 03 I²S MCLK 02 GND 01 TC:BUS"
- board text removed: "3V3 14 I²C DAT 13 I²S LRCK 12 I²S IN 11 I²S BCLK 10 VCC 09 TC:BUS 08"
- board text removed: "HP=47uF LN=1uF"
Changed lines of the file:
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@@
 	(footprint "Capacitor_SMD:C_0603_1608Metric"
 		(layer "F.Cu")
-		(at 190.29 84.3725)
+		(at 190.3 85.85)
 		(descr "Capacitor SMD 0603 (1608 Metric), square (rectangular) end terminal, IPC-7351 nominal, (Body size source: IPC-SM-782 page 76, https://www.pcb-3d.com/wordpress/wp-content/uploads/ipc-sm-782a_amendment_1_and_2.pdf), generated with kicad-footprint-generator")
 		(tags "capacitor")
@@
 	(footprint "Capacitor_SMD:C_0603_1608Metric"
 		(layer "F.Cu")
-		(at 190.29 85.8325)
+		(at 190.3 84.37)
 		(descr "Capacitor SMD 0603 (1608 Metric), square (rectangular) end terminal, IPC-7351 nominal, (Body size source: IPC-SM-782 page 76, https://www.pcb-3d.com/wordpress/wp-content/uploads/ipc-sm-782a_amendment_1_and_2.pdf), generated with kicad-footprint-generator")
 		(tags "capacitor")
@@
 		)
 	)
-	(gr_text "3V3 14\nI²C DAT 13\nI²S LRCK 12\nI²S IN 11\nI²S BCLK 10\nVCC 09\nTC:BUS 08"
+	(gr_text "LN"
+		(at 183.08 89.3 0)
+		(layer "B.SilkS")
+		(effects
+			(font
+				(size 0.8 0.8)
+				(thickness 0.2)
+				(bold yes)
+			)
+			(justify left bottom mirror)
+		)
+	)
+	(gr_text "TC:BUS 01\nGND 02\nI²S MCLK 03\nP4 04\nI²S OUT 05\nGND 06\nI²C CLK 07"
 		(at 190.92 93.1 0)
 		(layer "B.SilkS")
@@
 		)
 	)
-	(gr_text "07 I²C CLK\n06 GND\n05 I²S OUT\n04 P4\n03 I²S MCLK\n02 GND\n01 TC:BUS"
+	(gr_text "08 TC:BUS\n09 VCC\n10 I²S BCLK\n11 I²S IN\n12 I²S LRCK\n13 I²C DAT\n14 3V3"
 		(at 190.72 93.08 0)
 		(layer "B.SilkS")
@@
 		)
 	)
+	(gr_text "LN"
+		(at 183.08 86.65 0)
+		(layer "B.SilkS")
+		(effects
+			(font
+				(size 0.8 0.8)
+				(thickness 0.2)
+				(bold yes)
+			)
+			(justify left bottom mirror)
+		)
+	)
 	(gr_text "L2"
 		(at 203.99 86.71 0)
@@
 		)
 	)
-	(gr_text "HP=47uF\nLN=1uF"
+	(gr_text "HP 47uF\nLN 1uF"
 		(at 182.97 96.92 0)
 		(layer "B.SilkS")
@@
 	)
 	(via
+		(at 177.48 94.28)
+		(size 0.6)
+		(drill 0.3)
+		(layers "F.Cu" "B.Cu")
+		(free yes)
+		(net 1)
+	)
+	(via
 		(at 191.89 105.25)
 		(size 0.6)
@@
 	)
 	(via
+		(at 195.91 94.43)
+		(size 0.6)
+		(drill 0.3)
+		(layers "F.Cu" "B.Cu")
+		(free yes)
+		(net 1)
+	)
+	(via
 		(at 196.609977 83.112038)
 		(size 0.6)
@@
 	)
 	(via
-		(at 196.15 94.33)
+		(at 196.07 93.4)
 		(size 0.6)
 		(drill 0.3)
@@
 	)
 	(via
+		(at 181.32 89.57)
+		(size 0.6)
+		(drill 0.3)
+		(layers "F.Cu" "B.Cu")
+		(free yes)
+		(net 1)
+	)
+	(via
 		(at 189.45 91.7)
 		(size 0.6)
@@
 	)
 	(via
-		(at 181.94 86.59)
+		(at 181.42 86.64)
 		(size 0.6)
 		(drill 0.3)
@@
 	)
 	(via
-		(at 184.1 94.22)
+		(at 183.53 94.81)
 		(size 0.6)
 		(drill 0.3)
@@
 	)
 	(via
-		(at 181.96 88.09)
+		(at 181.31 88.07)
+		(size 0.6)
+		(drill 0.3)
+		(layers "F.Cu" "B.Cu")
+		(free yes)
+		(net 1)
+	)
+	(via
+		(at 178.72 94.26)
 		(size 0.6)
 		(drill 0.3)
@@
 	)
 	(segment
+		(start 190.8 86.77)
+		(end 190.8 88.18)
+		(width 0.6)
+		(layer "F.Cu")
+		(net 2)
+	)
+	(segment
 		(start 196.31 99.2)
 		(end 196.31 99.045)
@@
 	)
 	(segment
+		(start 191.08 84.3575)
+		(end 191.065 84.3725)
+		(width 0.6)
+		(layer "F.Cu")
+		(net 2)
+	)
+	(segment
+		(start 191.08 83.66)
+		(end 191.08 84.3575)
+		(width 0.6)
+		(layer "F.Cu")
+		(net 2)
+	)
+	(segment
 		(start 190.81 88.24)
 		(end 191 88.43)
@@
 	)
 	(segment
-		(start 191.08 84.3575)
-		(end 191.065 84.3725)
+		(start 191.08 85.8175)
+		(end 191.065 85.8325)
 		(width 0.6)
 		(layer "F.Cu")
@@
 	)
 	(segment
-		(start 191.07 85.8375)
-		(end 191.07 86.5)
+		(start 191.065 84.3725)
+		(end 191.075 84.3825)
 		(width 0.6)
 		(layer "F.Cu")
@@
 	)
 	(segment
-		(start 191.08 85.8175)
-		(end 191.065 85.8325)
+		(start 191.07 86.5)
+		(end 190.8 86.77)
 		(width 0.6)
 		(layer "F.Cu")
@@
 	)
 	(segment
-		(start 190.8 86.77)
-		(end 190.8 88.18)
-		(width 0.6)
+		(start 189.65 92.91)
+		(end 189.65 93.42)
+		(width 0.2)
 		(layer "F.Cu")
 		(net 2)
 	)
 	(segment
-		(start 189.65 92.91)
-		(end 189.65 93.42)
-		(width 0.2)
+		(start 191.075 85.8225)
+		(end 191.065 85.8325)
+		(width 0.6)
 		(layer "F.Cu")
 		(net 2)
@@
 	)
 	(segment
-		(start 191.07 85.8375)
-		(end 191.065 85.8325)
-		(width 0.6)
-		(layer "F.Cu")
-		(net 2)
-	)
-	(segment
 		(start 190.55 88.43)
 		(end 190.55 89.01)
@@
 	)
 	(segment
-		(start 191.07 86.5)
-		(end 190.8 86.77)
+		(start 191.075 84.3825)
+		(end 191.075 85.8225)
 		(width 0.6)
 		(layer "F.Cu")
@@
 	)
 	(segment
-		(start 191.08 83.66)
-		(end 191.08 84.3575)
-		(width 0.6)
-		(layer "F.Cu")
-		(net 2)
-	)
-	(segment
 		(start 189.2 92.91)
 		(end 189.2 93.43)
@@
 	)
 	(segment
-		(start 191.065 84.3725)
-		(end 191.065 85.8325)
+		(start 191.065 85.8325)
+		(end 191.07 85.8375)
 		(width 0.6)
 		(layer "F.Cu")
@@
 	)
 	(segment
+		(start 191.07 85.8375)
+		(end 191.07 86.5)
+		(width 0.6)
+		(layer "F.Cu")
+		(net 2)
+	)
+	(segment
 		(start 198.28 101.400001)
 		(end 198.28 100.47)
@@
 	)
 	(segment
-		(start 194.5025 91.7875)
-		(end 195.575 91.7875)
-		(width 0.2)
-		(layer "F.Cu")
-		(net 15)
-	)
-	(segment
-		(start 193.9775 92.3125)
-		(end 194.5025 91.7875)
+		(start 192.05 92.3125)
+		(end 195.05 92.3125)
 		(width 0.2)
 		(layer "F.Cu")
@@
 	)
 	(segment
-		(start 192.05 92.3125)
-		(end 193.9775 92.3125)
+		(start 195.05 92.3125)
+		(end 195.575 91.7875)
 		(width 0.2)
 		(layer "F.Cu")
@@
 	)
 	(segment
-		(start 193.555 101.18)
-		(end 194.547 101.18)
+		(start 192.31 102.425)
+		(end 193.555 101.18)
 		(width 0.2)
 		(layer "F.Cu")
@@
 	)
 	(segment
-		(start 192.31 103.215)
-		(end 192.31 102.425)
+		(start 195.28 96.25)
+		(end 197.225 94.305)
 		(width 0.2)
 		(layer "F.Cu")
@@
 	)
 	(segment
-		(start 192.31 102.425)
-		(end 193.555 101.18)
+		(start 197.225 94.305)
+		(end 197.225 91.7875)
 		(width 0.2)
 		(layer "F.Cu")
@@
 	)
 	(segment
-		(start 195.28 100.447)
-		(end 195.28 93.7325)
+		(start 192.31 103.215)
+		(end 192.31 102.425)
+		(width 0.2)
+		(layer "F.Cu")
+		(net 18)
+	)
+	(segment
+		(start 193.555 101.18)
+		(end 194.547 101.18)
 		(width 0.2)
 		(layer "F.Cu")
@@
 	)
 	(segment
-		(start 195.28 93.7325)
-		(end 197.225 91.7875)
+		(start 195.28 100.447)
+		(end 195.28 96.25)
 		(width 0.2)
 		(layer "F.Cu")

Commit message: WIP
Parts:
- R13, R14: footprint Resistor_SMD:R_0402_1005Metric -> Resistor_SMD:R_0603_1608Metric
- moved R13 1.69 mm to (198.5, 98.3)
- moved R14 0.71 mm to (198.5, 101.2)
Routing:
- net I2C_DAT: track 20.0 -> 20.7 mm

Commit message: WIP
Parts:
- J2: moved to B.Cu
- turned J2 to 0 degrees
Other:
- outline, holes or cut-outs redrawn

Commit message: WIP
Other:
- board text added: "08"
Changed lines of the file:
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@@
+		)
+	)
+	(gr_text "08"
+		(at 184.28 96.8 0)
+		(layer "F.SilkS")
+		(effects
+			(font
+				(size 0.8 0.8)
+				(thickness 0.2)
+			)
 		)
 	)
@@
 	)
 	(gr_text "14"
-		(at 196.3 97 0)
+		(at 196.29 96.92 0)
 		(layer "F.SilkS")
 		(effects

Commit message: WIP
Parts:
- added R7: 0, Resistor_SMD:R_0603_1608Metric, F.Cu at (91.5, 55.6)
- added R8: 0, Resistor_SMD:R_0603_1608Metric, F.Cu at (103.7, 52.6)
- C13, C7: value 47uF -> 1uF
- moved C13 98.9 mm to (103.0, 50.4)
- moved C2 98.9 mm to (97.7, 49.7)
- moved C20 98.9 mm to (90.8, 50.4)
- moved C5 98.9 mm to (91.5, 54.1)
- moved R15 98.9 mm to (93.8, 60.6)
- moved R17 98.9 mm to (101.1, 60.6)
- moved C10 98.9 mm to (96.7, 60.6)
- moved C12 98.9 mm to (87.6, 63.2)
- moved C14 98.9 mm to (95.3, 73.5)
- moved C7 98.9 mm to (100.6, 51.1)
- moved D1 98.9 mm to (86.5, 59.6)
- moved J2 98.9 mm to (85.1, 73.7)
- moved J5 98.9 mm to (85.1, 51.6)
- moved R13 98.9 mm to (105.9, 63.6)
- moved R14 98.9 mm to (105.9, 66.5)
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Connections:
- D2 pad 1: AUDIO_OUT_L1 -> Net-(D2-K)
- R6 pad 1: AUDIO_OUT_L1 -> Net-(D2-K)
- U1 pad 23: AUDIO_OUT_L1 -> Net-(U1-RIN1)
Routing:
- net Net-(D2-K): track 0.00 -> 27.9 mm, vias 0 -> 2
- net AUDIO_OUT_L1: track 42.2 -> 17.5 mm, vias 4 -> 2
- net Net-(U1-RIN1): track 0.00 -> 3.61 mm
- net Net-(D1-K): track 8.38 -> 6.85 mm
- net I2S_DAT_OUT: track 14.0 -> 12.6 mm
- net I2C_CLK: track 23.5 -> 22.5 mm
- net Net-(U1-CE): track 3.32 -> 4.08 mm
- net Net-(U1-ROUT1): track 4.48 -> 3.85 mm
- net AUDIO_OUT_R1: track 9.53 -> 8.92 mm
- net GND: vias 95 -> 92
- net AUDIO_OUT_R2: vias 1 -> 0
Other:
- board text added: "08 BUS 09 VCC 10 I²S BCLK 11 I²S DIN 12 I²S LRCK 13 I²C DAT 14 3V3"
- board text added: "BUS 01 GND 02 I²S MCLK 03 P4 04 I²S DOUT 05 GND 06 I²C CLK 07"
- board text removed: "08 TC:BUS 09 VCC 10 I²S BCLK 11 I²S IN 12 I²S LRCK 13 I²C DAT 14 3V3"
- board text removed: "HP"
- board text removed: "HP 47uF LN 1uF"
- board text removed: "LN"
- board text removed: "TC:BUS 01 GND 02 I²S MCLK 03 P4 04 I²S OUT 05 GND 06 I²C CLK 07"

Commit message: WIP
Parts:
- removed C6: 1uF, Capacitor_SMD:C_0603_1608Metric
- removed R1: 10, Resistor_SMD:R_0603_1608Metric
- added C4: 10uF, Capacitor_SMD:C_1206_3216Metric, F.Cu at (88.9, 63.6)
- added C8: 10uF, Capacitor_SMD:C_1206_3216Metric, F.Cu at (95.3, 75.0)
- added D3: CDSOD323-T03S, Diode_SMD:D_SOD-323, F.Cu at (85.6, 60.4)
- added D4: CDSOD323-T03S, Diode_SMD:D_SOD-323, F.Cu at (107.4, 55.5)
- added R10: 200, Resistor_SMD:R_1206_3216Metric, F.Cu at (99.8, 75.0)
- added R9: 0, Resistor_SMD:R_0603_1608Metric, F.Cu at (103.8, 55.6)
- J1: footprint Connector_PinHeader_2.54mm:PinHeader_1x04_P2.54mm_Vertical -> Connector_PinHeader_2.54mm:PinHeader_1x03_P2.54mm_Vertical
- moved D1 3.60 mm to (90.0, 60.3), turned to 0 degrees
- moved R4 1.47 mm to (91.5, 55.6)
- moved R7 1.46 mm to (91.5, 57.0)
- moved C12 1.03 mm to (86.6, 63.6)
- moved C14 0.77 mm to (95.3, 72.8)
- moved R6 0.76 mm to (99.8, 72.8)
- moved R8 0.72 mm to (103.7, 53.4)
- moved D2 0.70 mm to (107.4, 53.3)
Connections:
- C12 pad 2: Net-(D1-K) -> Net-(D3-K)
- J1 pad 3: AUDIO_OUT_R1 -> GND
- R4 pad 1: AUDIO_IN_L1 -> AUDIO_IN_R1
- R4 pad 2: Net-(D1-K) -> Net-(D3-K)
- R6 pad 1: Net-(D2-K) -> Net-(D4-K)
- R7 pad 1: Net-(U1-RIN1) -> AUDIO_IN_L1
- R7 pad 2: AUDIO_OUT_L1 -> Net-(D1-K)
- U1 pad 11: Net-(U1-ROUT1) -> AUDIO_OUT_R1
- U1 pad 23: Net-(U1-RIN1) -> AUDIO_IN_R1
Routing:
- net Net-(D4-K): track 0.00 -> 23.2 mm, vias 0 -> 2
- net BUS_WIRE1: track 0.00 -> 18.3 mm, vias 0 -> 2
- net AUDIO_OUT_L1: track 17.5 -> 4.51 mm, vias 2 -> 0
- net Net-(D3-K): track 0.00 -> 9.52 mm
- net AUDIO_OUT_R1: track 8.92 -> 3.79 mm
- net Net-(U1-ROUT1): track 3.85 -> 0.00 mm
- net Net-(U1-RIN1): track 3.61 -> 0.00 mm
- net AUDIO_IN_R1: track 0.00 -> 3.26 mm
- net Net-(D2-K): track 27.9 -> 30.4 mm
- net VCC: track 12.5 -> 14.3 mm
- net Net-(C8-Pad2): track 0.00 -> 1.64 mm
- net Net-(C6-Pad2): track 1.48 -> 0.00 mm
- net GND: vias 92 -> 102
Other:
- board text removed: "R1"
