File: pcb_extension_audio/doorman_audio_extension.kicad_sch (KiCad schematic)
At the start: 37 parts, among them J1 Audio Out, J4 Conn_02x07_Odd_Even, J5 Audio In, U1 ES8388

Commit message: WIP
Parts:
- J4: value Conn_02x07_Odd_Even -> Extension Board Connector
Connections:
- net AUDIO_IN_R1: now also J5.3 (Pin_3); no longer J5.1 (Pin_1)
- net AUDIO_IN_R2: now also J5.1 (Pin_1); no longer J5.3 (Pin_3)
Other:
- note added: "CONNECTORS"
- note removed: "Extension Board Connector"
Changed lines of the file:
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@@
 		)
 	)
-	(text "LINE OUT"
+	(text "CONNECTORS"
 		(exclude_from_sim no)
-		(at 166.116 82.804 0)
+		(at 195.834 108.966 0)
 		(effects
 			(font
-				(size 1 1)
+				(size 3 3)
 			)
+			(justify left bottom)
 		)
 	)
-	(text "LINE IN"
+	(text "LINE OUT"
 		(exclude_from_sim no)
-		(at 164.338 75.184 0)
+		(at 166.116 82.804 0)
 		(effects
 			(font
@@
 		)
 	)
-	(text "Extension Board Connector"
+	(text "LINE IN"
 		(exclude_from_sim no)
-		(at 220.218 107.696 0)
+		(at 164.338 75.184 0)
 		(effects
 			(font
-				(size 1.27 1.27)
+				(size 1 1)
 			)
-			(justify left bottom)
 		)
 	)
@@
 		)
 	)
-	(global_label "AUDIO_IN_R2"
-		(shape input)
-		(at 215.9 154.94 0)
-		(fields_autoplaced yes)
-		(effects
-			(font
-				(size 1.27 1.27)
-			)
-			(justify left)
-		)
-		(property "Intersheetrefs" "${INTERSHEET_REFS}"
-			(at 230.8596 154.94 0)
-			(effects
-				(font
-					(size 1.27 1.27)
-				)
-				(justify left)
-				(hide yes)
-			)
-		)
-	)
 	(global_label "AUDIO_OUT_R1"
 		(shape input)
@@
 		)
 	)
+	(global_label "AUDIO_IN_R2"
+		(shape input)
+		(at 215.9 149.86 0)
+		(fields_autoplaced yes)
+		(effects
+			(font
+				(size 1.27 1.27)
+			)
+			(justify left)
+		)
+		(property "Intersheetrefs" "${INTERSHEET_REFS}"
+			(at 230.8596 149.86 0)
+			(effects
+				(font
+					(size 1.27 1.27)
+				)
+				(justify left)
+				(hide yes)
+			)
+		)
+	)
 	(global_label "AUDIO_OUT_L1"
 		(shape input)
@@
 	(global_label "AUDIO_IN_R1"
 		(shape input)
-		(at 215.9 149.86 0)
+		(at 215.9 154.94 0)
 		(fields_autoplaced yes)
 		(effects
@@
 		)
 		(property "Intersheetrefs" "${INTERSHEET_REFS}"
-			(at 230.8596 149.86 0)
+			(at 230.8596 154.94 0)
 			(effects
 				(font
@@
 			)
 		)
-		(property "Value" "Conn_02x07_Odd_Even"
+		(property "Value" "Extension Board Connector"
 			(at 232.41 113.03 0)
 			(effects

Commit message: WIP
Parts:
- removed R20, R21: 10K, Resistor_SMD:R_0603_1608Metric, symbol Device:R
- R6: value 1K -> 200
Other:
- note added: "VMIDSEL = 10 (default) 500 kΩ divider enabled"
- moved on the sheet: C1, C10, C11, C12, C13, C14, C17, C18, C19, C2, C20, C21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

Commit message: WIP
Parts:
- C12, C14: value 1uF -> 10uF; LCSC C1848 -> C89632; MPN CL31B105KBHNNNE -> CL31B106KBHNNNE
- C13, C3, C4, C5, C6, C7, R1, R2, R3: now fitted
Changed lines of the file:
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@@
 		(in_bom yes)
 		(on_board yes)
-		(dnp yes)
+		(dnp no)
 		(property "Reference" "R2"
 			(at 148.59 78.994 90)
@@
 		(in_bom yes)
 		(on_board yes)
-		(dnp yes)
+		(dnp no)
 		(property "Reference" "C3"
 			(at 141.224 69.088 90)
@@
 		(in_bom yes)
 		(on_board yes)
-		(dnp yes)
+		(dnp no)
 		(property "Reference" "C5"
 			(at 136.398 66.548 90)
@@
 		(in_bom yes)
 		(on_board yes)
-		(dnp yes)
+		(dnp no)
 		(property "Reference" "R1"
 			(at 148.59 76.454 90)
@@
 			)
 		)
-		(property "Value" "1uF"
+		(property "Value" "10uF"
 			(at 250.19 67.818 90)
 			(effects
@@
 			)
 		)
-		(property "Description" "1uF 50V X7R ±10% 1206 Multilayer Ceramic Capacitors MLCC - SMD/SMT ROHS"
+		(property "Description" "10uF 50V X7R ±10% 1206 Multilayer Ceramic Capacitors MLCC - SMD/SMT ROHS"
 			(at 251.46 71.12 0)
 			(effects
@@
 			)
 		)
-		(property "LCSC" "C1848"
+		(property "LCSC" "C89632"
 			(at 251.46 71.12 0)
 			(effects
@@
 			)
 		)
-		(property "MPN" "CL31B105KBHNNNE"
+		(property "MPN" "CL31B106KBHNNNE"
 			(at 251.46 71.12 0)
 			(effects
@@
 			)
 		)
-		(property "Value" "1uF"
+		(property "Value" "10uF"
 			(at 250.19 36.068 90)
 			(effects
@@
 			)
 		)
-		(property "Description" "1uF 50V X7R ±10% 1206 Multilayer Ceramic Capacitors MLCC - SMD/SMT ROHS"
+		(property "Description" "10uF 50V X7R ±10% 1206 Multilayer Ceramic Capacitors MLCC - SMD/SMT ROHS"
 			(at 251.46 39.37 0)
 			(effects
@@
 			)
 		)
-		(property "LCSC" "C1848"
+		(property "LCSC" "C89632"
 			(at 251.46 39.37 0)
 			(effects
@@
 			)
 		)
-		(property "MPN" "CL31B105KBHNNNE"
+		(property "MPN" "CL31B106KBHNNNE"
 			(at 251.46 39.37 0)
 			(effects
@@
 		(in_bom yes)
 		(on_board yes)
-		(dnp yes)
+		(dnp no)
 		(property "Reference" "C13"
 			(at 134.62 81.534 90)
@@
 		(in_bom yes)
 		(on_board yes)
-		(dnp yes)
+		(dnp no)
 		(property "Reference" "C7"
 			(at 138.938 79.248 90)
@@
 		(in_bom yes)
 		(on_board yes)
-		(dnp yes)
+		(dnp no)
 		(property "Reference" "C6"
 			(at 133.858 76.708 90)
@@
 		(in_bom yes)
 		(on_board yes)
-		(dnp yes)
+		(dnp no)
 		(property "Reference" "C4"
 			(at 141.224 63.754 90)
@@
 		(in_bom yes)
 		(on_board yes)
-		(dnp yes)
+		(dnp no)
 		(property "Reference" "R3"
 			(at 148.59 81.534 90)

Commit message: WIP
Parts:
- removed C4: 1uF, Capacitor_SMD:C_0603_1608Metric, symbol Device:C_Small
- J5: footprint Connector_PinHeader_2.54mm:PinHeader_1x03_P2.54mm_Vertical -> Connector_PinHeader_2.54mm:PinHeader_1x02_P2.54mm_Vertical; symbol Connector:Conn_01x03_Pin -> Connector:Conn_01x02_Pin
Connections:
- net AUDIO_OUT_L1: now also U1.23 (RIN1)
- removed net AUDIO_IN_R1: J5.3 (Pin_3)
Other:
- note added: "Difference (L1 OUT)"
Changed lines of the file:
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@@
 		)
 	)
+	(text "Difference (L1 OUT)"
+		(exclude_from_sim no)
+		(at 175.26 65.024 0)
+		(effects
+			(font
+				(size 1 1)
+			)
+		)
+	)
 	(text "HP Out"
 		(exclude_from_sim no)
@@
 		)
 	)
-	(text "LINE IN"
-		(exclude_from_sim no)
-		(at 169.418 65.024 0)
-		(effects
-			(font
-				(size 1 1)
-			)
-		)
-	)
 	(text "CONNECTORS"
 		(exclude_from_sim no)
@@
 	(wire
 		(pts
-			(xy 140.97 64.77) (xy 151.13 64.77)
-		)
-		(stroke
-			(width 0)
-			(type default)
-		)
-	)
-	(wire
-		(pts
 			(xy 106.68 100.33) (xy 106.68 102.87)
 		)
@@
 		)
 	)
-	(wire
-		(pts
-			(xy 127 64.77) (xy 135.89 64.77)
-		)
-		(stroke
-			(width 0)
-			(type default)
-		)
-	)
 	(polyline
 		(pts
@@
 	(wire
 		(pts
+			(xy 151.13 64.77) (xy 127 64.77)
+		)
+		(stroke
+			(width 0)
+			(type default)
+		)
+	)
+	(wire
+		(pts
 			(xy 101.6 39.37) (xy 101.6 38.1)
 		)
@@
 		)
 	)
-	(global_label "AUDIO_OUT_R2"
+	(global_label "AUDIO_OUT_L1"
 		(shape input)
-		(at 151.13 82.55 0)
+		(at 151.13 64.77 0)
 		(fields_autoplaced yes)
 		(effects
@@
 		)
 		(property "Intersheetrefs" "${INTERSHEET_REFS}"
-			(at 167.7829 82.55 0)
+			(at 167.541 64.77 0)
 			(effects
 				(font
@@
 		)
 	)
-	(global_label "AUDIO_IN_R2"
+	(global_label "AUDIO_OUT_R2"
 		(shape input)
-		(at 151.13 69.85 0)
+		(at 151.13 82.55 0)
 		(fields_autoplaced yes)
 		(effects
@@
 		)
 		(property "Intersheetrefs" "${INTERSHEET_REFS}"
-			(at 166.0896 69.85 0)
+			(at 167.7829 82.55 0)
 			(effects
 				(font
@@
 		)
 	)
-	(global_label "AUDIO_IN_L2"
+	(global_label "AUDIO_IN_R2"
 		(shape input)
-		(at 215.9 152.4 0)
+		(at 151.13 69.85 0)
 		(fields_autoplaced yes)
 		(effects
@@
 		)
 		(property "Intersheetrefs" "${INTERSHEET_REFS}"
-			(at 230.6177 152.4 0)
+			(at 166.0896 69.85 0)
 			(effects
 				(font
@@
 		)
 	)
-	(global_label "AUDIO_IN_R1"
+	(global_label "AUDIO_IN_L2"
 		(shape input)
-		(at 151.13 64.77 0)
+		(at 215.9 154.94 0)
 		(fields_autoplaced yes)
 		(effects
@@
 		)
 		(property "Intersheetrefs" "${INTERSHEET_REFS}"
-			(at 166.0896 64.77 0)
+			(at 230.6177 154.94 0)
 			(effects
 				(font
@@
 	(global_label "AUDIO_IN_R2"
 		(shape input)
-		(at 215.9 149.86 0)
+		(at 215.9 152.4 0)
 		(fields_autoplaced yes)
 		(effects
@@
 		)
 		(property "Intersheetrefs" "${INTERSHEET_REFS}"
-			(at 230.8596 149.86 0)
+			(at 230.8596 152.4 0)
 			(effects
 				(font
@@
 		)
 	)
-	(global_label "AUDIO_IN_R1"
-		(shape input)
-		(at 215.9 154.94 0)
-		(fields_autoplaced yes)
-		(effects
-			(font
-				(size 1.27 1.27)
-			)
-			(justify left)
-		)
-		(property "Intersheetrefs" "${INTERSHEET_REFS}"
-			(at 230.8596 154.94 0)
-			(effects
-				(font
-					(size 1.27 1.27)
-				)
-				(justify left)
-				(hide yes)
-			)
-		)
-	)
 	(global_label "I2S_SCLK"
 		(shape input)
@@
 	)
 	(symbol
-		(lib_id "Connector:Conn_01x03_Pin")
+		(lib_id "Connector:Conn_01x02_Pin")
 		(at 210.82 152.4 0)
 		(unit 1)
@@
 		(fields_autoplaced yes)
 		(property "Reference" "J5"
-			(at 211.455 144.78 0)
+			(at 211.455 147.32 0)
 			(effects
 				(font
@@
 		)
 		(property "Value" "Audio In"
-			(at 211.455 147.32 0)
+			(at 211.455 149.86 0)
 			(effects
 				(font
@@
 			)
 		)
-		(property "Footprint" "Connector_PinHeader_2.54mm:PinHeader_1x03_P2.54mm_Vertical"
+		(property "Footprint" "Connector_PinHeader_2.54mm:PinHeader_1x02_P2.54mm_Vertical"
 			(at 210.82 152.4 0)
 			(effects
@@
 			)
 		)
-		(property "Description" "Generic connector, single row, 01x03, script generated"
+		(property "Description" "Generic connector, single row, 01x02, script generated"
 			(at 210.82 152.4 0)
 			(effects
@@
 		(pin "2"
 		)
-		(pin "3"
-		)
 		(instances
 			(project "doorman"
@@
 					(unit 1)
 				)
-			)
-		)
-	)
-	(symbol
-		(lib_id "Device:C_Small")
-		(at 138.43 64.77 90)
-		(unit 1)
-		(exclude_from_sim no)
-		(in_bom yes)
-		(on_board yes)
-		(dnp no)
-		(property "Reference" "C4"
-			(at 141.224 63.754 90)
-			(effects
-				(font
-					(size 1 1)
-				)
-				(justify left)
-			)
-		)
-		(property "Value" "1uF"
-			(at 141.478 65.532 90)
-			(effects
-				(font
-					(size 0.8 0.8)
-				)
-				(justify left)
-			)
-		)
-		(property "Footprint" "Capacitor_SMD:C_0603_1608Metric"
-			(at 138.43 64.77 0)
-			(effects
-				(font
-					(size 1.27 1.27)
-				)
-				(hide yes)
-			)
-		)
-		(property "Datasheet" ""
-			(at 138.43 64.77 0)
-			(effects
-				(font
-					(size 1.27 1.27)
-				)
-				(hide yes)
-			)
-		)
-		(property "Description" "1uF 50V X5R ±10% 0603 Multilayer Ceramic Capacitors MLCC - SMD/SMT ROHS"
-			(at 138.43 64.77 0)
-			(effects
-				(font
-					(size 1.27 1.27)
-				)
-				(hide yes)
-			)
-		)
-		(property "LCSC" "C15849"
-			(at 138.43 64.77 0)
-			(effects
-				(font
-					(size 1.27 1.27)
-				)
-				(hide yes)
-			)
-		)
-		(property "MPN" "CL10A105KB8NNNC"
-			(at 138.43 64.77 0)
-			(effects
-				(font
-					(size 1.27 1.27)
-				)
-				(hide yes)
-			)
-		)
-		(property "Height" ""
-			(at 138.43 64.77 0)
-			(effects
-				(font
-					(size 1.27 1.27)
-				)
-				(hide yes)
-			)
-		)
-		(property "Mouser Part Number" ""
-			(at 138.43 64.77 0)
-			(effects
-				(font
-					(size 1.27 1.27)
-				)
-				(hide yes)
-			)
-		)
-		(property "Mouser Price/Stock" ""
-			(at 138.43 64.77 0)
-			(effects
-				(font
-					(size 1.27 1.27)
-				)
-				(hide yes)
-			)
-		)
-		(property "Package" "0603"
-			(at 138.43 64.77 90)
-			(effects
-				(font
-					(size 1.27 1.27)
-				)
-				(hide yes)
-			)
-		)
-		(property "Price" ""
-			(at 138.43 64.77 0)
-			(effects
-				(font
-					(size 1.27 1.27)
-				)
-				(hide yes)
-			)
-		)
-		(property "Cheap Version" ""
-			(at 138.43 64.77 90)
-			(effects
-				(font
-					(size 1.27 1.27)
-				)
-				(hide yes)
-			)
-		)
-		(property "Expensive Version" ""
-			(at 138.43 64.77 90)
-			(effects
-				(font
-					(size 1.27 1.27)
-				)
-				(hide yes)
-			)
-		)
-		(property "LCSC Part" ""
-			(at 138.43 64.77 90)
-			(effects
-				(font
-					(size 1.27 1.27)
-				)
-				(hide yes)
-			)
-		)
-		(property "Manufacturer_Name" ""
-			(at 138.43 64.77 90)
-			(effects
-				(font
-					(size 1.27 1.27)
-				)
-				(hide yes)
-			)
-		)
-		(property "Manufacturer_Part_Number" ""
-			(at 138.43 64.77 90)
-			(effects
-				(font
-					(size 1.27 1.27)
-				)
-				(hide yes)
-			)
-		)
-		(pin "1"
-		)
-		(pin "2"
-		)
-		(instances
-			(project "doorman"
-				(path "/2048a046-8e00-475d-aeec-41a343368725"
-					(reference "C4")
-					(unit 1)
-				)

Commit message: WIP
Connections:
- net I2S_SCLK renamed I2S_BCLK
Changed lines of the file:
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@@
 		)
 	)
-	(global_label "I2S_SCLK"
+	(global_label "I2S_BCLK"
 		(shape input)
 		(at 68.58 46.99 90)
@@
 		)
 		(property "Intersheetrefs" "${INTERSHEET_REFS}"
-			(at 68.58 35.2358 90)
+			(at 68.58 35.1753 90)
 			(effects
 				(font
@@
 		)
 	)
-	(global_label "I2S_SCLK"
+	(global_label "I2S_BCLK"
 		(shape input)
 		(at 238.76 124.46 0)
@@
 		)
 		(property "Intersheetrefs" "${INTERSHEET_REFS}"
-			(at 249.3652 124.46 0)
+			(at 250.5747 124.46 0)
 			(effects
 				(font

Commit message: WIP
Parts:
- added U2: ES8388, Package_DFN_QFN:QFN-28-1EP_4x4mm_P0.45mm_EP2.6x2.6mm, symbol Audio:ES8388
- J4: symbol Connector_Generic:Conn_02x07_Odd_Even -> Connector_Generic:Conn_02x07_Top_Bottom
Connections:
- net BUS_WIRE1: now also J4.8 (Pin_8); no longer J4.2 (Pin_2)
- net GND: now also J4.2 (Pin_2), J4.6 (Pin_6), U2.29 (EPAD); no longer J4.11 (Pin_11), J4.3 (Pin_3)
- net I2C_CLK: now also J4.7 (Pin_7); no longer J4.13 (Pin_13)
- net I2C_DAT: now also J4.13 (Pin_13); no longer J4.12 (Pin_12)
- net I2S_BCLK: now also J4.4 (Pin_4); no longer J4.7 (Pin_7)
- net I2S_DAT_IN: now also J4.11 (Pin_11); no longer J4.8 (Pin_8)
- net I2S_DAT_OUT: now also J4.5 (Pin_5); no longer J4.9 (Pin_9)
- net I2S_LRCK: now also J4.12 (Pin_12); no longer J4.10 (Pin_10)
- net I2S_MCLK: now also J4.10 (Pin_10); no longer J4.6 (Pin_6)

Commit message: WIP
Parts:
- removed U2: ES8388, Package_DFN_QFN:QFN-28-1EP_4x4mm_P0.45mm_EP2.6x2.6mm, symbol Audio:ES8388

Commit message: WIP
Parts:
- added J2: GPIO, Connector_PinHeader_2.54mm:PinHeader_1x02_P2.54mm_Vertical, symbol Connector:Conn_01x02_Pin
Connections:
- net PIN3: now reaches J4.3 (Pin_3)
- net PIN3: now also J2.1 (Pin_1)
- net PIN9: now reaches J4.9 (Pin_9)
- net PIN9: now also J2.2 (Pin_2)
- no-connect marks 2 -> 0
Other:
- note added: "Free GPIOS"
- moved on the sheet: J1, J5
