File: pcb_extension_audio/doorman_audio_extension.kicad_sch (KiCad schematic)
At the start: 35 parts, among them J1 Audio Out, J2 GPIO, J4 Extension Board Connector, J5 Audio In, U1 ES8388

Commit message: WIP
Parts:
- added R4: 0, Resistor_SMD:R_0603_1608Metric, symbol Device:R
Connections:
- net PIN9 is gone; now on net VCC: J2.2 (Pin_2), J4.9 (Pin_9)
- net AUDIO_IN_L1: now also R4.1; no longer C12.2, D1.1 (K)
- net I2S_BCLK: now also J4.11 (Pin_11); no longer J4.4 (Pin_4)
- net I2S_DAT_IN: now also J4.4 (Pin_4); no longer J4.11 (Pin_11)
- new net: C12.2, D1.1 (K), R4.2
Changed lines of the file:
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@@
 	(text "VMIDSEL = 10 (default)\n500 kΩ divider enabled"
 		(exclude_from_sim no)
-		(at 222.504 37.338 0)
+		(at 221.488 35.814 0)
 		(effects
 			(font
@@
 	(wire
 		(pts
+			(xy 227.33 39.37) (xy 229.87 39.37)
+		)
+		(stroke
+			(width 0)
+			(type default)
+		)
+	)
+	(wire
+		(pts
 			(xy 55.88 87.63) (xy 55.88 93.98)
 		)
@@
 	(wire
 		(pts
-			(xy 218.44 39.37) (xy 229.87 39.37)
+			(xy 218.44 39.37) (xy 219.71 39.37)
 		)
 		(stroke
@@
 		)
 	)
-	(global_label "I2S_MCLK"
+	(global_label "PIN3"
 		(shape input)
-		(at 226.06 127 180)
+		(at 238.76 127 0)
 		(fields_autoplaced yes)
 		(effects
@@
 				(size 1.27 1.27)
 			)
-			(justify right)
+			(justify left)
 		)
 		(property "Intersheetrefs" "${INTERSHEET_REFS}"
-			(at 215.4548 127 0)
+			(at 247.3695 127 0)
 			(effects
 				(font
 					(size 1.27 1.27)
 				)
-				(justify right)
+				(justify left)
 				(hide yes)
 			)
@@
 		)
 	)
-	(global_label "AUDIO_IN_L1"
+	(global_label "VCC"
 		(shape input)
-		(at 218.44 39.37 180)
+		(at 226.06 129.54 180)
 		(fields_autoplaced yes)
 		(effects
@@
 		)
 		(property "Intersheetrefs" "${INTERSHEET_REFS}"
-			(at 203.7223 39.37 0)
+			(at 219.4462 129.54 0)
 			(effects
 				(font
@@
 		)
 	)
-	(global_label "I2S_BCLK"
+	(global_label "AUDIO_IN_L1"
 		(shape input)
-		(at 68.58 46.99 90)
+		(at 218.44 39.37 180)
 		(fields_autoplaced yes)
 		(effects
@@
 				(size 1.27 1.27)
 			)
-			(justify left)
+			(justify right)
 		)
 		(property "Intersheetrefs" "${INTERSHEET_REFS}"
-			(at 68.58 35.1753 90)
+			(at 203.7223 39.37 0)
 			(effects
 				(font
 					(size 1.27 1.27)
 				)
-				(justify left)
+				(justify right)
 				(hide yes)
 			)
 		)
 	)
-	(global_label "I2S_DAT_IN"
+	(global_label "I2S_BCLK"
 		(shape input)
-		(at 226.06 124.46 180)
+		(at 68.58 46.99 90)
 		(fields_autoplaced yes)
 		(effects
@@
 				(size 1.27 1.27)
 			)
-			(justify right)
+			(justify left)
 		)
 		(property "Intersheetrefs" "${INTERSHEET_REFS}"
-			(at 215.4548 124.46 0)
+			(at 68.58 35.1753 90)
 			(effects
 				(font
 					(size 1.27 1.27)
 				)
-				(justify right)
+				(justify left)
 				(hide yes)
 			)
@@
 		)
 		(property "Intersheetrefs" "${INTERSHEET_REFS}"
-			(at 223.2396 152.4 0)
+			(at 215.68 152.4 0)
 			(effects
 				(font
@@
 		)
 	)
-	(global_label "I2S_BCLK"
+	(global_label "I2S_DAT_IN"
 		(shape input)
 		(at 238.76 124.46 0)
@@
 		)
 		(property "Intersheetrefs" "${INTERSHEET_REFS}"
-			(at 250.5747 124.46 0)
+			(at 251.9657 124.46 0)
 			(effects
 				(font
@@
 		)
 	)
-	(global_label "PIN9"
-		(shape input)
-		(at 226.06 129.54 180)
-		(fields_autoplaced yes)
-		(effects
-			(font
-				(size 1.27 1.27)
-			)
-			(justify right)
-		)
-		(property "Intersheetrefs" "${INTERSHEET_REFS}"
-			(at 218.66 129.54 0)
-			(effects
-				(font
-					(size 1.27 1.27)
-				)
-				(justify right)
-				(hide yes)
-			)
-		)
-	)
 	(global_label "AUDIO_OUT_R2"
 		(shape input)
@@
 		)
 	)
-	(global_label "PIN3"
+	(global_label "I2S_BCLK"
 		(shape input)
-		(at 238.76 127 0)
+		(at 226.06 124.46 180)
 		(fields_autoplaced yes)
 		(effects
@@
 				(size 1.27 1.27)
 			)
-			(justify left)
+			(justify right)
 		)
 		(property "Intersheetrefs" "${INTERSHEET_REFS}"
-			(at 246.16 127 0)
+			(at 214.2453 124.46 0)
 			(effects
 				(font
 					(size 1.27 1.27)
 				)
-				(justify left)
+				(justify right)
 				(hide yes)
 			)
@@
 		)
 	)
+	(global_label "I2S_MCLK"
+		(shape input)
+		(at 226.06 127 180)
+		(fields_autoplaced yes)
+		(effects
+			(font
+				(size 1.27 1.27)
+			)
+			(justify right)
+		)
+		(property "Intersheetrefs" "${INTERSHEET_REFS}"
+			(at 214.0639 127 0)
+			(effects
+				(font
+					(size 1.27 1.27)
+				)
+				(justify right)
+				(hide yes)
+			)
+		)
+	)
 	(global_label "AUDIO_OUT_R1"
 		(shape input)
@@
 		)
 	)
-	(global_label "PIN9"
+	(global_label "VCC"
 		(shape input)
 		(at 208.28 154.94 0)
@@
 		)
 		(property "Intersheetrefs" "${INTERSHEET_REFS}"
-			(at 222.9977 154.94 0)
+			(at 214.8938 154.94 0)
 			(effects
 				(font
@@
 					(unit 1)
 				)
+			)
+		)
+	)
+	(symbol
+		(lib_id "Device:R")
+		(at 223.52 39.37 90)
+		(unit 1)
+		(exclude_from_sim no)
+		(in_bom yes)
+		(on_board yes)
+		(dnp no)
+		(property "Reference" "R4"
+			(at 223.52 36.83 90)
+			(effects
+				(font
+					(size 1 1)
+				)
+			)
+		)
+		(property "Value" "0"
+			(at 223.52 39.37 90)
+			(effects
+				(font
+					(size 1 1)
+				)
+			)
+		)
+		(property "Footprint" "Resistor_SMD:R_0603_1608Metric"
+			(at 223.52 41.148 90)
+			(effects
+				(font
+					(size 1.27 1.27)
+				)
+				(hide yes)
+			)
+		)
+		(property "Datasheet" "https://datasheet.lcsc.com/lcsc/2206010045_UNI-ROYAL-Uniroyal-Elec-0402WGF5101TCE_C25905.pdf"
+			(at 223.52 39.37 0)
+			(effects
+				(font
+					(size 1.27 1.27)
+				)
+				(hide yes)
+			)
+		)
+		(property "Description" "-55℃~+155℃ 0Ω 100mW 75V Thick Film Resistor ±1% 0603 Chip Resistor - Surface Mount ROHS"
+			(at 223.52 39.37 0)
+			(effects
+				(font
+					(size 1.27 1.27)
+				)
+				(hide yes)
+			)
+		)
+		(property "LCSC" "C21189"
+			(at 223.52 39.37 90)
+			(effects
+				(font
+					(size 1.27 1.27)
+				)
+				(hide yes)
+			)
+		)
+		(property "MPN" "0603WAF0000T5E"
+			(at 223.52 39.37 90)
+			(effects
+				(font
+					(size 1.27 1.27)
+				)
+				(hide yes)
+			)
+		)
+		(property "Height" ""
+			(at 223.52 39.37 0)
+			(effects
+				(font
+					(size 1.27 1.27)
+				)
+				(hide yes)
+			)
+		)
+		(property "Mouser Part Number" ""
+			(at 223.52 39.37 0)
+			(effects
+				(font
+					(size 1.27 1.27)
+				)
+				(hide yes)
+			)
+		)
+		(property "Mouser Price/Stock" ""
+			(at 223.52 39.37 0)
+			(effects
+				(font
+					(size 1.27 1.27)
+				)
+				(hide yes)
+			)
+		)
+		(property "Package" "0603"
+			(at 223.52 39.37 90)
+			(effects
+				(font
+					(size 1.27 1.27)
+				)
+				(hide yes)
+			)
+		)
+		(property "Price" ""
+			(at 223.52 39.37 0)
+			(effects
+				(font
+					(size 1.27 1.27)
+				)
+				(hide yes)
+			)
+		)
+		(property "Cheap Version" ""
+			(at 223.52 39.37 90)
+			(effects
+				(font
+					(size 1.27 1.27)
+				)
+				(hide yes)
+			)
+		)
+		(property "Expensive Version" ""
+			(at 223.52 39.37 90)
+			(effects
+				(font
+					(size 1.27 1.27)
+				)
+				(hide yes)
+			)
+		)
+		(property "LCSC Part" ""
+			(at 223.52 39.37 90)
+			(effects
+				(font
+					(size 1.27 1.27)
+				)
+				(hide yes)
+			)
+		)
+		(property "Manufacturer_Name" ""
+			(at 223.52 39.37 90)
+			(effects
+				(font
+					(size 1.27 1.27)
+				)
+				(hide yes)
+			)
+		)
+		(property "Manufacturer_Part_Number" ""
+			(at 223.52 39.37 90)
+			(effects
+				(font
+					(size 1.27 1.27)
+				)
+				(hide yes)
+			)
+		)
+		(pin "1"
+		)
+		(pin "2"
+		)
+		(instances
+			(project "doorman_audio_extension"
+				(path "/2048a046-8e00-475d-aeec-41a343368725"
+					(reference "R4")
+					(unit 1)
+				)

Commit message: WIP
Parts:
- J1: footprint Connector_PinHeader_2.54mm:PinHeader_1x03_P2.54mm_Vertical -> Connector_PinHeader_2.54mm:PinHeader_1x04_P2.54mm_Vertical; symbol Connector:Conn_01x03_Pin -> Connector:Conn_01x04_Pin
- J5: footprint Connector_PinHeader_2.54mm:PinHeader_1x02_P2.54mm_Vertical -> Connector_PinHeader_2.54mm:PinHeader_1x03_P2.54mm_Vertical; symbol Connector:Conn_01x02_Pin -> Connector:Conn_01x03_Pin
Connections:
- net GND: now also J1.4 (Pin_4), J5.3 (Pin_3)
Other:
- moved on the sheet: J2

Commit message: WIP
Changed lines of the file:
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@@
 	(wire
 		(pts
+			(xy 207.01 129.54) (xy 226.06 129.54)
+		)
+		(stroke
+			(width 0)
+			(type default)
+		)
+	)
+	(wire
+		(pts
 			(xy 219.71 71.12) (xy 229.87 71.12)
 		)
@@
 	(wire
 		(pts
+			(xy 213.36 152.4) (xy 208.28 152.4)
+		)
+		(stroke
+			(width 0)
+			(type default)
+		)
+	)
+	(wire
+		(pts
 			(xy 62.23 55.88) (xy 62.23 67.31)
 		)
@@
 		)
 	)
-	(global_label "VCC"
-		(shape input)
-		(at 226.06 129.54 180)
-		(fields_autoplaced yes)
-		(effects
-			(font
-				(size 1.27 1.27)
-			)
-			(justify right)
-		)
-		(property "Intersheetrefs" "${INTERSHEET_REFS}"
-			(at 219.4462 129.54 0)
-			(effects
-				(font
-					(size 1.27 1.27)
-				)
-				(justify right)
-				(hide yes)
-			)
-		)
-	)
 	(global_label "AUDIO_IN_L1"
 		(shape input)
@@
 		)
 	)
-	(global_label "VCC"
-		(shape input)
-		(at 208.28 152.4 0)
-		(fields_autoplaced yes)
-		(effects
-			(font
-				(size 1.27 1.27)
-			)
-			(justify left)
-		)
-		(property "Intersheetrefs" "${INTERSHEET_REFS}"
-			(at 214.8938 152.4 0)
-			(effects
-				(font
-					(size 1.27 1.27)
-				)
-				(justify left)
-				(hide yes)
-			)
-		)
-	)
 	(symbol
 		(lib_id "Device:R")
@@
 	)
 	(symbol
+		(lib_id "power:VCC")
+		(at 22.86 181.61 180)
+		(unit 1)
+		(exclude_from_sim no)
+		(in_bom yes)
+		(on_board yes)
+		(dnp no)
+		(fields_autoplaced yes)
+		(property "Reference" "#PWR017"
+			(at 22.86 177.8 0)
+			(effects
+				(font
+					(size 1.27 1.27)
+				)
+				(hide yes)
+			)
+		)
+		(property "Value" "VCC"
+			(at 22.86 186.69 0)
+			(effects
+				(font
+					(size 1.27 1.27)
+				)
+			)
+		)
+		(property "Footprint" ""
+			(at 22.86 181.61 0)
+			(effects
+				(font
+					(size 1.27 1.27)
+				)
+				(hide yes)
+			)
+		)
+		(property "Datasheet" ""
+			(at 22.86 181.61 0)
+			(effects
+				(font
+					(size 1.27 1.27)
+				)
+				(hide yes)
+			)
+		)
+		(property "Description" "Power symbol creates a global label with name \"VCC\""
+			(at 22.86 181.61 0)
+			(effects
+				(font
+					(size 1.27 1.27)
+				)
+				(hide yes)
+			)
+		)
+		(pin "1"
+		)
+		(instances
+			(project "doorman_audio_extension"
+				(path "/2048a046-8e00-475d-aeec-41a343368725"
+					(reference "#PWR017")
+					(unit 1)
+				)
+			)
+		)
+	)
+	(symbol
 		(lib_name "GND_7")
 		(lib_id "power:GND")
@@
 	)
 	(symbol
+		(lib_id "power:VCC")
+		(at 207.01 129.54 0)
+		(unit 1)
+		(exclude_from_sim no)
+		(in_bom yes)
+		(on_board yes)
+		(dnp no)
+		(fields_autoplaced yes)
+		(property "Reference" "#PWR016"
+			(at 207.01 133.35 0)
+			(effects
+				(font
+					(size 1.27 1.27)
+				)
+				(hide yes)
+			)
+		)
+		(property "Value" "VCC"
+			(at 207.01 124.46 0)
+			(effects
+				(font
+					(size 1.27 1.27)
+				)
+			)
+		)
+		(property "Footprint" ""
+			(at 207.01 129.54 0)
+			(effects
+				(font
+					(size 1.27 1.27)
+				)
+				(hide yes)
+			)
+		)
+		(property "Datasheet" ""
+			(at 207.01 129.54 0)
+			(effects
+				(font
+					(size 1.27 1.27)
+				)
+				(hide yes)
+			)
+		)
+		(property "Description" "Power symbol creates a global label with name \"VCC\""
+			(at 207.01 129.54 0)
+			(effects
+				(font
+					(size 1.27 1.27)
+				)
+				(hide yes)
+			)
+		)
+		(pin "1"
+		)
+		(instances
+			(project ""
+				(path "/2048a046-8e00-475d-aeec-41a343368725"
+					(reference "#PWR016")
+					(unit 1)
+				)
+			)
+		)
+	)
+	(symbol
 		(lib_name "GND_2")
 		(lib_id "power:GND")
@@
 	)
 	(symbol
+		(lib_id "power:VCC")
+		(at 213.36 152.4 180)
+		(unit 1)
+		(exclude_from_sim no)
+		(in_bom yes)
+		(on_board yes)
+		(dnp no)
+		(fields_autoplaced yes)
+		(property "Reference" "#PWR04"
+			(at 213.36 148.59 0)
+			(effects
+				(font
+					(size 1.27 1.27)
+				)
+				(hide yes)
+			)
+		)
+		(property "Value" "VCC"
+			(at 213.36 157.48 0)
+			(effects
+				(font
+					(size 1.27 1.27)
+				)
+			)
+		)
+		(property "Footprint" ""
+			(at 213.36 152.4 0)
+			(effects
+				(font
+					(size 1.27 1.27)
+				)
+				(hide yes)
+			)
+		)
+		(property "Datasheet" ""
+			(at 213.36 152.4 0)
+			(effects
+				(font
+					(size 1.27 1.27)
+				)
+				(hide yes)
+			)
+		)
+		(property "Description" "Power symbol creates a global label with name \"VCC\""
+			(at 213.36 152.4 0)
+			(effects
+				(font
+					(size 1.27 1.27)
+				)
+				(hide yes)
+			)
+		)
+		(pin "1"
+		)
+		(instances
+			(project "doorman_audio_extension"
+				(path "/2048a046-8e00-475d-aeec-41a343368725"
+					(reference "#PWR04")
+					(unit 1)
+				)
+			)
+		)
+	)
+	(symbol
 		(lib_id "Connector:Conn_01x03_Pin")
 		(at 228.6 151.13 0)
@@
 					(unit 1)
 				)
-			)
-		)
-	)
-	(symbol
-		(lib_id "power:+24V")
-		(at 22.86 181.61 180)
-		(unit 1)
-		(exclude_from_sim no)
-		(in_bom yes)
-		(on_board yes)
-		(dnp no)
-		(property "Reference" "#PWR04"
-			(at 22.86 177.8 0)
-			(effects
-				(font
-					(size 1.27 1.27)
-				)
-				(hide yes)
-			)
-		)
-		(property "Value" "VCC"
-			(at 22.86 186.69 0)
-			(effects
-				(font
-					(size 1.27 1.27)
-				)
-			)
-		)
-		(property "Footprint" ""
-			(at 22.86 181.61 0)
-			(effects
-				(font
-					(size 1.27 1.27)
-				)
-				(hide yes)
-			)
-		)
-		(property "Datasheet" ""
-			(at 22.86 181.61 0)
-			(effects
-				(font
-					(size 1.27 1.27)
-				)
-				(hide yes)
-			)
-		)
-		(property "Description" "Power symbol creates a global label with name \"VCC\""
-			(at 22.86 181.61 0)
-			(effects
-				(font
-					(size 1.27 1.27)
-				)
-				(hide yes)
-			)
-		)
-		(pin "1"
-		)
-		(instances
-			(project "doorman"
-				(path "/2048a046-8e00-475d-aeec-41a343368725"
-					(reference "#PWR04")
-					(unit 1)
-				)

Commit message: WIP
Parts:
- C13, C7: LCSC C140782 -> C730416; MPN GRM188R60J476ME15D -> CL10A476MQ8QRNC
- J4: LCSC C22373875 -> C3294446; MPN HC-PM200-4.3H-2x7PS -> PZ200-2-07-S
- R13, R14: footprint Resistor_SMD:R_0402_1005Metric -> Resistor_SMD:R_0603_1608Metric; LCSC C25744 -> C25804; MPN 0402WGF1002TCE -> 0603WAF1002T5E; Package 0402 -> 0603
- R6: LCSC C4410 -> C25361; MPN 1206W4F1001T5E -> 1206W4J0201T5E
Changed lines of the file:
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@@
 			)
 		)
-		(property "Footprint" "Resistor_SMD:R_0402_1005Metric"
+		(property "Footprint" "Resistor_SMD:R_0603_1608Metric"
 			(at 40.132 73.66 90)
 			(effects
@@
 			)
 		)
-		(property "Description" "-55℃~+155℃ 10kΩ 50V 62.5mW Thick Film Resistor ±1% ±100ppm/℃ 0402 Chip Resistor - Surface Mount ROHS"
+		(property "Description" "-55℃~+155℃ 100mW 10kΩ 75V Thick Film Resistor ±1% ±100ppm/℃ 0603 Chip Resistor - Surface Mount ROHS"
 			(at 41.91 73.66 0)
 			(effects
@@
 			)
 		)
-		(property "LCSC" "C25744"
+		(property "LCSC" "C25804"
 			(at 41.91 73.66 90)
 			(effects
@@
 			)
 		)
-		(property "MPN" "0402WGF1002TCE"
+		(property "MPN" "0603WAF1002T5E"
 			(at 41.91 73.66 90)
 			(effects
@@
 			)
 		)
-		(property "Package" "0402"
+		(property "Package" "0603"
 			(at 41.91 73.66 90)
 			(effects
@@
 			)
 		)
-		(property "Footprint" "Resistor_SMD:R_0402_1005Metric"
+		(property "Footprint" "Resistor_SMD:R_0603_1608Metric"
 			(at 43.688 83.82 90)
 			(effects
@@
 			)
 		)
-		(property "Description" "-55℃~+155℃ 10kΩ 50V 62.5mW Thick Film Resistor ±1% ±100ppm/℃ 0402 Chip Resistor - Surface Mount ROHS"
+		(property "Description" "-55℃~+155℃ 100mW 10kΩ 75V Thick Film Resistor ±1% ±100ppm/℃ 0603 Chip Resistor - Surface Mount ROHS"
 			(at 41.91 83.82 0)
 			(effects
@@
 			)
 		)
-		(property "LCSC" "C25744"
+		(property "LCSC" "C25804"
 			(at 41.91 83.82 90)
 			(effects
@@
 			)
 		)
-		(property "MPN" "0402WGF1002TCE"
+		(property "MPN" "0603WAF1002T5E"
 			(at 41.91 83.82 90)
 			(effects
@@
 			)
 		)
-		(property "Package" "0402"
+		(property "Package" "0603"
 			(at 41.91 83.82 90)
 			(effects
@@
 			)
 		)
-		(property "Description" "Generic connector, double row, 02x07, top/bottom pin numbering scheme (row 1: 1...pins_per_row, row2: pins_per_row+1 ... num_pins), script generated (kicad-library-utils/schlib/autogen/connector/)"
+		(property "Description" "-40℃~+105℃ 1.5A 14P 2 2mm 2mm 2mm 2x7P 3.8mm Black Brass Pin Header Surface Mount,Vertical SMD,P=2mm Pin Headers ROHS"
 			(at 233.68 124.46 0)
 			(effects
@@
 			)
 		)
-		(property "LCSC" "C22373875"
+		(property "LCSC" "C3294446"
 			(at 233.68 124.46 0)
 			(effects
@@
 			)
 		)
-		(property "MPN" "HC-PM200-4.3H-2x7PS "
+		(property "MPN" "PZ200-2-07-S"
 			(at 233.68 124.46 0)
 			(effects
@@
 			)
 		)
-		(property "Description" "-55℃~+155℃ 1kΩ 200V 250mW Thick Film Resistor ±1% ±100ppm/℃ 1206 Chip Resistor - Surface Mount ROHS"
+		(property "Description" "-55℃~+155℃ 200V 200Ω 250mW Thick Film Resistor ±100ppm/℃ ±5% 1206 Chip Resistor - Surface Mount ROHS"
 			(at 240.03 71.12 0)
 			(effects
@@
 			)
 		)
-		(property "LCSC" "C4410"
+		(property "LCSC" "C25361"
 			(at 240.03 71.12 90)
 			(effects
@@
 			)
 		)
-		(property "MPN" "1206W4F1001T5E"
+		(property "MPN" "1206W4J0201T5E"
 			(at 240.03 71.12 90)
 			(effects
@@
 			)
 		)
-		(property "LCSC" "C140782"
+		(property "LCSC" "C730416"
 			(at 130.81 82.55 0)
 			(effects
@@
 			)
 		)
-		(property "MPN" "GRM188R60J476ME15D"
+		(property "MPN" "CL10A476MQ8QRNC"
 			(at 130.81 82.55 0)
 			(effects
@@
 			)
 		)
-		(property "LCSC" "C140782"
+		(property "LCSC" "C730416"
 			(at 135.89 80.01 0)
 			(effects
@@
 			)
 		)
-		(property "MPN" "GRM188R60J476ME15D"
+		(property "MPN" "CL10A476MQ8QRNC"
 			(at 135.89 80.01 0)
 			(effects

Commit message: WIP
Parts:
- J1, J2, J5: now left out of the parts list
Changed lines of the file:
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@@
 		(unit 1)
 		(exclude_from_sim no)
-		(in_bom yes)
+		(in_bom no)
 		(on_board yes)
 		(dnp yes)
@@
 		(unit 1)
 		(exclude_from_sim no)
-		(in_bom yes)
+		(in_bom no)
 		(on_board yes)
 		(dnp yes)
@@
 		(unit 1)
 		(exclude_from_sim no)
-		(in_bom yes)
+		(in_bom no)
 		(on_board yes)
 		(dnp yes)

Commit message: WIP
Parts:
- added R7, R8: 0, Resistor_SMD:R_0603_1608Metric, symbol Device:R
- C13, C7: value 47uF -> 1uF; LCSC C730416 -> C15849; MPN CL10A476MQ8QRNC -> CL10A105KB8NNNC
Connections:
- net AUDIO_OUT_L1: now also R7.2, R8.1; no longer D2.1 (K), R6.1, U1.23 (RIN1)
- new net: D2.1 (K), R6.1, R8.2
- new net: R7.1, U1.23 (RIN1)
Other:
- note added: "DIFF (L1 OUT)"
- note added: "LINE OUT 1uF HP OUT 47uF"
- note removed: "Difference (L1 OUT)"
- note removed: "HP Out"
- note removed: "LINE 1uF HP 47uF"

Commit message: WIP
Parts:
- removed C6: 1uF, Capacitor_SMD:C_0603_1608Metric, symbol Device:C_Small
- removed R1: 10, Resistor_SMD:R_0603_1608Metric, symbol Device:R
- added C4, C8: 10uF, Capacitor_SMD:C_1206_3216Metric, symbol Device:C_Small
- added D3, D4: TPCDSOD323-T03SC, Diode_SMD:D_SOD-323, symbol Diode:PTVS5V0Z1USK
- added R10: 200, Resistor_SMD:R_1206_3216Metric, symbol Device:R
- added R9: 0, Resistor_SMD:R_0603_1608Metric, symbol Device:R
- D1, D2: value CDSOD323-T03S -> TPCDSOD323-T03SC
- J1: footprint Connector_PinHeader_2.54mm:PinHeader_1x04_P2.54mm_Vertical -> Connector_PinHeader_2.54mm:PinHeader_1x03_P2.54mm_Vertical; symbol Connector:Conn_01x04_Pin -> Connector:Conn_01x03_Pin; now in the parts list
Connections:
- net AUDIO_IN_L1: now also R7.1; no longer R4.1
- net AUDIO_OUT_L1: no longer R7.2
- net AUDIO_OUT_R1: now also U1.11 (ROUT1), R9.1; no longer J1.3 (Pin_3)
- net BUS_WIRE1: now also C4.1, C8.1
- net GND: now also J1.3 (Pin_3), D3.2 (A), D4.2 (A); no longer J1.4 (Pin_4)
- net at D2.1 (K), R8.2: now also R10.1; no longer R6.1
- net AUDIO_IN_R1: now reaches U1.23 (RIN1)
- net AUDIO_IN_R1: now also R4.1; no longer R7.1
- net at C12.2, R4.2: now also D3.1 (K); no longer D1.1 (K)
- new net: C4.2, D1.1 (K), R7.2
- new net: D4.1 (K), R6.1, R9.2
- new net: C8.2, R10.2
Other:
- note added: "LINE IN <- BUS (Diff)"
- note added: "LINE OUT -> BUS (Diff)"
- note removed: "DIFF (L1 OUT)"
- note removed: "LINE IN <- BUS"
- note removed: "LINE OUT -> BUS"
- moved on the sheet: C12, C13, C14, C3, C5, C7, D1, D2, J2, J4, J5, R6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
