File: pcb_extension_audio/doorman_audio_extension.kicad_sch (KiCad schematic)
At the start: 53 parts, among them J1 Audio Out, J2 GPIO, J4 Extension Board Connector, J5 Audio In, U1 ES8388

Commit message: WIP
Parts:
- removed C13: 1uF, Capacitor_SMD:C_0603_1608Metric, symbol Device:C_Small
- removed J5: Audio In, Connector_PinHeader_2.54mm:PinHeader_1x03_P2.54mm_Vertical, symbol Connector:Conn_01x03_Pin
- removed R4, R7, R8, R9: 0, Resistor_SMD:R_0603_1608Metric, symbol Device:R
- removed U1: ES8388, Package_DFN_QFN:QFN-28-1EP_4x4mm_P0.45mm_EP2.6x2.6mm, symbol Audio:ES8388
- added C6: 1uF, Capacitor_SMD:C_0603_1608Metric, symbol Device:C_Small
- added J3: Input, Connector_PinHeader_2.54mm:PinHeader_1x03_P2.54mm_Vertical, symbol Connector:Conn_01x03_Pin
- added R1, R11, R12: 10K, Resistor_SMD:R_0603_1608Metric, symbol Device:R
- added U2: ES8311, Doorman:QFN40P300X300X60-21N, symbol easyeda2kicad:ES8311
- C3, C5, C7: LCSC C15849 -> (none); MPN CL10A105KB8NNNC -> (none)
- J1: value Audio Out -> Output
- R2, R3: value 10 -> 10K; LCSC C22859 -> C25804; MPN 0603WAF100JT5E -> 0603WAF1002T5E
Connections:
- net +3.3V: now also R3.1, R1.1, R12.2, U2.11 (AVDD), U2.3 (PVDD), U2.4 (DVDD)
- net GND: now also J2.2 (Pin_2), J4.3 (Pin_3), J4.9 (Pin_9), R2.2, R5.2, J3.3 (Pin_3), R11.2, U2.10 (AGND), U2.21 (EP), U2.5 (DGND); no longer J4.2 (Pin_2), R5.1
- net I2C_CLK: now also U2.1 (CCLK)
- net I2C_DAT: now also U2.19 (CDATA)
- net I2S_BCLK: now also J4.4 (Pin_4); no longer J4.11 (Pin_11)
- net I2S_DAT_IN: now also J4.12 (Pin_12); no longer J4.4 (Pin_4)
- net I2S_LRCK: now also J4.11 (Pin_11); no longer J4.12 (Pin_12)
- net VCC: no longer J2.2 (Pin_2), J4.9 (Pin_9)
- net at C7.2: now also J3.1 (Pin_1); no longer R2.1
- net AUDIO_OUT_P: now reaches C3.1
- net AUDIO_OUT_P: now also D2.1 (K), R10.1, TP3.1, U2.13 (OUTN)
- net AUDIO_OUT_N: now reaches C5.1
- net AUDIO_OUT_N: now also D4.1 (K), R6.1, TP4.1, U2.12 (OUTP)
- net AUDIO_IN_N: now reaches C4.2, D1.1 (K), TP1.1
- net AUDIO_IN_N: now also C7.1, R2.1, R1.2, U2.17 (MIC1N)
- net at R18.1: now also U2.9 (DSDIN)
- net at R17.1: now also U2.8 (LRCK)
- net DACVREF: now reaches C17.2
- net DACVREF: now also U2.14 (DACVREF)
- net at R16.1: now also U2.6 (SCLK/DMIC_SCL)
- net VMID: now reaches C20.2, C21.2
- net VMID: now also U2.16 (VMID)
- net ADCVREF: now reaches C18.2, C19.2
- net ADCVREF: now also U2.15 (ADCVREF)
- net AUDIO_IN_P: now reaches C12.2, D3.1 (K), TP2.1
- net AUDIO_IN_P: now also R3.2, C6.1, R11.1, U2.18 (MIC1P/DMIC_SDA)
- net at R15.1: now also U2.2 (MCLK)
- net at R19.1: now also U2.7 (ASDOUT)
- net AUDIO_IN_L2: no longer names the net of C5.2
- net AUDIO_IN_L2: now also J1.1 (Pin_1)
- net AUDIO_IN_R2: no longer names the net of C3.2
- net AUDIO_IN_R2: now also J1.2 (Pin_2)
- removed net AUDIO_OUT_L2: J1.1 (Pin_1), R2.2
- removed net AUDIO_OUT_R2: J1.2 (Pin_2), R3.2
- net PIN3 renamed PIN2
- net PIN2: now also J4.2 (Pin_2); no longer J4.3 (Pin_3)
- new net: C6.2, J3.2 (Pin_2)
- new net CE: R12.1, R5.1, U2.20 (CE)
Other:
- note added: "Alternative Input & Output"
- note added: "ES8311"
- note added: "Free GPIO"
- note removed: "ES8388"
- note removed: "Free GPIOS"
- note removed: "LINE / Headphone Terminals"
- note removed: "LINE IN"
- note removed: "LINE IN <- BUS (Diff)"
- note removed: "LINE OUT"
- note removed: "LINE OUT -> BUS (Diff)"
- note removed: "LINE OUT 1uF HP OUT 47uF"
- note removed: "VMIDSEL = 10 (default) 500 kΩ divider enabled"
- moved on the sheet: C1, C10, C11, C12, C14, C17, C18, C19, C2, C20, C21, C4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

Commit message: WIP
Parts:
- added C13, C9: 10uF, Capacitor_SMD:C_0402_1005Metric, symbol Device:C_Small
- C11, C17, C19, C2, C21: LCSC C19702 -> C2959727; MPN CL10A106KP8NNNC -> GRM188Z71A106KA73D
- C3, C5, C6, C7: LCSC (none) -> C29936; MPN (none) -> CL10B105KA8NNNC
- R10, R6: LCSC C25361 -> C18002; MPN 1206W4J0201T5E -> 1206W4F2000T5E
- U2: LCSC (none) -> C962342; MPN (none) -> ES8311
Connections:
- net +3.3V: no longer R1.1, R3.1
- net AUDIO_IN_N: now also C9.1; no longer C4.2, D1.1 (K), R1.2, R2.1, TP1.1
- net AUDIO_IN_P: now also C13.1; no longer C12.2, D3.1 (K), R11.1, R3.2, TP2.1
- new net: C4.2, D1.1 (K), R1.1, TP1.1
- new net: C13.2, R11.1, R3.2
- new net: C9.2, R1.2, R2.1
- new net: C12.2, D3.1 (K), R3.1, TP2.1
Other:
- moved on the sheet: D1, D3, R1, R11, R2, R3, TP1, TP2

Commit message: WIP
Parts:
- R11, R2: now not fitted
Changed lines of the file:
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@@
 		(in_bom yes)
 		(on_board yes)
-		(dnp no)
+		(dnp yes)
 		(property "Reference" "R11"
 			(at 230.378 82.55 0)
@@
 		(in_bom yes)
 		(on_board yes)
-		(dnp no)
+		(dnp yes)
 		(property "Reference" "R2"
 			(at 229.87 48.26 0)

Commit message: Core Board V2.0.0
Parts:
- R11, R2: now fitted
Connections:
- net BUS_WIRE1: now also C14.1; no longer C8.1
- net BUS_WIRE2: now also C8.1; no longer C14.1
Changed lines of the file:
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@@
 		)
 	)
-	(global_label "BUS_WIRE2"
-		(shape input)
-		(at 255.27 142.24 0)
-		(fields_autoplaced yes)
-		(effects
-			(font
-				(size 1.27 1.27)
-			)
-			(justify left)
-		)
-		(property "Intersheetrefs" "${INTERSHEET_REFS}"
-			(at 268.7175 142.24 0)
-			(effects
-				(font
-					(size 1.27 1.27)
-				)
-				(justify left)
-				(hide yes)
-			)
-		)
-	)
 	(global_label "I2S_DAT_OUT"
 		(shape input)
@@
 		)
 	)
+	(global_label "BUS_WIRE2"
+		(shape input)
+		(at 255.27 111.76 0)
+		(fields_autoplaced yes)
+		(effects
+			(font
+				(size 1.27 1.27)
+			)
+			(justify left)
+		)
+		(property "Intersheetrefs" "${INTERSHEET_REFS}"
+			(at 268.7175 111.76 0)
+			(effects
+				(font
+					(size 1.27 1.27)
+				)
+				(justify left)
+				(hide yes)
+			)
+		)
+	)
 	(global_label "I2S_BCLK"
 		(shape input)
@@
 		)
 	)
-	(global_label "BUS_WIRE1"
-		(shape input)
-		(at 255.27 111.76 0)
-		(fields_autoplaced yes)
-		(effects
-			(font
-				(size 1.27 1.27)
-			)
-			(justify left)
-		)
-		(property "Intersheetrefs" "${INTERSHEET_REFS}"
-			(at 268.7175 111.76 0)
-			(effects
-				(font
-					(size 1.27 1.27)
-				)
-				(justify left)
-				(hide yes)
-			)
-		)
-	)
 	(global_label "I2S_DAT_IN"
 		(shape input)
@@
 	(global_label "BUS_WIRE1"
 		(shape input)
+		(at 255.27 142.24 0)
+		(fields_autoplaced yes)
+		(effects
+			(font
+				(size 1.27 1.27)
+			)
+			(justify left)
+		)
+		(property "Intersheetrefs" "${INTERSHEET_REFS}"
+			(at 268.7175 142.24 0)
+			(effects
+				(font
+					(size 1.27 1.27)
+				)
+				(justify left)
+				(hide yes)
+			)
+		)
+	)
+	(global_label "BUS_WIRE1"
+		(shape input)
 		(at 48.26 154.94 180)
 		(fields_autoplaced yes)
@@
 		(in_bom yes)
 		(on_board yes)
-		(dnp yes)
+		(dnp no)
 		(property "Reference" "R11"
 			(at 230.378 82.55 0)
@@
 		(in_bom yes)
 		(on_board yes)
-		(dnp yes)
+		(dnp no)
 		(property "Reference" "R2"
 			(at 229.87 48.26 0)
