File: pcb_panel/Doorman-S3-Panel.kicad_pcb (KiCad board)
At the start: 4 copper layers, 70 x 70 mm, 93 parts

Commit message: WIP
Parts:
- removed B0-C10, B0-C18, B0-C20: 100nF, Capacitor_SMD:C_0603_1608Metric
- removed B0-C11, B0-C17, B0-C19, B0-C21: 10uF, Capacitor_SMD:C_0603_1608Metric
- removed B0-C12, B0-C14: 1uF, Capacitor_SMD:C_1206_3216Metric
- removed B0-C13: 47uF, Capacitor_SMD:C_0603_1608Metric
- removed B0-J5: Audio In, Connector_PinHeader_2.54mm:PinHeader_1x03_P2.54mm_Vertical
- removed B0-R13, B0-R14: 10K, Resistor_SMD:R_0402_1005Metric
- removed B0-R15, B0-R16, B0-R17, B0-R18, B0-R19: 33, Resistor_SMD:R_0603_1608Metric
- removed B0-R20, B0-R21, B1-R12: 10K, Resistor_SMD:R_0603_1608Metric
- removed B0-U1: ES8388, Package_DFN_QFN:QFN-28-1EP_4x4mm_P0.45mm_EP2.6x2.6mm
- removed B1-D4: Red, LED_SMD:LED_0603_1608Metric
- removed B1-D5, B1-D6: 1N5819WS, Diode_SMD:D_SOD-323
- removed B1-D7: 6.2V, Diode_SMD:D_MELF
- removed B1-D8: XL-2020RGBC-SK6812B, Doorman:LED-SMD_6P-L2.0-W2.0_XL-2020RGBC
- removed the B1-G*** at (44.5, 55.6)
- removed B1-J2: Terminal, Doorman:CONN-TH_9P-P2.54_KF128-2.54-9P
- removed B1-J3: 3V3 Test Pad, TestPoint:TestPoint_Pad_D1.0mm
- removed B1-J6: BUS Test Pad, TestPoint:TestPoint_Pad_D1.0mm
- removed B1-J7: BUS RX Test Pad, TestPoint:TestPoint_Pad_D1.0mm
- removed B1-J8: TX Test Pad, TestPoint:TestPoint_Pad_D1.0mm
- removed B1-J9: RX Test Pad, TestPoint:TestPoint_Pad_D1.0mm
- removed B1-JP1: Bus power Jumper, Connector_PinHeader_1.27mm:PinHeader_1x02_P1.27mm_Vertical
- removed B1-L1: 3.9uH, Inductor_SMD:L_Abracon_ASPI-4030S
- removed B1-Q1: BC847BPN, Package_TO_SOT_SMD:SOT-363_SC-70-6
- removed B1-Q2: BC817, Package_TO_SOT_SMD:SOT-23
- removed B1-R10: 62, Resistor_SMD:R_1206_3216Metric
- removed B1-R11, B1-R8: 1.2, Resistor_SMD:R_0805_2012Metric
- removed B1-R7: 470, Resistor_SMD:R_0603_1608Metric
- removed B1-R9: 150, Resistor_SMD:R_0402_1005Metric
- removed B1-SW1: Reset Button, Button_Switch_SMD:SW_SPST_B3U-1000P-B
- removed B1-SW2: Flash Button, Button_Switch_SMD:SW_SPST_B3U-1000P-B
- removed B1-U2: AP63203WU, Package_TO_SOT_SMD:TSOT-23-6
- removed B1-U3: GAQY252G3S, Doorman:SOP-4_L4.4-W4.0-P2.54-LS7.0-TL
- removed B1-U4: ESP32-S3-MINI-1, RF_Module:ESP32-S2-MINI-1
- added B0-D4: Red, LED_SMD:LED_0603_1608Metric, F.Cu at (23.0, 46.8)
- added B0-D5: 1N5819WS, Diode_SMD:D_SOD-323, F.Cu at (54.7, 43.2)
- added B0-D6: 1N5819WS, Diode_SMD:D_SOD-323, F.Cu at (44.0, 75.0)
- added B0-D7: 6.2V, Diode_SMD:D_MELF, F.Cu at (44.9, 47.9)
- added B0-D8: XL-2020RGBC-SK6812B, Doorman:LED-SMD_6P-L2.0-W2.0_XL-2020RGBC, F.Cu at (23.0, 42.4)
- added B0-G***: LOGO, Doorman:esphome, B.Cu at (44.5, 57.8)
- added B0-J3: 3V3 Test Pad, TestPoint:TestPoint_Pad_D1.0mm, B.Cu at (33.9, 73.5)
- added B0-J6: BUS Test Pad, TestPoint:TestPoint_Pad_D1.0mm, B.Cu at (44.6, 48.4)
- added B0-J7: BUS RX Test Pad, TestPoint:TestPoint_Pad_D1.0mm, B.Cu at (37.2, 66.9)
- added B0-J8: TX Test Pad, TestPoint:TestPoint_Pad_D1.0mm, B.Cu at (30.9, 54.6)
- added B0-J9: RX Test Pad, TestPoint:TestPoint_Pad_D1.0mm, B.Cu at (28.9, 54.6)
- added B0-JP1: Bus power Jumper, Connector_PinHeader_1.27mm:PinHeader_1x02_P1.27mm_Vertical, F.Cu at (43.5, 71.3)
- added B0-L1: 3.9uH, Inductor_SMD:L_Abracon_ASPI-4030S, F.Cu at (32.2, 73.5)
- added B0-Q1: BC847BPN, Package_TO_SOT_SMD:SOT-363_SC-70-6, F.Cu at (32.5, 48.7)
- added B0-Q2: BC817, Package_TO_SOT_SMD:SOT-23, F.Cu at (39.6, 48.7)
- added B0-R10: 62, Resistor_SMD:R_1206_3216Metric, F.Cu at (41.2, 73.2)
- added B0-R11: 1.2, Resistor_SMD:R_0805_2012Metric, F.Cu at (36.0, 49.7)
- added B0-R12: 10K, Resistor_SMD:R_0603_1608Metric, F.Cu at (30.2, 48.7)
- added B0-R7: 470, Resistor_SMD:R_0603_1608Metric, F.Cu at (23.0, 45.2)
- added B0-R8: 1.2, Resistor_SMD:R_0805_2012Metric, F.Cu at (36.0, 47.8)
- added B0-R9: 150, Resistor_SMD:R_0402_1005Metric, F.Cu at (28.7, 49.2)
- added B0-SW1: Reset Button, Button_Switch_SMD:SW_SPST_B3U-1000P-B, F.Cu at (23.8, 73.7)
- added B0-SW2: Flash Button, Button_Switch_SMD:SW_SPST_B3U-1000P-B, F.Cu at (23.8, 69.5)
- added B0-U2: AP63203WU, Package_TO_SOT_SMD:TSOT-23-6, F.Cu at (37.2, 72.6)
- added B0-U3: GAQY252G3S, Doorman:SOP-4_L4.4-W4.0-P2.54-LS7.0-TL, F.Cu at (27.4, 43.9)
- added B0-U4: ESP32-S3-MINI-1, RF_Module:ESP32-S2-MINI-1, F.Cu at (30.4, 59.3)
- added B1-C10: 100nF, Capacitor_SMD:C_0603_1608Metric, F.Cu at (73.3, 67.5)
- added B1-C11: 10uF, Capacitor_SMD:C_0603_1608Metric, F.Cu at (73.3, 69.0)
- added B1-C12: 1uF, Capacitor_SMD:C_1206_3216Metric, F.Cu at (77.6, 72.2)
- added B1-C13: 47uF, Capacitor_SMD:C_0603_1608Metric, F.Cu at (63.0, 56.7)
- added B1-C14: 1uF, Capacitor_SMD:C_1206_3216Metric, F.Cu at (85.2, 64.5)
- added B1-C17: 10uF, Capacitor_SMD:C_0603_1608Metric, F.Cu at (68.2, 56.0)
- added B1-C18: 100nF, Capacitor_SMD:C_0603_1608Metric, F.Cu at (63.8, 65.0)
- added B1-C19: 10uF, Capacitor_SMD:C_0603_1608Metric, F.Cu at (62.3, 65.0)
- added B1-C20: 100nF, Capacitor_SMD:C_0603_1608Metric, F.Cu at (63.1, 68.9)
- added B1-C21: 10uF, Capacitor_SMD:C_0603_1608Metric, F.Cu at (63.1, 67.5)
- added B1-J5: Audio In, Connector_PinHeader_2.54mm:PinHeader_1x03_P2.54mm_Vertical, B.Cu at (64.2, 74.6)
- added B1-R13: 10K, Resistor_SMD:R_0402_1005Metric, F.Cu at (76.6, 54.1)
- added B1-R14: 10K, Resistor_SMD:R_0402_1005Metric, F.Cu at (79.8, 54.1)
- added B1-R15: 33, Resistor_SMD:R_0603_1608Metric, F.Cu at (71.1, 68.2)
- added B1-R16: 33, Resistor_SMD:R_0603_1608Metric, F.Cu at (74.0, 63.3)
- added B1-R17: 33, Resistor_SMD:R_0603_1608Metric, F.Cu at (71.2, 56.0)
- added B1-R18: 33, Resistor_SMD:R_0603_1608Metric, F.Cu at (74.0, 60.3)
- added B1-R19: 33, Resistor_SMD:R_0603_1608Metric, F.Cu at (69.7, 56.0)
- added B1-R20: 10K, Resistor_SMD:R_0603_1608Metric, F.Cu at (72.6, 71.4)
- added B1-R21: 10K, Resistor_SMD:R_0603_1608Metric, F.Cu at (74.1, 71.4)
- added B1-U1: ES8388, Package_DFN_QFN:QFN-28-1EP_4x4mm_P0.45mm_EP2.6x2.6mm, F.Cu at (68.9, 62.3)
- B0-C2: value 10uF -> 100nF
- B0-C3: value 1uF -> 470uF; footprint Capacitor_SMD:C_0603_1608Metric -> Capacitor_SMD:CP_Elec_8x10
- B0-C4: value 1uF -> 10uF; footprint Capacitor_SMD:C_0603_1608Metric -> Capacitor_SMD:C_1206_3216Metric
- B0-C5: value 1uF -> 100nF
- B0-C6: value 1uF -> 22uF
- B0-C7: value 47uF -> 22uF
- B0-D1: value CDSOD323-T03S -> 1N5819WS
- B0-D2: value CDSOD323-T03S -> MB6S; footprint Diode_SMD:D_SOD-323 -> Package_TO_SOT_SMD:TO-269AA
- B0-J1: value Audio Out -> USB_C_Receptacle_USB2.0; footprint Connector_PinHeader_2.54mm:PinHeader_1x03_P2.54mm_Vertical -> Connector_USB:USB_C_Receptacle_HRO_TYPE-C-31-M-12; moved to F.Cu
- B0-J2: value Conn_01x02_Pin -> Terminal; footprint Connector_JST:JST_SHL_SM02B-SHLS-TF_1x02-1MP_P1.00mm_Horizontal -> Doorman:CONN-TH_9P-P2.54_KF128-2.54-9P
- B0-J4: value Extension Board Connector -> Conn_02x07_Odd_Even; footprint Connector_PinHeader_2.00mm:PinHeader_2x07_P2.00mm_Vertical_SMD -> Connector_PinSocket_2.00mm:PinSocket_2x07_P2.00mm_Vertical_SMD
- B0-R1: value 10 -> 10K
- B0-R2: value 10 -> 2.2K; footprint Resistor_SMD:R_0603_1608Metric -> Resistor_SMD:R_0402_1005Metric
- B0-R3: value 10 -> 5.1K; footprint Resistor_SMD:R_0603_1608Metric -> Resistor_SMD:R_0402_1005Metric
- B0-R5: value 10K -> 47K
- B0-R6: value 1K -> 10K; footprint Resistor_SMD:R_1206_3216Metric -> Resistor_SMD:R_0603_1608Metric
- B1-C2: value 100nF -> 10uF
- B1-C3: value 470uF -> 1uF; footprint Capacitor_SMD:CP_Elec_8x10 -> Capacitor_SMD:C_0603_1608Metric
- B1-C4: value 10uF -> 1uF; footprint Capacitor_SMD:C_1206_3216Metric -> Capacitor_SMD:C_0603_1608Metric
- B1-C5: value 100nF -> 1uF
- B1-C6: value 22uF -> 1uF
- B1-C7: value 22uF -> 47uF
- B1-D1: value 1N5819WS -> CDSOD323-T03S
- B1-D2: value MB6S -> CDSOD323-T03S; footprint Package_TO_SOT_SMD:TO-269AA -> Diode_SMD:D_SOD-323
- B1-J1: value USB_C_Receptacle_USB2.0 -> Audio Out; footprint Connector_USB:USB_C_Receptacle_HRO_TYPE-C-31-M-12 -> Connector_PinHeader_2.54mm:PinHeader_1x03_P2.54mm_Vertical; moved to B.Cu
- B1-J4: value Conn_02x07_Odd_Even -> Extension Board Connector; footprint Connector_PinSocket_2.00mm:PinSocket_2x07_P2.00mm_Vertical_SMD -> Connector_PinHeader_2.00mm:PinHeader_2x07_P2.00mm_Vertical_SMD
- B1-R1: value 10K -> 10
- B1-R2: value 2.2K -> 10; footprint Resistor_SMD:R_0402_1005Metric -> Resistor_SMD:R_0603_1608Metric
- B1-R3: value 5.1K -> 10; footprint Resistor_SMD:R_0402_1005Metric -> Resistor_SMD:R_0603_1608Metric
- B1-R5: value 47K -> 10K
- B1-R6: value 10K -> 1K; footprint Resistor_SMD:R_0603_1608Metric -> Resistor_SMD:R_1206_3216Metric
- moved B0-REF** 56.8 mm to (25.4, 71.6)
- moved B1-REF** 54.9 mm to (76.5, 49.2)
- moved B1-G*** 45.6 mm to (79.3, 65.4)
- moved B0-G*** 44.9 mm to (34.6, 58.4)
- moved B0-R1 44.0 mm to (28.1, 75.1), turned to 180 degrees
- moved B1-R6 43.4 mm to (85.2, 59.9), turned to -90 degrees
- moved B0-R6 42.4 mm to (43.5, 50.2), turned to 180 degrees
- moved B1-R1 41.9 mm to (66.0, 55.3), turned to 0 degrees
- moved B0-C1 37.4 mm to (27.3, 72.9)
- moved B0-C2 36.8 mm to (27.9, 68.3), turned to 0 degrees
- moved B0-C6 36.2 mm to (32.8, 69.0), turned to 0 degrees
- moved B1-C1 36.1 mm to (62.3, 62.1)
- moved B1-C2 36.0 mm to (63.8, 62.1), turned to 90 degrees
- moved B1-C6 34.7 mm to (66.0, 56.7), turned to 180 degrees
- moved B1-J4 34.6 mm to (79.0, 62.1)
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Connections:
- B0-C1 pad 1: B0-GND -> B0-/EN
- B0-C1 pad 2: B0-+3.3V -> B0-GND
- B0-C3 pad 1: B0-Net-(U1-RIN2) -> B0-/VCC_IN
- B0-C3 pad 2: B0-AUDIO_IN_R2 -> B0-GND
- B0-C4 pad 1: B0-Net-(U1-RIN1) -> B0-/VCC_IN
- B0-C4 pad 2: B0-AUDIO_IN_R1 -> B0-GND
- B0-C5 pad 1: B0-Net-(U1-LIN2) -> B0-Net-(U2-BST)
- B0-C5 pad 2: B0-AUDIO_IN_L2 -> B0-Net-(U2-SW)
- B0-C6 pad 1: B0-Net-(U1-ROUT1) -> B0-+3.3V
- B0-C6 pad 2: B0-Net-(C6-Pad2) -> B0-GND
- B0-C7 pad 1: B0-Net-(U1-LOUT2) -> B0-+3.3V
- B0-C7 pad 2: B0-Net-(C7-Pad2) -> B0-GND
- B0-D1 pad 1: B0-AUDIO_IN_L1 -> B0-/VCC_IN
- B0-D1 pad 2: B0-GND -> B0-+5V
- B0-D2 pad 1: B0-AUDIO_OUT_L1 -> B0-BUS_WIRE1
- B0-D2 pad 2: B0-GND -> B0-BUS_WIRE2
- B0-J2 pad 1: B0-unconnected-(J2-Pin_1-Pad1) -> B0-VCC
- B0-J2 pad 2: B0-unconnected-(J2-Pin_2-Pad2) -> B0-BUS_WIRE2
- B0-J4 pad 1: B0-BUS_WIRE2 -> B0-I2C_CLK
- B0-J4 pad 10: B0-I2S_LRCK -> B0-IO7
- B0-J4 pad 12: B0-I2C_DAT -> B0-/VCC_IN
- B0-J4 pad 13: B0-I2C_CLK -> B0-BUS_WIRE2
- B0-J4 pad 14: B0-+3.3V -> B0-BUS_WIRE1
- B0-J4 pad 2: B0-BUS_WIRE1 -> B0-+3.3V
- B0-J4 pad 4: B0-unconnected-(J4-Pin_4-Pad4) -> B0-I2C_DAT
- B0-J4 pad 5: B0-unconnected-(J4-Pin_5-Pad5) -> B0-IO14
- B0-J4 pad 6: B0-I2S_MCLK -> B0-IO15
- B0-J4 pad 7: B0-I2S_SCLK -> B0-IO16
- B0-J4 pad 8: B0-I2S_DAT_IN -> B0-IO17
- B0-J4 pad 9: B0-I2S_DAT_OUT -> B0-IO18
- B0-R1 pad 1: B0-Net-(C6-Pad2) -> B0-+3.3V
- B0-R1 pad 2: B0-AUDIO_OUT_R1 -> B0-/EN
- B0-R2 pad 1: B0-Net-(C7-Pad2) -> B0-BUS_TX
- B0-R2 pad 2: B0-AUDIO_OUT_L2 -> B0-Net-(Q1A-C1)
- B0-R3 pad 1: B0-Net-(C13-Pad2) -> B0-Net-(J1-CC1)
- B0-R3 pad 2: B0-AUDIO_OUT_R2 -> B0-GND
- B0-R5 pad 1: B0-GND -> B0-Net-(Q1B-B2)
- B0-R5 pad 2: B0-Net-(U1-CE) -> B0-+24V Bus
- B0-R6 pad 1: B0-AUDIO_OUT_L1 -> B0-Net-(Q1B-B2)
- B0-R6 pad 2: B0-Net-(C14-Pad2) -> B0-GND
- B1-C1 pad 1: B1-/EN -> B1-GND
- B1-C1 pad 2: B1-GND -> B1-+3.3V
- B1-C3 pad 1: B1-/VCC_IN -> B1-Net-(U1-RIN2)
- B1-C3 pad 2: B1-GND -> B1-AUDIO_IN_R2
- B1-C4 pad 1: B1-/VCC_IN -> B1-Net-(U1-RIN1)
- B1-C4 pad 2: B1-GND -> B1-AUDIO_IN_R1
- B1-C5 pad 1: B1-Net-(U2-BST) -> B1-Net-(U1-LIN2)
- B1-C5 pad 2: B1-Net-(U2-SW) -> B1-AUDIO_IN_L2
- B1-C6 pad 1: B1-+3.3V -> B1-Net-(U1-ROUT1)
- B1-C6 pad 2: B1-GND -> B1-Net-(C6-Pad2)
- B1-C7 pad 1: B1-+3.3V -> B1-Net-(U1-LOUT2)
- B1-C7 pad 2: B1-GND -> B1-Net-(C7-Pad2)
- B1-D1 pad 1: B1-/VCC_IN -> B1-AUDIO_IN_L1
- B1-D1 pad 2: B1-+5V -> B1-GND
- B1-D2 pad 1: B1-BUS_WIRE1 -> B1-AUDIO_OUT_L1
- B1-D2 pad 2: B1-BUS_WIRE2 -> B1-GND
- B1-J4 pad 1: B1-I2C_CLK -> B1-BUS_WIRE2
- B1-J4 pad 10: B1-IO7 -> B1-I2S_LRCK
- B1-J4 pad 12: B1-/VCC_IN -> B1-I2C_DAT
- B1-J4 pad 13: B1-BUS_WIRE2 -> B1-I2C_CLK
- B1-J4 pad 14: B1-BUS_WIRE1 -> B1-+3.3V
- B1-J4 pad 2: B1-+3.3V -> B1-BUS_WIRE1
- B1-J4 pad 4: B1-I2C_DAT -> B1-unconnected-(J4-Pin_4-Pad4)
- B1-J4 pad 5: B1-IO14 -> B1-unconnected-(J4-Pin_5-Pad5)
- B1-J4 pad 6: B1-IO15 -> B1-I2S_MCLK
- B1-J4 pad 7: B1-IO16 -> B1-I2S_SCLK
- B1-J4 pad 8: B1-IO17 -> B1-I2S_DAT_IN
- B1-J4 pad 9: B1-IO18 -> B1-I2S_DAT_OUT
- B1-R1 pad 1: B1-+3.3V -> B1-Net-(C6-Pad2)
- B1-R1 pad 2: B1-/EN -> B1-AUDIO_OUT_R1
- B1-R2 pad 1: B1-BUS_TX -> B1-Net-(C7-Pad2)
- B1-R2 pad 2: B1-Net-(Q1A-C1) -> B1-AUDIO_OUT_L2
- B1-R3 pad 1: B1-Net-(J1-CC1) -> B1-Net-(C13-Pad2)
- B1-R3 pad 2: B1-GND -> B1-AUDIO_OUT_R2
- B1-R5 pad 1: B1-Net-(Q1B-B2) -> B1-GND
- B1-R5 pad 2: B1-+24V Bus -> B1-Net-(U1-CE)
- B1-R6 pad 1: B1-Net-(Q1B-B2) -> B1-AUDIO_OUT_L1
- B1-R6 pad 2: B1-GND -> B1-Net-(C14-Pad2)
Routing:
- net B1-/VCC_IN: track 71.5 -> 0.00 mm, vias 4 -> 0
- net B0-/VCC_IN: track 0.00 -> 71.5 mm, vias 0 -> 4
- net B0-AUDIO_OUT_L1: track 34.2 -> 0.00 mm, vias 2 -> 0
- net B1-AUDIO_OUT_L1: track 0.00 -> 34.2 mm, vias 0 -> 2
- net B1-+24V Bus: track 30.6 -> 0.00 mm, vias 1 -> 0
- net B0-+24V Bus: track 0.00 -> 30.6 mm, vias 0 -> 1
- net B1-LED_RGB: track 27.7 -> 0.00 mm, vias 2 -> 0
- net B0-LED_RGB: track 0.00 -> 27.7 mm, vias 0 -> 2
- net B1-/EN: track 26.5 -> 0.00 mm, vias 2 -> 0
- net B0-/EN: track 0.00 -> 26.5 mm, vias 0 -> 2
- net B1-BUS_WIRE1: track 24.7 -> 0.00 mm, vias 2 -> 0
- net B0-BUS_WIRE1: track 0.00 -> 24.7 mm, vias 0 -> 2
- net B1-+3.3V: track 77.6 -> 53.0 mm, vias 7 -> 3
- net B0-+3.3V: track 53.0 -> 77.6 mm, vias 3 -> 7
- net B1-LED_RED: track 24.3 -> 0.00 mm, vias 2 -> 0
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- added copper zone on F.Cu, net B0-+3.3V
- added copper zone on F.Cu, net B0-/VCC_IN
- added copper zone on F.Cu, net B0-Net-(U2-SW)
- removed copper zone on F.Cu, net B1-+3.3V
- removed copper zone on F.Cu, net B1-/VCC_IN
- removed copper zone on F.Cu, net B1-Net-(U2-SW)
Other:
- outline, holes or cut-outs redrawn
- board text added: "V-CUT 39.35 mm"
- board text added: "V-CUT 60.43 mm"
- board text added: "V-CUT 76.40 mm"
- board text removed: "J2"

Commit message: WIP
Parts:
- removed B1-C4: 1uF, Capacitor_SMD:C_0603_1608Metric
- removed B1-R20, B1-R21: 10K, Resistor_SMD:R_0603_1608Metric
- added B1-G***: LOGO, Doorman:doorman-web-qr, B.Cu at (76.5, 49.5)
- added B1-J2: GPIO, Connector_PinHeader_2.54mm:PinHeader_1x02_P2.54mm_Vertical, F.Cu at (86.3, 74.6)
- added B1-R4: 0, Resistor_SMD:R_0603_1608Metric, F.Cu at (68.2, 68.2)
- B0-J1: value USB_C_Receptacle_USB2.0 -> USB-C Connector
- B0-J2: value Terminal -> Screw Terminals
- B0-J4: value Conn_02x07_Odd_Even -> Extension Board Connector
- B0-R10: value 62 -> 62R
- B0-R11, B0-R8: value 1.2 -> 1R2
- B0-R12: value 10K -> 47K5
- B0-R2: value 2.2K -> 2K2
- B0-R3: value 5.1K -> 5K1
- B0-R5: value 47K -> 47K5
- B0-R7: value 470 -> 470R
- B0-R9: value 150 -> 150R
- B0-SW1: value Reset Button -> Button
- B0-SW2: value Flash Button -> Button
- B1-C12, B1-C14: value 1uF -> 10uF
- B1-J1: footprint Connector_PinHeader_2.54mm:PinHeader_1x03_P2.54mm_Vertical -> Connector_PinHeader_2.54mm:PinHeader_1x04_P2.54mm_Vertical
- B1-R13, B1-R14: footprint Resistor_SMD:R_0402_1005Metric -> Resistor_SMD:R_0603_1608Metric
- B1-R6: value 1K -> 200
- B1-REF**: moved to F.Cu
- moved B1-C11 4.46 mm to (73.2, 64.5)
- moved B1-C10 4.46 mm to (73.2, 63.0)
- moved B1-R17 3.38 mm to (73.2, 58.7), turned to 0 degrees
- moved B1-R15 3.09 mm to (73.2, 66.0), turned to 0 degrees
- moved B1-R16 1.91 mm to (73.2, 61.6), turned to 0 degrees
- moved B1-C12 1.71 mm to (75.8, 72.1)
- moved B1-D1 1.64 mm to (72.2, 73.2), turned to -90 degrees
- moved B1-C1 1.48 mm to (63.8, 62.1)
- moved B1-C2 1.46 mm to (62.3, 62.1)
- moved B1-C14 0.94 mm to (86.1, 64.5)
- moved B1-R6 0.93 mm to (86.1, 59.9)
- moved B1-R18 0.84 mm to (73.2, 60.1), turned to 0 degrees
- moved B1-R14 0.71 mm to (79.2, 53.8)
- moved B1-R13 0.45 mm to (76.2, 53.8)
- moved B1-REF** 0.32 mm to (76.7, 49.0), turned to 90 degrees
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Connections:
- B0-J7 pad 1: B0-BUS_CONN -> B0-BUS_RX
- B0-Q1 pad 3: B0-+3.3V -> B0-BUS_RX
- B0-Q1 pad 4: B0-BUS_CONN -> B0-+3.3V
- B0-R12 pad 1: B0-BUS_CONN -> B0-BUS_RX
- B0-U4 pad 13: B0-BUS_CONN -> B0-BUS_RX
- B0-U4 pad 14: B0-BUS_CONN -> B0-BUS_RX
- B1-C12 pad 2: B1-AUDIO_IN_L1 -> B1-Net-(D1-K)
- B1-D1 pad 1: B1-AUDIO_IN_L1 -> B1-Net-(D1-K)
- B1-J4 pad 10: B1-I2S_LRCK -> B1-I2S_MCLK
- B1-J4 pad 11: B1-GND -> B1-I2S_BCLK
- B1-J4 pad 12: B1-I2C_DAT -> B1-I2S_LRCK
- B1-J4 pad 13: B1-I2C_CLK -> B1-I2C_DAT
- B1-J4 pad 2: B1-BUS_WIRE1 -> B1-GND
- B1-J4 pad 3: B1-GND -> B1-PIN3
- B1-J4 pad 4: B1-unconnected-(J4-Pin_4-Pad4) -> B1-I2S_DAT_IN
- B1-J4 pad 5: B1-unconnected-(J4-Pin_5-Pad5) -> B1-I2S_DAT_OUT
- B1-J4 pad 6: B1-I2S_MCLK -> B1-GND
- B1-J4 pad 7: B1-I2S_SCLK -> B1-I2C_CLK
- B1-J4 pad 8: B1-I2S_DAT_IN -> B1-BUS_WIRE1
- B1-J4 pad 9: B1-I2S_DAT_OUT -> B1-VCC
- B1-J5 pad 3: B1-AUDIO_IN_R1 -> B1-GND
- B1-R16 pad 2: B1-I2S_SCLK -> B1-I2S_BCLK
- B1-U1 pad 23: B1-Net-(U1-RIN1) -> B1-AUDIO_OUT_L1
Routing:
- net B0-BUS_RX: track 0.00 -> 26.9 mm, vias 0 -> 3
- net B0-BUS_CONN: track 23.7 -> 0.00 mm, vias 3 -> 0
- net B1-PIN3: track 0.00 -> 14.7 mm, vias 0 -> 1
- net B1-+3.3V: track 53.0 -> 40.3 mm
- net B1-AUDIO_IN_L1: track 16.0 -> 3.29 mm, vias 2 -> 0
- net B1-VCC: track 0.00 -> 12.5 mm, vias 0 -> 1
- net B1-Net-(D1-K): track 0.00 -> 8.38 mm
- net B1-AUDIO_OUT_L1: track 34.2 -> 42.2 mm, vias 2 -> 4
- net B1-I2S_SCLK: track 7.95 -> 0.00 mm
- net B1-I2S_DAT_OUT: track 21.1 -> 14.0 mm, vias 2 -> 0
- net B1-AUDIO_IN_R1: track 6.10 -> 0.00 mm
- net B1-I2S_MCLK: track 10.2 -> 4.13 mm, vias 2 -> 0
- net B1-I2S_LRCK: track 8.60 -> 3.49 mm
- net B1-I2S_DAT_IN: track 3.29 -> 7.94 mm
- net B0-+3.3V: track 77.6 -> 82.2 mm
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Other:
- outline, holes or cut-outs redrawn
- board text added: "01"
- board text added: "07"
- board text added: "08 TC:BUS 09 VCC 10 I²S BCLK 11 I²S IN 12 I²S LRCK 13 I²C DAT 14 3V3"
- board text added: "14"
- board text added: "ES8388"
- board text added: "EXTENSION CONNECTOR"
- board text added: "EXTRAS"
- board text added: "HP"
- board text added: "HP 47uF LN 1uF"
- board text added: "INPUTS"
- board text added: "LN"
- board text added: "OUTPUTS"
- board text added: "P3"
- board text added: "SCAN QR CODE FOR DOCS"
- board text added: "TC:BUS 01 GND 02 I²S MCLK 03 P4 04 I²S OUT 05 GND 06 I²C CLK 07"
- board text added: "VCC"
- board text removed: "DO NOT USE THIS WITH NON TC:BUS INTERCOM SYSTEMS"
