File: pcb_core_board/doorman.kicad_pcb (KiCad board)
At the start: 4 copper layers, 37 x 37.2 mm, 60 parts, among them J1 USB-C Connector, J10 VCC Test Pad, J2 Screw Terminals, J3 3V3 Test Pad, J4 Extension Board Connector, J5 Siedle BUS RX Test Pad, J6 BUS Test Pad, J7 BUS RX Test Pad, J8 TX Test Pad, J9 RX Test Pad, Q1 BC847BPN, Q2 BC817-40, Q3 BC817-40, Q4 BC817-40, Q6 BC847BPN, SW1 Button, SW2 Button, U2 AP63203WU, U3 GAQY252G3S, U4 ESP32-S3-MINI-1

Commit message: Core Board V2.0.0
Parts:
- D1, D5, D6: value 1N5819WS -> PMEG6010CEJ
- moved J10 14.4 mm to (88.6, 59.9)
Connections:
- J4 pad 11: GND -> IO12
- J4 pad 12: /VCC_IN -> GND
- J4 pad 9: IO12 -> GND
Routing:
- net /VCC_IN: track 67.6 -> 52.3 mm, vias 4 -> 3
- net IO12: track 14.3 -> 15.8 mm
- net GND: vias 129 -> 134
Other:
- board size 37 x 37.2 mm -> 37.2 x 37.2 mm
