File: pcb_core_board/doorman.kicad_sch (KiCad schematic)
At the start: 57 parts, among them J1 USB-C Connector, J10 VCC Test Pad, J2 Screw Terminals, J3 3V3 Test Pad, J4 Extension Board Connector, J5 Siedle BUS RX Test Pad, J6 BUS Test Pad, J7 BUS RX Test Pad, J8 TX Test Pad, J9 RX Test Pad, Q1 BC847BPN, Q2 BC817-40, Q3 BC817-40, Q4 BC817-40, Q6 BC847BPN, SW1 Button, SW2 Button, U2 AP63203WU, U3 GAQY252G3S, U4 ESP32-S3-MINI-1

Commit message: Core Board V2.0.0
Parts:
- D1, D5, D6: value 1N5819WS -> PMEG6010CEJ; LCSC C191023 -> C27636122; MPN 1N5819WS -> PMEG6010CEJ
