File: hardware/extension_audio/doorman_extension_audio.kicad_pcb (KiCad board)
At the start: 4 copper layers, 31.4 x 29.6 mm, 57 parts, among them J1 Output, J2 GPIO, J3 Input, J4 Extension Board Connector, U2 ES8311

Commit message: Change structure
Parts:
- added kibuzzard-69BBCF9C: G***, kibuzzard-69BBCF9C, B.Cu at (111.0, 48.6)
- added kibuzzard-69BBD00D: G***, kibuzzard-69BBD00D, B.Cu at (98.7, 48.6)
- added kibuzzard-69BBD06F: G***, kibuzzard-69BBD06F, B.Cu at (86.7, 48.6)
- added kibuzzard-69BBD0F2: G***, kibuzzard-69BBD0F2, F.Cu at (87.0, 48.6)
- added kibuzzard-69BBD107: G***, kibuzzard-69BBD107, F.Cu at (110.7, 48.6)
- added kibuzzard-69BBD4A4: G***, kibuzzard-69BBD4A4, F.Cu at (86.9, 76.6)
- added kibuzzard-69BBEEE6: G***, kibuzzard-69BBEEE6, B.Cu at (94.3, 75.2)
- moved TP6 4.02 mm to (103.8, 61.6)
- moved TP7 3.11 mm to (90.6, 57.4)
- moved J2 2.60 mm to (85.1, 73.6), turned to 0 degrees
- moved C6 2.24 mm to (88.4, 52.1), turned to -90 degrees
- moved TP8 1.72 mm to (97.6, 70.5)
- moved TP9 1.10 mm to (90.5, 60.5)
- moved R12 0.41 mm to (93.0, 51.9)
- moved R5 0.41 mm to (91.5, 51.9)
- moved TP5 0.40 mm to (105.1, 65.8)
- moved C7 0.19 mm to (88.4, 55.1)
Routing:
- net AVDD: track 37.9 -> 39.7 mm
- net I2C_DAT: track 26.2 -> 24.7 mm
- net Net-(D1-K): track 23.6 -> 25.1 mm
- net Net-(J3-Pin_2): track 4.95 -> 3.69 mm
- net I2S_BCLK: track 14.4 -> 13.3 mm
- net PIN2: track 17.0 -> 18.0 mm
- net AUDIO_IN_P: track 9.62 -> 10.2 mm
- net BUS_WIRE1: track 14.3 -> 13.7 mm
- net I2S_LRCK: track 11.5 -> 12.1 mm
- net GND: vias 98 -> 112
Other:
- board text removed: "EXTENSION CONNECTOR"
- board text removed: "GND"
- board text removed: "GPIO"
- board text removed: "INPUT"
- board text removed: "OUTPUT"
- board text removed: "SCAN QR CODE FOR DOCS"

Commit message: Update PCB files
Connections:
- C14 pad 1: BUS_WIRE1 -> BUS_WIRE2
- C3 pad 1: AUDIO_OUT_P -> AUDIO_OUT_N
- C5 pad 1: AUDIO_OUT_N -> AUDIO_OUT_P
- C8 pad 1: BUS_WIRE2 -> BUS_WIRE1
- D2 pad 1: AUDIO_OUT_P -> AUDIO_OUT_N
- D4 pad 1: AUDIO_OUT_N -> AUDIO_OUT_P
- R10 pad 1: AUDIO_OUT_P -> AUDIO_OUT_N
- R6 pad 1: AUDIO_OUT_N -> AUDIO_OUT_P
- TP3 pad 1: AUDIO_OUT_P -> AUDIO_OUT_N
- TP4 pad 1: AUDIO_OUT_N -> AUDIO_OUT_P
- U2 pad 12: AUDIO_OUT_N -> AUDIO_OUT_P
- U2 pad 13: AUDIO_OUT_P -> AUDIO_OUT_N
Routing:
- net AUDIO_OUT_P: track 34.1 -> 28.3 mm
- net AUDIO_OUT_N: track 28.3 -> 34.1 mm
Changed lines of the file:
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@@
 			(layers "F.Cu" "F.Mask" "F.Paste")
 			(roundrect_rratio 0.25)
-			(net 25 "AUDIO_OUT_P")
+			(net 27 "AUDIO_OUT_N")
 			(pintype "passive")
 		)
@@
 			(layers "F.Cu" "F.Mask" "F.Paste")
 			(roundrect_rratio 0.217391)
-			(net 6 "BUS_WIRE1")
+			(net 4 "BUS_WIRE2")
 			(pintype "passive")
 		)
@@
 			(layers "F.Cu" "F.Mask" "F.Paste")
 			(roundrect_rratio 0.25)
-			(net 27 "AUDIO_OUT_N")
+			(net 25 "AUDIO_OUT_P")
 			(pinfunction "K")
 			(pintype "passive")
@@
 			(layers "F.Cu" "F.Mask" "F.Paste")
 			(roundrect_rratio 0.222222)
-			(net 25 "AUDIO_OUT_P")
+			(net 27 "AUDIO_OUT_N")
 			(pintype "passive")
 		)
@@
 			(layers "F.Cu" "F.Mask" "F.Paste")
 			(roundrect_rratio 0.25)
-			(net 25 "AUDIO_OUT_P")
+			(net 27 "AUDIO_OUT_N")
 			(pinfunction "K")
 			(pintype "passive")
@@
 			(size 0.75 0.2)
 			(layers "F.Cu" "F.Mask" "F.Paste")
-			(net 27 "AUDIO_OUT_N")
+			(net 25 "AUDIO_OUT_P")
 			(pinfunction "OUTP")
 			(pintype "unspecified")
@@
 			(size 0.75 0.2)
 			(layers "F.Cu" "F.Mask" "F.Paste")
-			(net 25 "AUDIO_OUT_P")
+			(net 27 "AUDIO_OUT_N")
 			(pinfunction "OUTN")
 			(pintype "unspecified")
@@
 			(layers "F.Cu" "F.Mask" "F.Paste")
 			(roundrect_rratio 0.222222)
-			(net 27 "AUDIO_OUT_N")
+			(net 25 "AUDIO_OUT_P")
 			(pintype "passive")
 		)
@@
 			(layers "F.Cu" "F.Mask" "F.Paste")
 			(roundrect_rratio 0.217391)
-			(net 4 "BUS_WIRE2")
+			(net 6 "BUS_WIRE1")
 			(pintype "passive")
 		)
@@
 			(layers "F.Cu" "F.Mask" "F.Paste")
 			(roundrect_rratio 0.25)
-			(net 27 "AUDIO_OUT_N")
+			(net 25 "AUDIO_OUT_P")
 			(pintype "passive")
 		)
@@
 			(size 1 1)
 			(layers "B.Cu" "B.Mask")
-			(net 27 "AUDIO_OUT_N")
+			(net 25 "AUDIO_OUT_P")
 			(pinfunction "1")
 			(pintype "passive")
@@
 			(size 1 1)
 			(layers "B.Cu" "B.Mask")
-			(net 25 "AUDIO_OUT_P")
+			(net 27 "AUDIO_OUT_N")
 			(pinfunction "1")
 			(pintype "passive")
@@
 		)
 	)
-	(gr_text "-"
+	(gr_text "+"
 		(at 111.8 55.26 180)
 		(layer "F.SilkS")
@@
 		)
 	)
-	(gr_text "+"
-		(at 110.72 52.55 270)
+	(gr_text "-"
+		(at 111.79 52.75 180)
 		(layer "F.SilkS")
 		(effects
@@
 		)
 	)
-	(gr_text "-"
+	(gr_text "+"
 		(at 110.36 55.26 180)
 		(layer "B.SilkS")
@@
 		)
 	)
-	(gr_text "+"
-		(at 110.6 53.74 270)
+	(gr_text "-"
+		(at 110.38 52.75 180)
 		(layer "B.SilkS")
 		(effects
@@
 	)
 	(segment
-		(start 110.475 58.42)
-		(end 113 55.895)
+		(start 110.43 58.42)
+		(end 113 55.85)
+		(width 0.2)
+		(layer "F.Cu")
+		(net 21)
+	)
+	(segment
+		(start 113 55.85)
+		(end 113 55.69)
 		(width 0.2)
 		(layer "F.Cu")
@@
 	(segment
 		(start 109.105 58.42)
-		(end 110.475 58.42)
+		(end 110.43 58.42)
 		(width 0.2)
 		(layer "F.Cu")
@@
 	(segment
 		(start 109.105 56.6)
+		(end 109.105 56.595)
+		(width 0.2)
+		(layer "F.Cu")
+		(net 22)
+	)
+	(segment
+		(start 109.105 56.6)
 		(end 109.105 56.565)
 		(width 0.2)
@@
 	)
 	(segment
-		(start 112.52 53.15)
+		(start 112.55 53.15)
 		(end 113 53.15)
 		(width 0.2)
@@
 	)
 	(segment
-		(start 109.105 56.565)
-		(end 112.52 53.15)
+		(start 109.105 56.595)
+		(end 112.55 53.15)
 		(width 0.2)
 		(layer "F.Cu")
@@
 	)
 	(segment
-		(start 107.475 56.68)
-		(end 107.555 56.6)
+		(start 106.36 58.43)
+		(end 107.545 58.43)
 		(width 0.2)
 		(layer "F.Cu")
@@
 	)
 	(segment
-		(start 99.805001 55.625001)
-		(end 98.25 55.625001)
+		(start 107.545 58.43)
+		(end 107.555 58.42)
 		(width 0.2)
 		(layer "F.Cu")
@@
 	)
 	(segment
-		(start 106.34 56.68)
-		(end 107.475 56.68)
+		(start 99.335001 56.025001)
+		(end 101.74 58.43)
 		(width 0.2)
 		(layer "F.Cu")
@@
 	)
 	(segment
-		(start 102.989998 75.01)
-		(end 102.024998 75.01)
+		(start 98.25 56.025001)
+		(end 99.335001 56.025001)
 		(width 0.2)
 		(layer "F.Cu")
@@
 	)
 	(segment
-		(start 106.34 56.68)
-		(end 100.86 56.68)
+		(start 101.74 58.43)
+		(end 106.36 58.43)
 		(width 0.2)
 		(layer "F.Cu")
@@
 	)
 	(segment
-		(start 100.86 56.68)
-		(end 99.805001 55.625001)
+		(start 103.01625 72.41)
+		(end 102.02875 72.41)
 		(width 0.2)
 		(layer "F.Cu")
@@
 	)
 	(via
-		(at 106.34 56.68)
+		(at 106.36 58.43)
 		(size 0.6)
 		(drill 0.3)
@@
 	)
 	(via
-		(at 102.989998 75.01)
+		(at 103.01625 72.41)
 		(size 0.6)
 		(drill 0.3)
@@
 	)
 	(segment
-		(start 104.13 70.88)
-		(end 104.13 73.869998)
-		(width 0.2)
-		(layer "B.Cu")
-		(net 25)
-	)
-	(segment
-		(start 110.09 64.92)
-		(end 104.13 70.88)
+		(start 103.01625 70.064276)
+		(end 103.01625 72.41)
 		(width 0.2)
 		(layer "B.Cu")
@@
 	)
 	(segment
-		(start 107.31 56.68)
-		(end 110.09 59.46)
+		(start 107.81 65.270526)
+		(end 103.01625 70.064276)
 		(width 0.2)
 		(layer "B.Cu")
@@
 	)
 	(segment
-		(start 104.13 73.869998)
-		(end 102.989998 75.01)
+		(start 107.05 58.43)
+		(end 107.81 59.19)
 		(width 0.2)
 		(layer "B.Cu")
@@
 	)
 	(segment
-		(start 106.34 56.68)
-		(end 107.31 56.68)
+		(start 107.81 59.19)
+		(end 107.81 65.270526)
 		(width 0.2)
 		(layer "B.Cu")
@@
 	)
 	(segment
-		(start 110.09 59.46)
-		(end 110.09 64.92)
+		(start 106.36 58.43)
+		(end 107.05 58.43)
 		(width 0.2)
 		(layer "B.Cu")
@@
 	)
 	(segment
-		(start 106.36 58.43)
-		(end 107.545 58.43)
+		(start 107.475 56.68)
+		(end 107.555 56.6)
 		(width 0.2)
 		(layer "F.Cu")
@@
 	)
 	(segment
-		(start 99.375 56.025)
-		(end 98.25 56.025)
+		(start 106.34 56.68)
+		(end 107.475 56.68)
 		(width 0.2)
 		(layer "F.Cu")
@@
 	)
 	(segment
-		(start 107.545 58.43)
-		(end 107.555 58.42)
+		(start 99.805001 55.625001)
+		(end 98.25 55.625001)
 		(width 0.2)
 		(layer "F.Cu")
@@
 	)
 	(segment
-		(start 103.01625 72.41)
-		(end 102.02875 72.41)
+		(start 100.86 56.68)
+		(end 99.805001 55.625001)
 		(width 0.2)
 		(layer "F.Cu")
@@
 	)
 	(segment
-		(start 106.36 58.43)
-		(end 101.78 58.43)
+		(start 102.989998 75.01)
+		(end 102.024998 75.01)
 		(width 0.2)
 		(layer "F.Cu")
@@
 	)
 	(segment
-		(start 101.78 58.43)
-		(end 99.375 56.025)
+		(start 106.34 56.68)
+		(end 100.86 56.68)
 		(width 0.2)
 		(layer "F.Cu")
@@
 	)
 	(via
-		(at 106.36 58.43)
+		(at 106.34 56.68)
 		(size 0.6)
 		(drill 0.3)
@@
 	)
 	(via
-		(at 103.01625 72.41)
+		(at 102.989998 75.01)
 		(size 0.6)
 		(drill 0.3)
@@
 	)
 	(segment
-		(start 103.01625 70.064276)
-		(end 103.01625 72.41)
+		(start 104.13 70.88)
+		(end 104.13 73.869998)
 		(width 0.2)
 		(layer "B.Cu")
@@
 	)
 	(segment
-		(start 107.81 65.270526)
-		(end 103.01625 70.064276)
+		(start 110.09 64.92)
+		(end 104.13 70.88)
 		(width 0.2)
 		(layer "B.Cu")
@@
 	)
 	(segment
-		(start 107.05 58.43)
-		(end 107.81 59.19)
+		(start 107.31 56.68)
+		(end 110.09 59.46)
 		(width 0.2)
 		(layer "B.Cu")
@@
 	)
 	(segment
-		(start 107.81 59.19)
-		(end 107.81 65.270526)
+		(start 104.13 73.869998)
+		(end 102.989998 75.01)
 		(width 0.2)
 		(layer "B.Cu")
@@
 	)
 	(segment
-		(start 106.36 58.43)
-		(end 107.05 58.43)
+		(start 106.34 56.68)
+		(end 107.31 56.68)
+		(width 0.2)
+		(layer "B.Cu")
+		(net 27)
+	)
+	(segment
+		(start 110.09 59.46)
+		(end 110.09 64.92)
 		(width 0.2)
 		(layer "B.Cu")

Commit message: WIP
Parts:
- removed REF**: OSHW-Logo_5.7x6mm_SilkScreen, Symbol:OSHW-Logo_5.7x6mm_SilkScreen
- removed kibuzzard-69BBD06F: G***, kibuzzard-69BBD06F
- added C22: 100nF, Capacitor_SMD:C_0603_1608Metric, F.Cu at (107.5, 64.6)
- added R4: 10K, Resistor_SMD:R_0603_1608Metric, F.Cu at (109.0, 62.2)
- added R7: 10K, Resistor_SMD:R_0603_1608Metric, F.Cu at (109.0, 60.7)
- added R8: 10K, Resistor_SMD:R_0603_1608Metric, F.Cu at (112.5, 60.7)
- added R9: 10K, Resistor_SMD:R_0603_1608Metric, F.Cu at (112.5, 62.2)
- added U3: TLV9002IDSGR, Doorman:WSON-8_L2.0-W2.0-P0.65-BL-EP, F.Cu at (110.8, 64.7)
- added kibuzzard-69DCDFB0: G***, kibuzzard-69DCDFB0, B.Cu at (86.5, 48.6)
- C12, C4: value 10uF -> 2.2uF
- C14, C8: footprint Capacitor_SMD:C_1206_3216Metric -> Capacitor_SMD:C_0603_1608Metric
- J2: moved to F.Cu
- R10, R6: value 200 -> 150R
- R15, R16, R17, R18, R19: value 33 -> 33R
- moved C8 19.3 mm to (102.0, 56.7)
- moved C14 15.5 mm to (102.0, 58.2)
- moved TP4 11.3 mm to (118.6, 56.0)
- moved TP3 10.7 mm to (118.7, 53.1)
- moved TP8 10.4 mm to (90.6, 62.8)
- moved C5 7.83 mm to (109.3, 50.6)
- moved C12 5.38 mm to (87.8, 68.5), turned to 180 degrees
- moved J1 5.08 mm to (113.0, 50.6), turned to 0 degrees
- moved C3 3.55 mm to (109.3, 53.2)
- moved R6 3.54 mm to (97.0, 72.2)
- moved R10 3.53 mm to (97.0, 74.7), turned to 0 degrees
- moved TP6 1.96 mm to (103.3, 63.5)
- moved C4 1.26 mm to (87.8, 64.8), turned to 180 degrees
- moved J2 1.07 mm to (84.7, 72.6)
- moved R14 1.06 mm to (105.9, 67.6)
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Connections:
- C14 pad 1: BUS_WIRE2 -> AUDIO_OUT_P
- C14 pad 2: Net-(C14-Pad2) -> Net-(D4-K)
- C8 pad 1: BUS_WIRE1 -> AUDIO_OUT_N
- C8 pad 2: Net-(C8-Pad2) -> Net-(D2-K)
- D2 pad 1: AUDIO_OUT_N -> Net-(D2-K)
- D4 pad 1: AUDIO_OUT_P -> Net-(D4-K)
- R10 pad 1: AUDIO_OUT_N -> Net-(D1-K)
- R10 pad 2: Net-(C8-Pad2) -> Net-(U3A-IN1-)
- R6 pad 1: AUDIO_OUT_P -> Net-(U3B-IN2-)
- R6 pad 2: Net-(C14-Pad2) -> Net-(D3-K)
- TP3 pad 1: AUDIO_OUT_N -> Net-(D2-K)
- TP4 pad 1: AUDIO_OUT_P -> Net-(D4-K)
Routing:
- net AUDIO_OUT_N: track 34.1 -> 3.40 mm, vias 2 -> 0
- net AUDIO_OUT_P: track 28.3 -> 3.86 mm, vias 2 -> 0
- net Net-(D1-K): track 25.1 -> 44.5 mm, vias 2 -> 4
- net Net-(D3-K): track 21.1 -> 37.9 mm, vias 2 -> 3
- net Net-(D2-K): track 0.00 -> 16.6 mm
- net AVDD: track 39.7 -> 55.8 mm, vias 3 -> 5
- net BUS_WIRE1: track 13.7 -> 2.52 mm, vias 2 -> 0
- net Net-(D4-K): track 0.00 -> 10.4 mm
- net BUS_WIRE2: track 16.8 -> 9.28 mm
- net PIN2: track 18.0 -> 12.4 mm, vias 1 -> 0
- net Net-(J1-Pin_2): track 5.36 -> 2.97 mm
- net Net-(J1-Pin_1): track 5.40 -> 3.31 mm
- net Net-(C14-Pad2): track 1.64 -> 0.00 mm
- net Net-(C8-Pad2): track 1.64 -> 0.00 mm
- net I2C_DAT: track 24.7 -> 23.1 mm
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Other:
- board size 31.4 x 29.6 mm -> 31.8 x 30.3 mm
- board text removed: "01"
- board text removed: "07"
- board text removed: "08"
- board text removed: "14"
