File: hardware/core_board/doorman_core_board.kicad_pcb (KiCad board)
At the start: 4 copper layers, 37.2 x 37.2 mm, 60 parts, among them J1 USB-C Connector, J10 VCC Test Pad, J2 Screw Terminals, J3 3V3 Test Pad, J4 Extension Board Connector, J5 Siedle BUS RX Test Pad, J6 BUS Test Pad, J7 BUS RX Test Pad, J8 TX Test Pad, J9 RX Test Pad, Q1 BC847BPN, Q2 BC817-40, Q3 BC817-40, Q4 BC817-40, Q6 BC847BPN, SW1 Button, SW2 Button, U2 AP63203WU, U3 GAQY252G3S, U4 ESP32-S3-MINI-1

Commit message: Change structure
Parts:
- added D9: 4.3V, Diode_SMD:D_SOD-123, B.Cu at (105.1, 61.1)
- added R19: 1M, Resistor_SMD:R_0603_1608Metric, B.Cu at (108.5, 51.7)
- added R20: 120K, Resistor_SMD:R_0603_1608Metric, B.Cu at (106.8, 49.6)
- added kibuzzard-69BAB542: G***, kibuzzard-69BAB542, F.Cu at (111.8, 60.5)
- added kibuzzard-69BAB57C: G***, kibuzzard-69BAB57C, F.Cu at (111.9, 58.1)
- added kibuzzard-69BAB7C5: G***, kibuzzard-69BAB7C5, F.Cu at (88.5, 60.2)
- added kibuzzard-69BABEC4: G***, kibuzzard-69BABEC4, F.Cu at (111.8, 64.2)
- added kibuzzard-69BACA52: G***, kibuzzard-69BACA52, F.Cu at (112.0, 36.9)
- added kibuzzard-69BACA90: G***, kibuzzard-69BACA90, F.Cu at (85.5, 36.9)
- added kibuzzard-69BACB1F: G***, kibuzzard-69BACB1F, F.Cu at (111.8, 48.7)
- added kibuzzard-69BACB5F: G***, kibuzzard-69BACB5F, F.Cu at (111.8, 68.2)
- added kibuzzard-69BD6C3C: G***, kibuzzard-69BD6C3C, F.Cu at (111.8, 52.8)
- added kibuzzard-69BD6F46: G***, kibuzzard-69BD6F46, F.Cu at (111.8, 55.3)
- D3: value 5.1V -> 4.3V
- R12: value 47K5 -> 10K
- R18: value 1K -> 10K; footprint Resistor_SMD:R_0402_1005Metric -> Resistor_SMD:R_0603_1608Metric
- R5: value 47K5 -> 59K
- moved J6 1.27 mm to (108.2, 63.4)
- moved R18 0.32 mm to (90.7, 55.1)
- moved J5 0.13 mm to (89.8, 57.3)
Connections:
- J2 pad 7: IO41 -> ERT
- U4 pad 37: IO41 -> unconnected-(U4-IO41-Pad37)
- U4 pad 8: unconnected-(U4-IO4-Pad8) -> ERT_DETECT
Routing:
- net ERT_DETECT: track 0.00 -> 18.1 mm, vias 0 -> 1
- net IO41: track 13.5 -> 0.00 mm, vias 1 -> 0
- net ERT: track 0.00 -> 6.84 mm
- net BUS_WIRE1: track 25.8 -> 28.4 mm
- net Net-(D9-K): track 16.0 -> 16.8 mm
- net BUS_RX_IHB: track 13.0 -> 12.3 mm
- net IO40: track 14.0 -> 14.6 mm
Other:
- board text added: "IO04"
- board text removed: "B U S"
- board text removed: "BUS PWR"
- board text removed: "G"
- board text removed: "I40"
- board text removed: "I41"
- board text removed: "IO41"
- board text removed: "P"
- board text removed: "PRG"
- board text removed: "RELAY"
- board text removed: "RST"
- board text removed: "STATUS LEDS"

Commit message: Update PCB files
Parts:
- moved C8 0.48 mm to (82.6, 55.4)
- moved R3 0.43 mm to (93.2, 68.3)
- moved J9 0.35 mm to (101.5, 45.0)
Routing:
- net Net-(D6-K): track 4.31 -> 3.81 mm
- net GND: vias 140 -> 141

Commit message: WIP
Parts:
- added R21: 100K, Resistor_SMD:R_0603_1608Metric, B.Cu at (106.2, 62.8)
- added R25: 10K, Resistor_SMD:R_0603_1608Metric, B.Cu at (103.3, 62.8)
- R19: value 1M -> 100K
- R2: value 2K2 -> 1K
- R20: value 120K -> 10K
- moved D9 1.81 mm to (106.9, 60.9)
- moved J6 1.61 mm to (107.1, 64.6)
- moved R2 1.22 mm to (107.1, 55.7)
- moved R18 0.41 mm to (90.5, 54.8)
- moved J10 0.28 mm to (88.3, 60.0)
- moved U4 0.05 mm to (98.0, 48.9)
Connections:
- net I2C_CLK renamed IO13
- net I2C_DAT renamed IO14
- J4 pad 11: IO12 -> VBUS
- U4 pad 14: BUS_RX_IHB -> BUS_VOLTAGE
- U4 pad 15: unconnected-(U4-IO11-Pad15) -> BUS_RX_IHB
- U4 pad 16: IO12 -> unconnected-(U4-IO12-Pad16)
Routing:
- net BUS_VOLTAGE: track 0.00 -> 21.7 mm, vias 0 -> 1
- net IO12: track 15.6 -> 0.00 mm, vias 2 -> 0
- net VBUS: track 38.3 -> 43.7 mm, vias 3 -> 4
- net Net-(Q1A-C1): track 15.7 -> 11.8 mm
- net BUS_TX_TC: track 18.2 -> 17.2 mm
- net GND: vias 141 -> 149
Other:
- board text added: "3.3V"
- board text added: "ESP32-S3"
- board text added: "ET"
- board text removed: "IO04"
- board text removed: "IO48"

Commit message: chore: Update pcb files core board 2.2.0
Parts:
- removed D3, D9: 4.3V, Diode_SMD:D_SOD-123
- removed R21: 100K, Resistor_SMD:R_0603_1608Metric
- removed R25: 10K, Resistor_SMD:R_0603_1608Metric
- added R26: 100K, Resistor_SMD:R_0603_1608Metric, B.Cu at (92.9, 58.8)
- added R27: 100K, Resistor_SMD:R_0603_1608Metric, B.Cu at (90.6, 63.0)
- C8: value 10uF -> 1uF
- R17, R18: value 10K -> 100K
- R22, R3: moved to B.Cu
- moved R3 9.74 mm to (102.4, 71.7), turned to 0 degrees
- moved R18 8.36 mm to (95.1, 61.7), turned to 90 degrees
- moved R22 4.87 mm to (97.7, 71.8), turned to 180 degrees
- moved R17 2.32 mm to (93.5, 65.4), turned to 0 degrees
- moved J10 2.30 mm to (88.2, 57.6)
- moved J6 1.95 mm to (108.5, 63.2)
- moved J5 1.82 mm to (90.3, 55.5)
- moved Q6 1.62 mm to (92.9, 61.2), turned to 90 degrees
- moved R16 0.89 mm to (93.5, 63.9), turned to 180 degrees
- moved R2 0.20 mm to (106.9, 55.7)
Connections:
- Q6 pad 1: unconnected-(Q6A-E1-Pad1) -> GND
- Q6 pad 2: unconnected-(Q6A-B1-Pad2) -> Net-(Q6A-B1)
- Q6 pad 5: Net-(D3-K) -> Net-(Q6A-C1)
- Q6 pad 6: unconnected-(Q6A-C1-Pad6) -> Net-(Q6A-C1)
- R16 pad 1: VBUS -> BUS_VOLTAGE
- R16 pad 2: Net-(D3-K) -> GND
- R17 pad 1: Net-(D3-K) -> VBUS
- R17 pad 2: GND -> BUS_VOLTAGE
- R18 pad 1: BUS_RX_IHB -> BUS_VOLTAGE
- R18 pad 2: GND -> Net-(Q6A-B1)
Routing:
- net Net-(D3-K): track 6.57 -> 0.00 mm
- net BUS_VOLTAGE: track 21.7 -> 16.5 mm
- net Net-(J1-CC2): track 10.7 -> 6.27 mm, vias 0 -> 1
- net VBUS: track 43.7 -> 39.4 mm
- net Net-(Q6A-B1): track 0.00 -> 3.07 mm
- net /VCC_IN: track 52.2 -> 49.9 mm
- net Net-(Q6A-C1): track 0.00 -> 2.16 mm
- net BUS_RX_IHB: track 12.6 -> 11.5 mm
- net Net-(Q1B-B2): track 16.8 -> 15.7 mm
- net Net-(J1-CC1): track 6.49 -> 5.78 mm, vias 0 -> 1
- net GND: vias 149 -> 146
Other:
- board text added: "5-30VDC"
- board text removed: "5-30V DC"

Commit message: chore: Update PCB files 2.2.0
Parts:
- removed Q4: BC817-40, Package_TO_SOT_SMD:SOT-23
- added J11: TC BUS RX Test Pad, TestPoint:TestPoint_Pad_D1.0mm, B.Cu at (106.2, 61.2)
- added J12: Bus Voltage Test Pad, TestPoint:TestPoint_Pad_D1.0mm, B.Cu at (96.4, 64.0)
- added Q5: IRLML0030, Package_TO_SOT_SMD:SOT-23, B.Cu at (85.6, 63.9)
- added R21: 10K, Resistor_SMD:R_0603_1608Metric, B.Cu at (83.1, 64.0)
- added R24: 10K, Resistor_SMD:R_0603_1608Metric, B.Cu at (84.9, 71.3)
- Q3: value BC817-40 -> IRLML0030
- R14, R4: value 10K -> 1K; footprint Resistor_SMD:R_0603_1608Metric -> Resistor_SMD:R_0402_1005Metric
- moved Q3 5.00 mm to (85.0, 68.9), turned to 0 degrees
- moved R14 4.44 mm to (82.3, 61.0)
- moved R15 2.31 mm to (89.4, 66.5)
- moved R13 2.27 mm to (89.4, 68.8)
- moved D1 1.15 mm to (91.6, 70.2), turned to -90 degrees
- moved R4 0.87 mm to (84.5, 61.0)
Connections:
- Q3 pad 1: Net-(Q3-B) -> Net-(Q3-G)
- R14 pad 1: BUS_TX_IHB -> BUS_TX_IHB_CAR
- R14 pad 2: Net-(Q4-B) -> Net-(Q3-G)
- R4 pad 1: BUS_TX_IHB_CAR -> BUS_TX_IHB
- R4 pad 2: Net-(Q3-B) -> Net-(Q5-G)
Routing:
- net Net-(Q3-G): track 0.00 -> 11.3 mm
- net BUS_TX_IHB: track 19.9 -> 13.9 mm
- net Net-(Q4-B): track 4.77 -> 0.00 mm
- net /VCC_IN: track 49.9 -> 46.7 mm
- net +3.3V: track 83.7 -> 86.8 mm
- net Net-(Q5-G): track 0.00 -> 3.12 mm
- net +5V: track 16.3 -> 19.4 mm
- net Net-(Q3-D): track 4.24 -> 2.00 mm
- net BUS_VOLTAGE: track 16.5 -> 18.7 mm
- net Net-(Q3-B): track 1.85 -> 0.00 mm
- net BUS_TX_IHB_CAR: track 13.9 -> 15.7 mm
- net Net-(Q5-D): track 2.00 -> 3.53 mm
- net Net-(Q1B-B2): track 15.7 -> 17.1 mm
- net VBUS: track 39.4 -> 38.8 mm
- net GND: vias 146 -> 152
Other:
- board text added: "VDA"
- board text added: "VDTC"

Commit message: chore: Update pcb files 2.2.0
Parts:
- added J13: ERT Test Pad, TestPoint:TestPoint_Pad_D1.0mm, B.Cu at (95.0, 46.8)
- added R23: 10K, Resistor_SMD:R_0603_1608Metric, B.Cu at (109.4, 56.9)
- D1: moved to B.Cu
- D2: value MB6S -> MB10S
- R9: value 150R -> 120R
- moved D1 5.49 mm to (97.0, 69.7), turned to 0 degrees
- moved J7 3.25 mm to (93.0, 50.0)
- moved J11 2.74 mm to (107.6, 58.9)
- moved R27 1.88 mm to (89.7, 61.4)
- moved J6 1.05 mm to (108.7, 62.2)
- moved G*** 0.92 mm to (114.7, 44.4)
- turned D2 to -90 degrees
Connections:
- D2 pad 1: BUS_WIRE1 -> VBUS
- D2 pad 2: BUS_WIRE2 -> GND
- D2 pad 3: VBUS -> BUS_WIRE1
- D2 pad 4: GND -> BUS_WIRE2
Routing:
- net +5V: track 19.4 -> 11.7 mm, vias 3 -> 2
- net BUS_RX: track 31.8 -> 28.3 mm
- net ERT_DETECT: track 18.6 -> 20.7 mm
- net /VCC_IN: track 46.7 -> 48.6 mm
- net BUS_WIRE1: track 28.4 -> 26.5 mm
- net Net-(Q1A-C1): track 12.1 -> 13.3 mm
- net BUS_TX_IHB_CAR: track 15.7 -> 14.8 mm
- net BUS_TX_IHB: track 13.9 -> 13.0 mm
- net +3.3V: track 86.8 -> 86.1 mm
- net VBUS: track 38.8 -> 39.3 mm
- net GND: vias 152 -> 153
Other:
- outline, holes or cut-outs redrawn
- board text added: "IO04"
- board text added: "VDERT"
- board text added: "VDIHB"
- board text removed: "ET"
- board text removed: "VDA"
