File: hardware/core_board/doorman_core_board.kicad_pcb (KiCad board)
At the start: 4 copper layers, 37.2 x 37.2 mm, 79 parts, among them J1 USB-C Connector, J10 VCC Test Pad, J11 TC BUS RX Test Pad, J12 Bus Voltage Test Pad, J13 ERT Test Pad, J2 Screw Terminals, J3 3V3 Test Pad, J4 Extension Board Connector, J5 Siedle BUS RX Test Pad, J6 BUS Test Pad, J7 BUS RX Test Pad, J8 TX Test Pad, J9 RX Test Pad, Q1 BC847BPN, Q2 BC817-40, Q3 IRLML0030, Q5 IRLML0030, Q6 BC847BPN, SW1 Button, SW2 Button, U2 AP63203WU, U3 GAQY252G3S, U4 ESP32-S3-MINI-1

Commit message: PCB rev 2.2.1
Parts:
- Q3, Q5: value IRLML0030 -> IRLML0040
- R14, R4: value 1K -> 0
Changed lines of the file:
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@@
 		(title "Doorman S3")
 		(date "2026-05-20")
-		(rev "2.2.0")
+		(rev "2.2.1")
 		(comment 1 "Compatible with TCS (DE), Koch (CH), Scantron (DK), Niko, JUNG (DE) and SIEDLE (DE)")
 		(comment 3 "For TC:BUS and IN-HOME-BUS based intercom systems")
@@
 			)
 		)
-		(property "Value" "1K"
+		(property "Value" "0"
 			(at 0 -1.17 90)
 			(layer "B.Fab")
@@
 			)
 		)
-		(property "Description" "-55℃~+155℃ 1kΩ 50V 62.5mW Thick Film Resistor ±1% ±100ppm/℃ 0402 Chip Resistor - Surface Mount ROHS"
+		(property "Description" "-55℃~+155℃ 0Ω 50V 62.5mW Thick Film Resistor ±1% ±800ppm/℃ 0402 Chip Resistor - Surface Mount ROHS"
 			(at 0 0 90)
 			(layer "B.Fab")
@@
 			)
 		)
-		(property "LCSC" "C11702"
+		(property "LCSC" "C17168"
 			(at 0 0 90)
 			(unlocked yes)
@@
 			)
 		)
-		(property "MPN" "0402WGF1001TCE"
+		(property "MPN" "0402WGF0000TCE"
 			(at 0 0 90)
 			(unlocked yes)
@@
 			)
 		)
-		(property "Value" "IRLML0030"
+		(property "Value" "IRLML0040"
 			(at 0 -2.4 90)
 			(layer "B.Fab")
@@
 			)
 		)
-		(property "Description" "-55℃~+150℃ 1 N-channel 1.4W 28mΩ@10V 30V 5.8A 700mV 78pF 825pF SOT-23 MOSFETs ROHS"
+		(property "Description" "-55℃~+150℃ 1 N-channel 1.3W 2.5V 266pF 29pF 3.6A 3.9nC 40V 56mΩ@10V SOT-23 MOSFETs ROHS"
 			(at 0 0 90)
 			(layer "B.Fab")
@@
 			)
 		)
-		(property "MPN" "IRLML0030TRPBF-HXY"
+		(property "MPN" "IRLML0040"
 			(at 0 0 270)
 			(unlocked yes)
@@
 			)
 		)
-		(property "LCSC" "C6285737"
+		(property "LCSC" "C5364305"
 			(at 0 0 270)
 			(unlocked yes)
@@
 			)
 		)
-		(property "Value" "1K"
+		(property "Value" "0"
 			(at 0 -1.17 90)
 			(layer "B.Fab")
@@
 			)
 		)
-		(property "Description" "-55℃~+155℃ 1kΩ 50V 62.5mW Thick Film Resistor ±1% ±100ppm/℃ 0402 Chip Resistor - Surface Mount ROHS"
+		(property "Description" "-55℃~+155℃ 0Ω 50V 62.5mW Thick Film Resistor ±1% ±800ppm/℃ 0402 Chip Resistor - Surface Mount ROHS"
 			(at 0 0 90)
 			(layer "B.Fab")
@@
 			)
 		)
-		(property "LCSC" "C11702"
+		(property "LCSC" "C17168"
 			(at 0 0 90)
 			(unlocked yes)
@@
 			)
 		)
-		(property "MPN" "0402WGF1001TCE"
+		(property "MPN" "0402WGF0000TCE"
 			(at 0 0 90)
 			(unlocked yes)
@@
 			)
 		)
-		(property "Value" "IRLML0030"
+		(property "Value" "IRLML0040"
 			(at 0 -2.4 0)
 			(layer "B.Fab")
@@
 			)
 		)
-		(property "Description" "-55℃~+150℃ 1 N-channel 1.4W 28mΩ@10V 30V 5.8A 700mV 78pF 825pF SOT-23 MOSFETs ROHS"
+		(property "Description" "-55℃~+150℃ 1 N-channel 1.3W 2.5V 266pF 29pF 3.6A 3.9nC 40V 56mΩ@10V SOT-23 MOSFETs ROHS"
 			(at 0 0 0)
 			(layer "B.Fab")
@@
 			)
 		)
-		(property "LCSC" "C6285737"
+		(property "LCSC" "C5364305"
 			(at 0 0 0)
 			(unlocked yes)
@@
 			)
 		)
-		(property "MPN" "IRLML0030TRPBF-HXY"
+		(property "MPN" "IRLML0040"
 			(at 0 0 0)
 			(unlocked yes)
