File: hardware/core_board/doorman_core_board.kicad_sch (KiCad schematic)
At the start: 66 parts, among them J1 USB-C Connector, J10 VCC Test Pad, J11 TC BUS RX Test Pad, J12 Bus Voltage Test Pad, J13 ERT Test Pad, J2 Screw Terminals, J3 3V3 Test Pad, J4 Extension Board Connector, J5 Siedle BUS RX Test Pad, J6 BUS Test Pad, J7 BUS RX Test Pad, J8 TX Test Pad, J9 RX Test Pad, Q1 BC847BPN, Q2 BC817-40, Q3 IRLML0030, Q5 IRLML0030, Q6 BC847BPN, SW1 Button, SW2 Button, U2 AP63203WU, U3 GAQY252G3S, U4 ESP32-S3-MINI-1

Commit message: PCB rev 2.2.1
Parts:
- Q3, Q5: value IRLML0030 -> IRLML0040; LCSC C6285737 -> C5364305; MPN IRLML0030TRPBF-HXY -> IRLML0040
- R14, R4: value 1K -> 0; LCSC C11702 -> C17168; MPN 0402WGF1001TCE -> 0402WGF0000TCE
Other:
- note added: "TC:BUS Data(Idle ~22-24V) Low 8V, High 24V In-Home-Bus Carrier (Idle ~27-30V) Low 3V, High 30V(max) 1+n (Idle ~15V) Low ~15V, High ~24V Triggers at ~15.5V"
- note removed: "TC:BUS Data(Idle ~22-24V) Low 8V, High 24V In-Home-Bus Carrier (Idle ~27-30V) Low 3V, High 30V(max) 1+n (Idle ~15V) Low ~15V, High ~24V"
Changed lines of the file:
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@@
 		(title "Doorman S3")
 		(date "2026-05-20")
-		(rev "2.2.0")
+		(rev "2.2.1")
 		(comment 1 "Compatible with TCS (DE), Koch (CH), Scantron (DK), Niko, JUNG (DE) and SIEDLE (DE)")
 		(comment 3 "For TC:BUS and IN-HOME-BUS based intercom systems")
@@
 		)
 	)
-	(text "TC:BUS Data(Idle ~22-24V)\nLow 8V, High 24V\n\nIn-Home-Bus Carrier (Idle ~27-30V)\nLow 3V, High 30V(max)\n\n1+n (Idle ~15V)\nLow ~15V, High ~24V"
+	(text "TC:BUS Data(Idle ~22-24V)\nLow 8V, High 24V\n\nIn-Home-Bus Carrier (Idle ~27-30V)\nLow 3V, High 30V(max)\n\n1+n (Idle ~15V)\nLow ~15V, High ~24V\n\nTriggers at ~15.5V"
 		(exclude_from_sim no)
-		(at 115.062 231.648 0)
+		(at 115.062 233.68 0)
 		(effects
 			(font
@@
 			)
 		)
-		(property "Value" "IRLML0030"
+		(property "Value" "IRLML0040"
 			(at 203.454 99.568 0)
 			(effects
@@
 			)
 		)
-		(property "Description" "-55℃~+150℃ 1 N-channel 1.4W 28mΩ@10V 30V 5.8A 700mV 78pF 825pF SOT-23 MOSFETs ROHS"
+		(property "Description" "-55℃~+150℃ 1 N-channel 1.3W 2.5V 266pF 29pF 3.6A 3.9nC 40V 56mΩ@10V SOT-23 MOSFETs ROHS"
 			(at 198.12 99.06 0)
 			(effects
@@
 			)
 		)
-		(property "MPN" "IRLML0030TRPBF-HXY"
+		(property "MPN" "IRLML0040"
 			(at 198.12 99.06 0)
 			(effects
@@
 			)
 		)
-		(property "LCSC" "C6285737"
+		(property "LCSC" "C5364305"
 			(at 198.12 99.06 0)
 			(effects
@@
 			)
 		)
-		(property "Value" "1K"
+		(property "Value" "0"
 			(at 186.69 139.7 90)
 			(effects
@@
 			)
 		)
-		(property "Description" "-55℃~+155℃ 1kΩ 50V 62.5mW Thick Film Resistor ±1% ±100ppm/℃ 0402 Chip Resistor - Surface Mount ROHS"
+		(property "Description" "-55℃~+155℃ 0Ω 50V 62.5mW Thick Film Resistor ±1% ±800ppm/℃ 0402 Chip Resistor - Surface Mount ROHS"
 			(at 186.69 139.7 0)
 			(effects
@@
 			)
 		)
-		(property "LCSC" "C11702"
+		(property "LCSC" "C17168"
 			(at 186.69 139.7 0)
 			(effects
@@
 			)
 		)
-		(property "MPN" "0402WGF1001TCE"
+		(property "MPN" "0402WGF0000TCE"
 			(at 186.69 139.7 0)
 			(effects
@@
 			)
 		)
-		(property "Value" "IRLML0030"
+		(property "Value" "IRLML0040"
 			(at 203.454 140.2081 0)
 			(effects
@@
 			)
 		)
-		(property "Description" "-55℃~+150℃ 1 N-channel 1.4W 28mΩ@10V 30V 5.8A 700mV 78pF 825pF SOT-23 MOSFETs ROHS"
+		(property "Description" "-55℃~+150℃ 1 N-channel 1.3W 2.5V 266pF 29pF 3.6A 3.9nC 40V 56mΩ@10V SOT-23 MOSFETs ROHS"
 			(at 198.12 139.7 0)
 			(effects
@@
 			)
 		)
-		(property "LCSC" "C6285737"
+		(property "LCSC" "C5364305"
 			(at 198.12 139.7 0)
 			(effects
@@
 			)
 		)
-		(property "MPN" "IRLML0030TRPBF-HXY"
+		(property "MPN" "IRLML0040"
 			(at 198.12 139.7 0)
 			(effects
@@
 			)
 		)
-		(property "Value" "1K"
+		(property "Value" "0"
 			(at 186.69 99.06 90)
 			(effects
@@
 			)
 		)
-		(property "Description" "-55℃~+155℃ 1kΩ 50V 62.5mW Thick Film Resistor ±1% ±100ppm/℃ 0402 Chip Resistor - Surface Mount ROHS"
+		(property "Description" "-55℃~+155℃ 0Ω 50V 62.5mW Thick Film Resistor ±1% ±800ppm/℃ 0402 Chip Resistor - Surface Mount ROHS"
 			(at 186.69 99.06 0)
 			(effects
@@
 			)
 		)
-		(property "LCSC" "C11702"
+		(property "LCSC" "C17168"
 			(at 186.69 99.06 0)
 			(effects
@@
 			)
 		)
-		(property "MPN" "0402WGF1001TCE"
+		(property "MPN" "0402WGF0000TCE"
 			(at 186.69 99.06 0)
 			(effects
